File: audio.kicad_sch (KiCad schematic)
At the start: 38 parts, among them IC1 TAC5212IRGER, J16 Debug, J18 Jack 6.35mm, J19 Jack 6.35mm, J20 Jack 6.35mm, J22 Jack 6.35mm, U14 OPA1656ID, U7 74AHCT1G32SE-7

Commit message: updated docs from chatgpt discussions.
Parts:
- added C64: 100nF, Capacitor_SMD:C_1206_3216Metric_Pad1.33x1.80mm_HandSolder, symbol Device:C_Small
Connections:
- net at C56.2, R33.1, U14.3 (+): now also C64.2
- net at C56.1, D3.2 (A2), J18.T: now also C64.1
Other:
- moved on the sheet: C56, C57, C58, C62, D3, J18, R33, R34, R37, R38, R39, R40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

Commit message: added datasheets - wired up line level input components.
Parts:
- removed JP4: SJP, symbol Jumper:SolderJumper_2_Bridged
Connections:
- net in_L+ is gone; now on an unnamed net: J22.T
- net in_L- is gone; now on an unnamed net: J22.R
- net GND: now also J22.RN, J22.S, J22.TN, R41.2, R42.1
- net at R41.1: now also C62.1
- net at C63.1: now also R42.2
- net at C63.2: now also R44.2
- net TAC_IN2P: now reaches R43.1
- net TAC_IN2P: now also IC1.17 (IN2P)
- net at R43.2: now also C62.2
- net TAC_IN2M: now reaches R44.1
- net TAC_IN2M: now also IC1.18 (IN2M)
- no-connect marks 44 -> 45
Other:
- moved on the sheet: C61, C62, C63, CM1A, J22, R41, R42, R43, R44, U14C

Commit message: Supply work on TAC5212
Parts:
- added C65, C66, C70: 100n, Capacitor_SMD:C_0603_1608Metric, symbol Device:C_Small
- added C67, C68: 10u, Capacitor_SMD:C_0805_2012Metric, symbol Device:C_Small
- added C69: 1u, Capacitor_SMD:C_0805_2012Metric, symbol Device:C_Small
Connections:
- net GND: now also IC1.25 (VSS_1), IC1.A1 (VSS_2), IC1.A2 (VSS_3), IC1.A3 (VSS_4), IC1.A4 (VSS_5), C65.2, C66.2, C67.2, C68.2, C69.2, C70.2
- net at IC1.1 (DREG): now also C65.1
- net 3V3_CODEC: now reaches IC1.23 (AVDD)
- net 3V3_CODEC: now also C66.1, C67.1
- net at IC1.24 (VREF): now also C69.1
- net +3V3: now reaches IC1.6 (IOVDD)
- net +3V3: now also C68.1, C70.1
- net audio_in_stereo: no longer names the net of CM1.48 (GPIO27)
- no-connect marks 45 -> 47
Other:
- company: https://github.com/pedalboard -> https://github.com/arjepsen/Pedalboard-integrated-audio
- moved on the sheet: IC1, R41, R42

Commit message: Checkpoint before CM5 connectivity migration
Parts:
- removed JP5, JP6: SJP, symbol Jumper:SolderJumper_2_Open
- added C73, C74: 220uF, Capacitor_THT:CP_Radial_D6.3mm_P2.50mm, symbol Device:C_Polarized_Small_US
- added C75, C77: 4.7uF, Capacitor_SMD:C_1206_3216Metric, symbol Device:C_Small
- added C76, C78: 2.2nF, Capacitor_SMD:C_0603_1608Metric, symbol Device:C_Small
- added D4, D5, D8, D9: H5VUD5BB, Diode_SMD:D_SOD-523, symbol Device:D_TVS
- added J13: Headphones 3.5mm, Connector_Audio:Jack_3.5mm_CUI_SJ1-3525N_Horizontal, symbol Connector_Audio:AudioJack3_SwitchTR
- added R45, R46: 10k, Resistor_SMD:R_0603_1608Metric, symbol Device:R_Small
- added R47, R49: 470R, Resistor_SMD:R_0603_1608Metric, symbol Device:R_Small
- added R48, R50: 100k, Resistor_SMD:R_0603_1608Metric, symbol Device:R_Small
Connections:
- net GND_out is gone; now on net GND: J20.S
- net GND: now also IC1.13 (ADDR), J19.S, J20.R, C76.2, C78.2, D4.1 (A1), D5.1 (A1), D8.1 (A1), D9.1 (A1), J13.S, R45.2, R46.2, R48.2, R50.2
- net audio_pcm_clk: now also IC1.2 (BCLK)
- net audio_pcm_din: now also IC1.4 (DOUT)
- net audio_pcm_dout: now also IC1.5 (DIN)
- net audio_pcm_fs: now also IC1.3 (FSYNC)
- net conf_i2c_scl: now also IC1.7 (SCL)
- net conf_i2c_sda: now also IC1.8 (SDA)
- net at J19.T: now also C76.1, D9.2 (A2), R47.1, R48.1
- net at J20.T: now also C78.1, D8.2 (A2), R49.1, R50.1
- net TAC_OUT1M: now reaches IC1.19 (OUT1M)
- net TAC_OUT1M: now also C77.1
- net TAC_OUT1P: now reaches IC1.20 (OUT1P)
- net TAC_OUT1P: now also C75.1
- net TAC_OUT2P: now reaches IC1.21 (OUT2P)
- net TAC_OUT2P: now also C73.1
- net TAC_OUT2M: now reaches IC1.22 (OUT2M)
- net TAC_OUT2M: now also C74.1
- new net: C77.2, R49.2
- new net: C74.2, D5.2 (A2), J13.R, R46.1
- new net: C73.2, D4.2 (A2), J13.T, R45.1
- new net: C75.2, R47.2
- no-connect marks 47 -> 55
Other:
- note removed: "JP4 and JP6: Close to support differential output. HIFIberry has 5V on these outputs!"
- moved on the sheet: C65, C66, C67, C68, C69, C70, IC1, J19, J20, JP3

Commit message: Changed to CM5, removed unnecessary USB chips, Changing RP2024 to STM32.
Parts:
- removed CM1: CM4, Pedalboard Library:Raspberry-Pi-4-Compute-Module, symbol pedalboard:CM4
- removed D7: LED R, LED_SMD:LED_0805_2012Metric, symbol Device:LED
- removed J16: Debug, Connector_PinHeader_2.54mm:PinHeader_1x03_P2.54mm_Vertical, symbol Connector:Conn_01x03_Pin
- removed JP3: SJP, symbol Jumper:SolderJumper_2_Bridged
- removed R17: 2K2, Resistor_SMD:R_0805_2012Metric, symbol Device:R_Small
- removed U7: 74AHCT1G32SE-7, Package_TO_SOT_SMD:SOT-353_SC-70-5, symbol pedalboard:74AHCT1G32SE-7
- added CM2: ComputeModule5-CM5, CM5IO:Raspberry-Pi-5-Compute-Module, symbol CM5IO:ComputeModule5-CM5
- added R51, R52: 4.7k, Resistor_SMD:R_0603_1608Metric, symbol Device:R_Small
Connections:
- net +5VP: now also CM2.77 (+5v_(Input)), CM2.79 (+5v_(Input)), CM2.81 (+5v_(Input)), CM2.83 (+5v_(Input)), CM2.85 (+5v_(Input)), CM2.87 (+5v_(Input))
- net CM_BOOT: now also CM2.93 (nRPIBOOT)
- net GND: now also J19.SN, CM2.1 (GND), CM2.13 (GND), CM2.14 (GND), CM2.2 (GND), CM2.22 (GND), CM2.23 (GND), CM2.32 (GND), CM2.33 (GND), CM2.42 (GND), CM2.43 (GND), CM2.52 (GND), CM2.53 (GND), CM2.59 (GND), CM2.60 (GND), CM2.65 (GND), CM2.66 (GND), CM2.7 (GND), CM2.71 (GND), CM2.74 (GND), CM2.8 (GND), CM2.98 (GND)
- net audio_pcm_clk: now also CM2.49 (GPIO18)
- net audio_pcm_din: now also CM2.27 (GPIO20)
- net audio_pcm_dout: now also CM2.25 (GPIO21)
- net audio_pcm_fs: now also CM2.26 (GPIO19)
- net conf_i2c_scl: now also CM2.56 (GPIO3), R52.2
- net conf_i2c_sda: now also CM2.58 (GPIO2), R51.1
- net CM4_3V renamed CM5_3V
- net CM5_3V: now also CM2.78 (GPIO_VREF(1.8v/3.3v_Input)), CM2.84 (+3.3v_(Output)), CM2.86 (+3.3v_(Output)), R51.2, R52.1
- net CM4_LED_ACT renamed CM5_LED_ACT
- net CM5_LED_ACT: now also CM2.21 (LED_nACT)
- new net CM5_UART_RX: CM2.51 (GPIO15)
- new net CM5_UART_TX: CM2.55 (GPIO14)
- no-connect marks 55 -> 17
Other:
- moved on the sheet: C56, C57, C58, C61, C62, C63, C64, C65, C66, C67, C68, C69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

Commit message: add more cap
Parts:
- added C79: 10u, Capacitor_SMD:C_0805_2012Metric, symbol Device:C_Small
Connections:
- net GND: now also C79.2
- net at C65.1, IC1.1 (DREG): now also C79.1
Changed lines of the file:
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@@
 	)
 	(junction
+		(at 250.19 49.53)
+		(diameter 0)
+		(color 0 0 0 0)
+	)
+	(junction
 		(at 269.24 152.4)
 		(diameter 0)
@@
 	)
 	(junction
+		(at 265.43 49.53)
+		(diameter 0)
+		(color 0 0 0 0)
+	)
+	(junction
 		(at 270.51 124.46)
 		(diameter 0)
@@
 	(wire
 		(pts
+			(xy 265.43 49.53) (xy 267.97 49.53)
+		)
+		(stroke
+			(width 0)
+			(type default)
+		)
+	)
+	(wire
+		(pts
 			(xy 80.01 180.34) (xy 93.98 180.34)
 		)
@@
 	(wire
 		(pts
+			(xy 250.19 45.72) (xy 250.19 49.53)
+		)
+		(stroke
+			(width 0)
+			(type default)
+		)
+	)
+	(wire
+		(pts
 			(xy 105.41 91.44) (xy 109.22 91.44)
 		)
@@
 	(wire
 		(pts
+			(xy 259.08 45.72) (xy 265.43 45.72)
+		)
+		(stroke
+			(width 0)
+			(type default)
+		)
+	)
+	(wire
+		(pts
 			(xy 110.49 114.3) (xy 114.3 114.3)
 		)
@@
 	(wire
 		(pts
-			(xy 259.08 49.53) (xy 267.97 49.53)
+			(xy 259.08 49.53) (xy 265.43 49.53)
 		)
 		(stroke
@@
 	(wire
 		(pts
+			(xy 265.43 45.72) (xy 265.43 49.53)
+		)
+		(stroke
+			(width 0)
+			(type default)
+		)
+	)
+	(wire
+		(pts
 			(xy 102.87 185.42) (xy 111.76 185.42)
 		)
@@
 	(wire
 		(pts
+			(xy 254 45.72) (xy 250.19 45.72)
+		)
+		(stroke
+			(width 0)
+			(type default)
+		)
+	)
+	(wire
+		(pts
 			(xy 25.4 121.92) (xy 27.94 121.92)
 		)
@@
 	)
 	(symbol
+		(lib_id "Device:C_Small")
+		(at 256.54 45.72 90)
+		(unit 1)
+		(body_style 1)
+		(exclude_from_sim no)
+		(in_bom yes)
+		(on_board yes)
+		(in_pos_files yes)
+		(dnp no)
+		(property "Reference" "C79"
+			(at 254.762 44.45 90)
+			(show_name no)
+			(do_not_autoplace no)
+			(effects
+				(font
+					(size 1.27 1.27)
+				)
+				(justify left)
+			)
+		)
+		(property "Value" "10u"
+			(at 261.366 44.45 90)
+			(show_name no)
+			(do_not_autoplace no)
+			(effects
+				(font
+					(size 1.27 1.27)
+				)
+				(justify left)
+			)
+		)
+		(property "Footprint" "Capacitor_SMD:C_0805_2012Metric"
+			(at 260.35 44.7548 0)
+			(hide yes)
+			(show_name no)
+			(do_not_autoplace no)
+			(effects
+				(font
+					(size 1.27 1.27)
+				)
+			)
+		)
+		(property "Datasheet" ""
+			(at 256.54 45.72 0)
+			(hide yes)
+			(show_name no)
+			(do_not_autoplace no)
+			(effects
+				(font
+					(size 1.27 1.27)
+				)
+			)
+		)
+		(property "Description" ""
+			(at 256.54 45.72 0)
+			(hide yes)
+			(show_name no)
+			(do_not_autoplace no)
+			(effects
+				(font
+					(size 1.27 1.27)
+				)
+			)
+		)
+		(property "Supplier" "Samsung CL21A106KAYNNNE"
+			(at 256.54 45.72 0)
+			(hide yes)
+			(show_name no)
+			(do_not_autoplace no)
+			(effects
+				(font
+					(size 1.27 1.27)
+				)
+			)
+		)
+		(property "Notes" ""
+			(at 256.54 45.72 0)
+			(hide yes)
+			(show_name no)
+			(do_not_autoplace no)
+			(effects
+				(font
+					(size 1.27 1.27)
+				)
+			)
+		)
+		(property "JLCPCB part" "C15850"
+			(at 256.54 45.72 0)
+			(hide yes)
+			(show_name no)
+			(do_not_autoplace no)
+			(effects
+				(font
+					(size 1.27 1.27)
+				)
+			)
+		)
+		(pin "1"
+		)
+		(pin "2"
+		)
+		(instances
+			(project "pedalboard-hw"
+				(path "/df521c2a-9827-4355-b809-366f4b88d5d7/6bd0afd4-cd8b-4c1d-a236-891eed0b2d91"
+					(reference "C79")
+					(unit 1)
+				)
+			)
+		)
+	)
+	(symbol
 		(lib_id "Device:R_Small")
 		(at 93.98 187.96 90)
@@
 		(dnp no)
 		(property "Reference" "C65"
-			(at 258.318 45.212 90)
+			(at 255.524 48.006 90)
 			(show_name no)
 			(do_not_autoplace no)
@@
 		)
 		(property "Value" "100n"
-			(at 259.334 46.99 90)
+			(at 262.636 48.006 90)
 			(show_name no)
 			(do_not_autoplace no)

Commit message: updated cap
Parts:
- C73, C74: value 220uF -> 680uF; footprint Capacitor_THT:CP_Radial_D6.3mm_P2.50mm -> Capacitor_THT:CP_Radial_D8.0mm_P3.50mm; Manufacturer (none) -> Panasonic; Manufacturer part EEU-FM1A221 -> EEU-FR1A681
Changed lines of the file:
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@@
 	)
 	(symbol
+		(lib_id "Device:C_Polarized_Small_US")
+		(at 240.03 116.84 90)
+		(unit 1)
+		(body_style 1)
+		(exclude_from_sim no)
+		(in_bom yes)
+		(on_board yes)
+		(in_pos_files yes)
+		(dnp no)
+		(property "Reference" "C74"
+			(at 240.284 120.396 90)
+			(show_name no)
+			(do_not_autoplace no)
+			(effects
+				(font
+					(size 1.27 1.27)
+				)
+			)
+		)
+		(property "Value" "680uF"
+			(at 240.284 122.682 90)
+			(show_name no)
+			(do_not_autoplace no)
+			(effects
+				(font
+					(size 1.27 1.27)
+				)
+			)
+		)
+		(property "Footprint" "Capacitor_THT:CP_Radial_D8.0mm_P3.50mm"
+			(at 240.03 116.84 0)
+			(hide yes)
+			(show_name no)
+			(do_not_autoplace no)
+			(effects
+				(font
+					(size 1.27 1.27)
+				)
+			)
+		)
+		(property "Datasheet" ""
+			(at 240.03 116.84 0)
+			(hide yes)
+			(show_name no)
+			(do_not_autoplace no)
+			(effects
+				(font
+					(size 1.27 1.27)
+				)
+			)
+		)
+		(property "Description" ""
+			(at 240.03 116.84 0)
+			(hide yes)
+			(show_name no)
+			(do_not_autoplace no)
+			(effects
+				(font
+					(size 1.27 1.27)
+				)
+			)
+		)
+		(property "Manufacturer part" "EEU-FR1A681"
+			(at 240.03 116.84 0)
+			(hide yes)
+			(show_name no)
+			(do_not_autoplace no)
+			(effects
+				(font
+					(size 1.27 1.27)
+				)
+			)
+		)
+		(property "Manufacturer" "Panasonic"
+			(at 240.03 116.84 90)
+			(hide yes)
+			(show_name no)
+			(do_not_autoplace no)
+			(effects
+				(font
+					(size 1.27 1.27)
+				)
+			)
+		)
+		(pin "2"
+		)
+		(pin "1"
+		)
+		(instances
+			(project "pedalboard-hw"
+				(path "/df521c2a-9827-4355-b809-366f4b88d5d7/6bd0afd4-cd8b-4c1d-a236-891eed0b2d91"
+					(reference "C74")
+					(unit 1)
+				)
+			)
+		)
+	)
+	(symbol
 		(lib_id "power:GND")
 		(at 161.29 74.93 0)
@@
 	)
 	(symbol
-		(lib_id "Device:C_Polarized_Small_US")
-		(at 240.03 116.84 90)
-		(unit 1)
-		(body_style 1)
-		(exclude_from_sim no)
-		(in_bom yes)
-		(on_board yes)
-		(in_pos_files yes)
-		(dnp no)
-		(property "Reference" "C74"
-			(at 240.538 120.142 90)
-			(show_name no)
-			(do_not_autoplace no)
-			(effects
-				(font
-					(size 1.27 1.27)
-				)
-			)
-		)
-		(property "Value" "220uF"
-			(at 240.538 122.682 90)
-			(show_name no)
-			(do_not_autoplace no)
-			(effects
-				(font
-					(size 1.27 1.27)
-				)
-			)
-		)
-		(property "Footprint" "Capacitor_THT:CP_Radial_D6.3mm_P2.50mm"
-			(at 240.03 116.84 0)
-			(hide yes)
-			(show_name no)
-			(do_not_autoplace no)
-			(effects
-				(font
-					(size 1.27 1.27)
-				)
-			)
-		)
-		(property "Datasheet" ""
-			(at 240.03 116.84 0)
-			(hide yes)
-			(show_name no)
-			(do_not_autoplace no)
-			(effects
-				(font
-					(size 1.27 1.27)
-				)
-			)
-		)
-		(property "Description" "Panasonic FM 220uF, 10V"
-			(at 240.03 116.84 0)
-			(hide yes)
-			(show_name no)
-			(do_not_autoplace no)
-			(effects
-				(font
-					(size 1.27 1.27)
-				)
-			)
-		)
-		(property "Manufacturer part" "EEU-FM1A221"
-			(at 240.03 116.84 0)
-			(hide yes)
-			(show_name no)
-			(do_not_autoplace no)
-			(effects
-				(font
-					(size 1.27 1.27)
-				)
-			)
-		)
-		(pin "2"
-		)
-		(pin "1"
-		)
-		(instances
-			(project "pedalboard-hw"
-				(path "/df521c2a-9827-4355-b809-366f4b88d5d7/6bd0afd4-cd8b-4c1d-a236-891eed0b2d91"
-					(reference "C74")
-					(unit 1)
-				)
-			)
-		)
-	)
-	(symbol
 		(lib_id "Device:R_Small")
 		(at 114.3 185.42 270)
@@
 			)
 		)
-		(property "Value" "220uF"
+		(property "Value" "680uF"
 			(at 239.5982 107.95 90)
 			(show_name no)
@@
 			)
 		)
-		(property "Footprint" "Capacitor_THT:CP_Radial_D6.3mm_P2.50mm"
+		(property "Footprint" "Capacitor_THT:CP_Radial_D8.0mm_P3.50mm"
 			(at 240.03 111.76 0)
 			(hide yes)
@@
 			)
 		)
-		(property "Description" "Panasonic FM 220uF, 10V"
+		(property "Description" ""
 			(at 240.03 111.76 0)
 			(hide yes)
@@
 			)
 		)
-		(property "Manufacturer part" "EEU-FM1A221"
+		(property "Manufacturer part" "EEU-FR1A681"
 			(at 240.03 111.76 0)
 			(hide yes)
 			(show_name no)
+			(do_not_autoplace no)
+			(effects
+				(font
+					(size 1.27 1.27)
+				)
+			)
+		)
+		(property "Manufacturer" "Panasonic"
+			(at 240.03 111.76 90)
+			(hide yes)
+			(show_name no)
