File: audio.kicad_sch (KiCad schematic)
At the start: 57 parts, among them IC1 TAC5212IRGER, J13 Headphones 3.5mm, J18 Jack 6.35mm, J19 Jack 6.35mm, J20 Jack 6.35mm, J22 Jack 6.35mm, U14 OPA1656ID

Commit message: changd diode.
Parts:
- D3: value H5VUD5BB -> ESD451; footprint Diode_SMD:D_SOD-523 -> Package_SON:Texas_DPY0002A_0.6x1mm_P0.65mm; Manufacturer (none) -> Texas Instruments; Manufacturer part (none) -> ESD451DPYR
Changed lines of the file:
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@@
 			)
 		)
-		(property "Value" "H5VUD5BB"
+		(property "Value" "ESD451"
 			(at 83.312 167.386 90)
 			(show_name no)
@@
 			)
 		)
-		(property "Footprint" "Diode_SMD:D_SOD-523"
+		(property "Footprint" "Package_SON:Texas_DPY0002A_0.6x1mm_P0.65mm"
 			(at 81.28 166.37 0)
 			(hide yes)
@@
 			(hide yes)
 			(show_name no)
+			(do_not_autoplace no)
+			(effects
+				(font
+					(size 1.27 1.27)
+				)
+			)
+		)
+		(property "Manufacturer" "Texas Instruments"
+			(at 81.28 166.37 90)
+			(hide yes)
+			(show_name no)
+			(do_not_autoplace no)
+			(effects
+				(font
+					(size 1.27 1.27)
+				)
+			)
+		)
+		(property "Manufacturer part" "ESD451DPYR"
+			(at 81.28 166.37 90)
+			(hide yes)
+			(show_name no)

Commit message: some stuff
Parts:
- IC1: footprint SamacSys_Parts:TAC5212IRGER -> Pedalboard Library:TAC5212IRGER
Changed lines of the file:
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@@
 			)
 		)
-		(property "Footprint" "SamacSys_Parts:TAC5212IRGER"
+		(property "Footprint" "Pedalboard Library:TAC5212IRGER"
 			(at 220.98 145.72 0)
 			(hide yes)

Commit message: a few edits
Connections:
- no-connect marks 17 -> 76
Changed lines of the file:
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@@
+	)
+	(no_connect
+		(at 105.41 68.58)
 	)
 	(no_connect
@@
 	)
 	(no_connect
+		(at 105.41 142.24)
+	)
+	(no_connect
+		(at 105.41 96.52)
+	)
+	(no_connect
+		(at 44.45 76.2)
+	)
+	(no_connect
+		(at 105.41 139.7)
+	)
+	(no_connect
+		(at 105.41 73.66)
+	)
+	(no_connect
 		(at 270.51 139.7)
 	)
 	(no_connect
+		(at 44.45 45.72)
+	)
+	(no_connect
+		(at 44.45 22.86)
+	)
+	(no_connect
+		(at 44.45 83.82)
+	)
+	(no_connect
 		(at 250.19 78.74)
 	)
 	(no_connect
+		(at 44.45 104.14)
+	)
+	(no_connect
 		(at 270.51 144.78)
 	)
 	(no_connect
+		(at 44.45 116.84)
+	)
+	(no_connect
+		(at 44.45 73.66)
+	)
+	(no_connect
 		(at 250.19 71.12)
 	)
 	(no_connect
+		(at 105.41 53.34)
+	)
+	(no_connect
+		(at 44.45 58.42)
+	)
+	(no_connect
+		(at 44.45 50.8)
+	)
+	(no_connect
+		(at 44.45 111.76)
+	)
+	(no_connect
 		(at 213.36 149.86)
 	)
@@
 	)
 	(no_connect
+		(at 105.41 60.96)
+	)
+	(no_connect
+		(at 44.45 66.04)
+	)
+	(no_connect
+		(at 105.41 93.98)
+	)
+	(no_connect
+		(at 105.41 20.32)
+	)
+	(no_connect
+		(at 105.41 38.1)
+	)
+	(no_connect
 		(at 270.51 147.32)
 	)
 	(no_connect
+		(at 44.45 35.56)
+	)
+	(no_connect
+		(at 44.45 71.12)
+	)
+	(no_connect
+		(at 44.45 40.64)
+	)
+	(no_connect
+		(at 105.41 22.86)
+	)
+	(no_connect
+		(at 44.45 106.68)
+	)
+	(no_connect
+		(at 44.45 101.6)
+	)
+	(no_connect
 		(at 270.51 109.22)
 	)
 	(no_connect
+		(at 44.45 20.32)
+	)
+	(no_connect
+		(at 105.41 27.94)
+	)
+	(no_connect
+		(at 105.41 88.9)
+	)
+	(no_connect
+		(at 105.41 101.6)
+	)
+	(no_connect
 		(at 250.19 73.66)
 	)
 	(no_connect
+		(at 44.45 142.24)
+	)
+	(no_connect
+		(at 44.45 78.74)
+	)
+	(no_connect
 		(at 74.93 168.91)
 	)
 	(no_connect
+		(at 44.45 129.54)
+	)
+	(no_connect
+		(at 44.45 127)
+	)
+	(no_connect
+		(at 44.45 96.52)
+	)
+	(no_connect
+		(at 105.41 35.56)
+	)
+	(no_connect
+		(at 44.45 30.48)
+	)
+	(no_connect
+		(at 105.41 63.5)
+	)
+	(no_connect
+		(at 44.45 119.38)
+	)
+	(no_connect
+		(at 44.45 134.62)
+	)
+	(no_connect
+		(at 44.45 137.16)
+	)
+	(no_connect
+		(at 44.45 38.1)
+	)
+	(no_connect
+		(at 44.45 60.96)
+	)
+	(no_connect
+		(at 105.41 66.04)
+	)
+	(no_connect
+		(at 44.45 132.08)
+	)
+	(no_connect
+		(at 105.41 109.22)
+	)
+	(no_connect
+		(at 44.45 93.98)
+	)
+	(no_connect
 		(at 73.66 187.96)
 	)
 	(no_connect
+		(at 105.41 104.14)
+	)
+	(no_connect
+		(at 44.45 63.5)
+	)
+	(no_connect
+		(at 105.41 111.76)
+	)
+	(no_connect
+		(at 105.41 129.54)
+	)
+	(no_connect
 		(at 213.36 144.78)
 	)
 	(no_connect
+		(at 105.41 76.2)
+	)
+	(no_connect
+		(at 105.41 132.08)
+	)
+	(no_connect
 		(at 250.19 76.2)
 	)
 	(no_connect
+		(at 44.45 27.94)
+	)
+	(no_connect
+		(at 105.41 55.88)
+	)
+	(no_connect
 		(at 250.19 83.82)
 	)
 	(no_connect
+		(at 105.41 30.48)
+	)
+	(no_connect
+		(at 44.45 53.34)
+	)
+	(no_connect
 		(at 270.51 114.3)
 	)
+	(no_connect
+		(at 105.41 40.64)
+	)
 	(wire

Commit message: Standardize values.
Parts:
- C61, C65, C66, C70: value 100n -> 100nF
- C67, C68, C79: value 10u -> 10uF
- C69: value 1u -> 1uF
- R16, R34, R37, R40: value 1K -> 1k
- R43, R44: value 7.5k -> 7k5
- R51, R52: value 4.7k -> 4k7
Changed lines of the file:
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@@
 			)
 		)
-		(property "Value" "1u"
+		(property "Value" "1uF"
 			(at 210.312 75.438 0)
 			(show_name no)
@@
 			)
 		)
-		(property "Value" "1K"
+		(property "Value" "1k"
 			(at 141.986 167.386 0)
 			(show_name no)
@@
 			)
 		)
-		(property "Value" "100n"
+		(property "Value" "100nF"
 			(at 152.146 66.294 0)
 			(show_name no)
@@
 			)
 		)
-		(property "Value" "100n"
+		(property "Value" "100nF"
 			(at 201.93 74.168 0)
 			(show_name no)
@@
 			)
 		)
-		(property "Value" "7.5k"
+		(property "Value" "7k5"
 			(at 109.22 178.562 90)
 			(show_name no)
@@
 			)
 		)
-		(property "Value" "10u"
+		(property "Value" "10uF"
 			(at 265.176 67.564 0)
 			(show_name no)
@@
 			)
 		)
-		(property "Value" "100n"
+		(property "Value" "100nF"
 			(at 276.606 68.072 0)
 			(show_name no)
@@
 			)
 		)
-		(property "Value" "10u"
+		(property "Value" "10uF"
 			(at 196.596 74.168 0)
 			(show_name no)
@@
 			)
 		)
-		(property "Value" "10u"
+		(property "Value" "10uF"
 			(at 261.366 44.45 90)
 			(show_name no)
@@
 			)
 		)
-		(property "Value" "1K"
+		(property "Value" "1k"
 			(at 127.254 171.45 90)
 			(show_name no)
@@
 			)
 		)
-		(property "Value" "1K"
+		(property "Value" "1k"
 			(at 260.35 22.86 90)
 			(show_name no)
@@
 			)
 		)
-		(property "Value" "7.5k"
+		(property "Value" "7k5"
 			(at 114.3 183.642 90)
 			(show_name no)
@@
 			)
 		)
-		(property "Value" "4.7k"
+		(property "Value" "4k7"
 			(at 22.352 96.266 0)
 			(show_name no)
@@
 			)
 		)
-		(property "Value" "4.7k"
+		(property "Value" "4k7"
 			(at 31.496 96.266 0)
 			(show_name no)
@@
 			)
 		)
-		(property "Value" "100n"
+		(property "Value" "100nF"
 			(at 262.636 48.006 90)
 			(show_name no)
@@
 			)
 		)
-		(property "Value" "1K"
+		(property "Value" "1k"
 			(at 115.824 167.64 90)
 			(show_name no)

Commit message: edited metadata
Parts:
- IC1: Height 1 -> (none); JLCPCB part (none) -> C44853694; Manufacturer (none) -> Texas Instruments; Manufacturer part (none) -> TAC5212IRGER; Manufacturer_Name Texas Instruments -> (none); Manufacturer_Part_Number TAC5212IRGER -> (none); Notes (none) -> ADC1/2: differential AC-coupled, 5k/pin, 2Vrms differential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
- U14: JLCPCB part (none) -> C1346368; Manufacturer (none) -> Texas Instruments; Manufacturer part (none) -> OPA1656ID
Other:
- moved on the sheet: C61, CM2A, H4, H5, H6, H7, R51, R52, U14C

Commit message: more meta
Parts:
- C61: Digikey 1276-1180-1-ND -> (none); JLCPCB part (none) -> C49678; Manufacturer (none) -> Yageo; Manufacturer part (none) -> CC0805KRX7R9BB104; Notes 10% 16V Ceramic Capacitor X7R -> (none); Supplier https://www.digikey.ch/de/products/detail/samsung-electro-m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 -> (none)
- R16: JLCPCB part (none) -> C17513; Manufacturer part (none) -> 0805W8F1001T5E; Supplier https://www.digikey.ch/de/products/detail/stackpole-electro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 -> (none)
- R33: JLCPCB part (none) -> C22935; Manufacturer part (none) -> 0603WAF1004T5E; Notes C22935 -> (none)
Changed lines of the file:
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@@
 		)
 		(property "Value" "1uF"
-			(at 210.312 75.438 0)
+			(at 209.296 75.692 0)
 			(show_name no)
 			(do_not_autoplace no)
@@
 	)
 	(symbol
-		(lib_id "Device:C_Small")
-		(at 25.4 176.53 0)
-		(unit 1)
-		(body_style 1)
-		(exclude_from_sim no)
-		(in_bom yes)
-		(on_board yes)
-		(in_pos_files yes)
-		(dnp no)
-		(property "Reference" "C61"
-			(at 21.082 174.752 0)
-			(show_name no)
-			(do_not_autoplace no)
-			(effects
-				(font
-					(size 1.27 1.27)
-				)
-				(justify left)
-			)
-		)
-		(property "Value" "100nF"
-			(at 20.066 178.054 0)
-			(show_name no)
-			(do_not_autoplace no)
-			(effects
-				(font
-					(size 1.27 1.27)
-				)
-				(justify left)
-			)
-		)
-		(property "Footprint" "Capacitor_SMD:C_0805_2012Metric"
-			(at 26.3652 180.34 0)
-			(hide yes)
-			(show_name no)
-			(do_not_autoplace no)
-			(effects
-				(font
-					(size 1.27 1.27)
-				)
-			)
-		)
-		(property "Datasheet" "https://www.samsungsem.com/resources/file/global/support/product_catalog/MLCC.pdf"
-			(at 25.4 176.53 0)
-			(hide yes)
-			(show_name no)
-			(do_not_autoplace no)
-			(effects
-				(font
-					(size 1.27 1.27)
-				)
-			)
-		)
-		(property "Description" ""
-			(at 25.4 176.53 0)
-			(hide yes)
-			(show_name no)
-			(do_not_autoplace no)
-			(effects
-				(font
-					(size 1.27 1.27)
-				)
-			)
-		)
-		(property "Supplier" "https://www.digikey.ch/de/products/detail/samsung-electro-mechanics/CL21B104KBCNNNC/3886661"
-			(at 25.4 176.53 0)
-			(hide yes)
-			(show_name no)
-			(do_not_autoplace no)
-			(effects
-				(font
-					(size 1.27 1.27)
-				)
-			)
-		)
-		(property "Notes" "10% 16V Ceramic Capacitor X7R"
-			(at 25.4 176.53 0)
-			(hide yes)
-			(show_name no)
-			(do_not_autoplace no)
-			(effects
-				(font
-					(size 1.27 1.27)
-				)
-			)
-		)
-		(property "Digikey" "1276-1180-1-ND"
-			(at 25.4 176.53 0)
-			(hide yes)
-			(show_name no)
-			(do_not_autoplace no)
-			(effects
-				(font
-					(size 1.27 1.27)
-				)
-			)
-		)
-		(pin "1"
-		)
-		(pin "2"
-		)
-		(instances
-			(project "pedalboard-hw"
-				(path "/df521c2a-9827-4355-b809-366f4b88d5d7/6bd0afd4-cd8b-4c1d-a236-891eed0b2d91"
-					(reference "C61")
-					(unit 1)
-				)
-			)
-		)
-	)
-	(symbol
 		(lib_id "Device:C_Polarized_Small_US")
 		(at 240.03 116.84 90)
@@
 		)
 		(property "Value" "100nF"
-			(at 201.93 74.168 0)
+			(at 200.914 74.422 0)
 			(show_name no)
 			(do_not_autoplace no)
@@
 		)
 		(property "Value" "100nF"
-			(at 276.606 68.072 0)
+			(at 275.59 68.326 0)
 			(show_name no)
 			(do_not_autoplace no)
@@
 		)
 		(property "Value" "10uF"
-			(at 196.596 74.168 0)
+			(at 195.326 74.422 0)
 			(show_name no)
 			(do_not_autoplace no)
@@
 		(in_pos_files yes)
 		(dnp no)
-		(fields_autoplaced yes)
 		(property "Reference" "D6"
 			(at 251.1425 20.32 0)
@@
 		)
 		(property "Sim.Pins" "1=K 2=A"
-			(at 252.73 26.67 0)
+			(at 252.222 30.226 0)
+			(hide yes)
 			(show_name no)
 			(do_not_autoplace no)
@@
 		)
 		(property "Value" "10uF"
-			(at 261.366 44.45 90)
+			(at 263.144 44.45 90)
 			(show_name no)
 			(do_not_autoplace no)
@@
 		(in_pos_files yes)
 		(dnp no)
-		(fields_autoplaced yes)
 		(property "Reference" "R16"
-			(at 260.35 20.32 90)
+			(at 260.35 22.606 90)
 			(show_name no)
 			(do_not_autoplace no)
@@
 		)
 		(property "Value" "1k"
-			(at 260.35 22.86 90)
+			(at 260.35 24.638 90)
 			(show_name no)
 			(do_not_autoplace no)
@@
 			)
 		)
-		(property "Supplier" "https://www.digikey.ch/de/products/detail/stackpole-electronics-inc/RNCP0805FTD1K00/2240229"
+		(property "Manufacturer" ""
 			(at 260.35 26.67 0)
 			(hide yes)
@@
 			)
 		)
+		(property "Manufacturer part" "0805W8F1001T5E"
+			(at 260.35 26.67 90)
+			(hide yes)
+			(show_name no)
+			(do_not_autoplace no)
+			(effects
+				(font
+					(size 1.27 1.27)
+				)
+			)
+		)
+		(property "JLCPCB part" "C17513"
+			(at 260.35 26.67 90)
+			(hide yes)
+			(show_name no)
+			(do_not_autoplace no)
+			(effects
+				(font
+					(size 1.27 1.27)
+				)
+			)
+		)
 		(pin "1"
 		)
@@
 			)
 		)
-		(property "Supplier" ""
+		(property "Manufacturer" ""
 			(at 93.98 157.48 0)
 			(hide yes)
@@
 			)
 		)
-		(property "Notes" "C22935"
+		(property "JLCPCB part" "C22935"
 			(at 93.98 157.48 90)
 			(hide yes)
@@
 			)
 		)
+		(property "Manufacturer part" "0603WAF1004T5E"
+			(at 93.98 157.48 0)
+			(hide yes)
+			(show_name no)
+			(do_not_autoplace no)
+			(effects
+				(font
+					(size 1.27 1.27)
+				)
+			)
+		)
 		(pin "1"
 		)
@@
 	)
 	(symbol
+		(lib_id "Device:C_Small")
+		(at 25.4 176.53 0)
+		(unit 1)
+		(body_style 1)
+		(exclude_from_sim no)
+		(in_bom yes)
+		(on_board yes)
+		(in_pos_files yes)
+		(dnp no)
+		(property "Reference" "C61"
+			(at 19.558 175.006 0)
+			(show_name no)
+			(do_not_autoplace no)
+			(effects
+				(font
+					(size 1.27 1.27)
+				)
+				(justify left)
+			)
+		)
+		(property "Value" "100nF"
+			(at 19.05 178.308 0)
+			(show_name no)
+			(do_not_autoplace no)
+			(effects
+				(font
+					(size 1.27 1.27)
+				)
+				(justify left)
+			)
+		)
+		(property "Footprint" "Capacitor_SMD:C_0805_2012Metric"
+			(at 26.3652 180.34 0)
+			(hide yes)
+			(show_name no)
+			(do_not_autoplace no)
+			(effects
+				(font
+					(size 1.27 1.27)
+				)
+			)
+		)
+		(property "Datasheet" ""
+			(at 25.4 176.53 0)
+			(hide yes)
+			(show_name no)
+			(do_not_autoplace no)
+			(effects
+				(font
+					(size 1.27 1.27)
+				)
+			)
+		)
+		(property "Description" ""
+			(at 25.4 176.53 0)
+			(hide yes)
+			(show_name no)
+			(do_not_autoplace no)
+			(effects
+				(font
+					(size 1.27 1.27)
+				)
+			)
+		)
+		(property "Manufacturer" "Yageo"
+			(at 25.4 176.53 0)
+			(hide yes)
+			(show_name no)
+			(do_not_autoplace no)
+			(effects
+				(font
+					(size 1.27 1.27)
+				)
+			)
+		)
+		(property "Manufacturer part" "CC0805KRX7R9BB104"
+			(at 25.4 176.53 0)
+			(hide yes)
+			(show_name no)
+			(do_not_autoplace no)
+			(effects
+				(font
+					(size 1.27 1.27)
+				)
+			)
+		)
+		(property "JLCPCB part" "C49678"
+			(at 25.4 176.53 0)
+			(hide yes)
+			(show_name no)
+			(do_not_autoplace no)
+			(effects
+				(font
+					(size 1.27 1.27)
+				)
+			)
+		)
+		(pin "1"
+		)
+		(pin "2"
+		)
+		(instances
+			(project "pedalboard-hw"
+				(path "/df521c2a-9827-4355-b809-366f4b88d5d7/6bd0afd4-cd8b-4c1d-a236-891eed0b2d91"
+					(reference "C61")
+					(unit 1)
+				)
+			)
+		)
+	)
+	(symbol
 		(lib_id "power:+3V3")
 		(at 270.51 63.5 0)
@@
 		)
 		(property "Value" "100nF"
-			(at 262.636 48.006 90)
+			(at 263.906 48.006 90)
 			(show_name no)
 			(do_not_autoplace no)

Commit message: Updated various metadata
Parts:
- removed J19, J20: Jack 6.35mm, Pedalboard Library:Jack_6.35mm_Horizontal, symbol Connector_Audio:NMJ6HCD2
- added C81: 47uF, Capacitor_SMD:CP_Elec_6.3x5.8, symbol Device:C_Polarized_Small_US
- added J19: LINE OUT LEFT, Connector_Audio:Jack_6.35mm_Neutrik_NMJ4HCD2_Horizontal, symbol Connector_Audio:NMJ4HCD2
- added J20: LINE OUT RIGHT, Connector_Audio:Jack_6.35mm_Neutrik_NMJ4HCD2_Horizontal, symbol Connector_Audio:NMJ4HCD2
- added R54, R56: 820R, Resistor_SMD:R_0603_1608Metric, symbol Device:R_Small
- added R55: 390R, Resistor_SMD:R_0603_1608Metric, symbol Device:R_Small
- added R57: 1k, Resistor_SMD:R_0603_1608Metric, symbol Device:R_Small
- added SW11: EM-02-Q, Button_Switch_SMD:SW_DIP_SPSTx02_Slide_6.7x6.64mm_W8.61mm_P2.54mm_LowProfile, symbol Switch:SW_DIP_x02
- C57, C58, C62, C63: JLCPCB part (none) -> C50394238; Manufacturer (none) -> Rubycon; Manufacturer part (none) -> 16MF475KB23225; Notes Rubycon 16MF475KB23225 -> 4.7uF, 16V, non-polar polymer. Extended part.
- C65, C66, C70: Manufacturer (none) -> Yageo; Manufacturer part (none) -> CC0603KRX7R9BB104; Supplier Yageo CC0603KRX7R9BB104 -> (none)
- C67, C68, C79: Manufacturer (none) -> Samsung Electro-Mechanics; Manufacturer part (none) -> CL21A106KAYNNNE; Supplier Samsung CL21A106KAYNNNE -> (none)
- C69: Manufacturer (none) -> Samsung Electro-Mechanics; Manufacturer part (none) -> CL21B105KBFNNNE; Supplier Samsung CL21B105KBFNNNE -> (none)
- C73, C74: Notes (none) -> 680uF, 10V, low-ESR aluminum electrolytic. Hand-fitted. Pos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
- C75, C77: Manufacturer FH / Fenghua -> FH; Manufacturer part (none) -> 1206B475K500NT
- CM2: value ComputeModule5-CM5 -> Raspberry Pi CM5; Field4 Amphenol -> (none); Field5 2x 10164227-1001A1RLF -> (none); Manufacturer (none) -> Raspberry Pi ltd; Notes (none) -> CM5 module supplied separately. Carrier requires 2x Ampheno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
- D4, D5, D8, D9: JLCPCB part (none) -> C20615820; Manufacturer (none) -> Hongjiacheng; Manufacturer part (none) -> H5VUD5BB; now fitted
- D6: JLCPCB part (none) -> C2296; Manufacturer (none) -> Hubei KENTO Elec; Manufacturer part (none) -> KT-0805Y; Supplier https://www.digikey.ch/en/products/detail/harvatek-corporat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 -> (none)
- J13: Manufacturer (none) -> Same Sky; Manufacturer part (none) -> SJ1-3525N
- J18: value Jack 6.35mm -> GUITAR INPUT; footprint Pedalboard Library:Jack_6.35mm_Horizontal -> Connector_Audio:Jack_6.35mm_Neutrik_NMJ4HCD2_Horizontal; symbol Connector_Audio:NMJ6HCD2 -> Connector_Audio:NMJ4HCD2; Manufacturer (none) -> Neutrik; Manufacturer part (none) -> NMJ4HCD2; Notes Audio IN Right -> 6.35 mm TS guitar input. Tip-normal contact grounds the inp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; Supplier https://www.digikey.ch/de/products/detail/schurter-inc/4833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 -> (none)
- J22: value Jack 6.35mm -> BALANCED LINE INPUT; footprint Pedalboard Library:Jack_6.35mm_Horizontal -> Connector_Audio:Jack_6.35mm_Neutrik_NMJ6HCD2_Horizontal; Manufacturer (none) -> Neutrik; Manufacturer part (none) -> NMJ6HCD2; Notes Audio IN Left -> 6.35 mm TRS balanced line input. Through-hole, manual fit.; Supplier https://www.digikey.ch/de/products/detail/schurter-inc/4833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 -> (none)
- R16, R33: Manufacturer (none) -> UNI-ROYAL
- R34, R37, R40: Manufacturer (none) -> UNI-ROYAL; Manufacturer part (none) -> 0603WAF1001T5E; Supplier UNI-ROYAL 0603WAF1001T5E -> (none)
- R38, R39: Manufacturer (none) -> UNI-ROYAL; Manufacturer part (none) -> 0603WAF4700T5E; Supplier UNI-ROYAL 0603WAF4700T5E -> (none)
- R41, R42: Manufacturer (none) -> UNI-ROYAL; Manufacturer part (none) -> 0603WAF1003T5E; Notes UNI-ROYAL 0603WAF1003T5E -> (none)
- R43, R44: Manufacturer (none) -> UNI-ROYAL; Manufacturer part (none) -> 0603WAF7501T5E; Notes UNI-ROYAL 0603WAF7501T5E -> (none)
- R45, R46: Manufacturer (none) -> UNI-ROYAL; Supplier UNI-ROYAL -> (none)
Connections:
- net GND: now also C81.2, J19.S, J20.S; no longer J18.RN
- net at C76.1, D9.2 (A2), R47.1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: now also J19.T
- net at R34.2, R39.2, U14.1: now also R55.1; no longer U14.2 (-)
- net at C78.1, D8.2 (A2), R49.1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: now also J20.T
- new net: R56.2, R57.1, SW11.3, U14.2 (-)
- new net: R54.1, R55.2, SW11.4
- new net: R54.2, R56.1, SW11.1, SW11.2
- new net: C81.1, R57.2
- no-connect marks 76 -> 73
Other:
- note added: "Input gain: 1+2 ON: LOW 1.39x 1 ON, 2 OFF (or reverse): MID 2.21x 1+2 OFF: HIGH 3.03x"
- moved on the sheet: C56, C57, C64, C65, C66, C67, C68, C69, C70, C73, C75, C76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
