File: audio.kicad_sch (KiCad schematic)
At the start: 63 parts, among them IC1 TAC5212IRGER, J13 Headphones 3.5mm, J18 GUITAR INPUT, J19 LINE OUT LEFT, J20 LINE OUT RIGHT, J22 BALANCED LINE INPUT, SW11 EM-02-Q, U14 OPA1656ID

Commit message: Moving to seperate ui board using ESP32
Connections:
- net UI_UART_RX: now reaches CM2.34 (GPIO5)
- net ESP_RESET: now reaches CM2.46 (GPIO22)
- net ESP_BOOT: now reaches CM2.47 (GPIO23)
- net UI_UART_TX: now reaches CM2.54 (GPIO4)
- net CM5_UART_RX renamed CM5_DEBUG_UART_RX
- net CM5_UART_TX renamed CM5_DEBUG_UART_TX
- no-connect marks 73 -> 69
Changed lines of the file:
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@@
 	)
 	(no_connect
-		(at 57.15 83.82)
-	)
-	(no_connect
 		(at 124.46 184.15)
 	)
@@
 	)
 	(no_connect
-		(at 57.15 73.66)
-	)
-	(no_connect
 		(at 208.28 143.51)
 	)
@@
 	)
 	(no_connect
-		(at 57.15 58.42)
-	)
-	(no_connect
 		(at 57.15 50.8)
 	)
@@
 	)
 	(no_connect
-		(at 118.11 76.2)
-	)
-	(no_connect
 		(at 118.11 132.08)
 	)
@@
 	(wire
 		(pts
+			(xy 50.8 58.42) (xy 57.15 58.42)
+		)
+		(stroke
+			(width 0)
+			(type default)
+		)
+	)
+	(wire
+		(pts
 			(xy 232.41 114.3) (xy 232.41 124.46)
 		)
@@
 	(wire
 		(pts
+			(xy 124.46 73.66) (xy 124.46 76.2)
+		)
+		(stroke
+			(width 0)
+			(type default)
+		)
+	)
+	(wire
+		(pts
 			(xy 118.11 78.74) (xy 138.43 78.74)
 		)
@@
 	(wire
 		(pts
+			(xy 124.46 76.2) (xy 118.11 76.2)
+		)
+		(stroke
+			(width 0)
+			(type default)
+		)
+	)
+	(wire
+		(pts
 			(xy 91.44 186.69) (xy 91.44 189.23)
 		)
@@
 	(wire
 		(pts
+			(xy 127 73.66) (xy 124.46 73.66)
+		)
+		(stroke
+			(width 0)
+			(type default)
+		)
+	)
+	(wire
+		(pts
 			(xy 207.01 146.05) (xy 207.01 153.67)
 		)
@@
 	(wire
 		(pts
+			(xy 50.8 83.82) (xy 57.15 83.82)
+		)
+		(stroke
+			(width 0)
+			(type default)
+		)
+	)
+	(wire
+		(pts
 			(xy 181.61 64.77) (xy 181.61 66.04)
 		)
@@
 	(wire
 		(pts
+			(xy 50.8 73.66) (xy 57.15 73.66)
+		)
+		(stroke
+			(width 0)
+			(type default)
+		)
+	)
+	(wire
+		(pts
 			(xy 87.63 189.23) (xy 90.17 189.23)
 		)
@@
 		)
 	)
-	(global_label "CM5_UART_TX"
+	(global_label "CM5_DEBUG_UART_TX"
 		(shape input)
 		(at 125.73 86.36 0)
@@
 		)
 		(property "Intersheetrefs" "${INTERSHEET_REFS}"
-			(at 141.4151 86.36 0)
+			(at 148.6722 86.36 0)
 			(hide yes)
 			(show_name no)
@@
 		)
 	)
+	(global_label "UI_UART_TX"
+		(shape input)
+		(at 50.8 83.82 180)
+		(fields_autoplaced yes)
+		(effects
+			(font
+				(size 1.27 1.27)
+			)
+			(justify right)
+		)
+		(property "Intersheetrefs" "${INTERSHEET_REFS}"
+			(at 37.1105 83.82 0)
+			(hide yes)
+			(show_name no)
+			(do_not_autoplace no)
+			(effects
+				(font
+					(size 1.27 1.27)
+				)
+				(justify right)
+			)
+		)
+	)
 	(global_label "CM5_3V"
 		(shape input)
@@
 		)
 	)
+	(global_label "ESP_RESET"
+		(shape input)
+		(at 50.8 73.66 180)
+		(fields_autoplaced yes)
+		(effects
+			(font
+				(size 1.27 1.27)
+			)
+			(justify right)
+		)
+		(property "Intersheetrefs" "${INTERSHEET_REFS}"
+			(at 37.4736 73.66 0)
+			(hide yes)
+			(show_name no)
+			(do_not_autoplace no)
+			(effects
+				(font
+					(size 1.27 1.27)
+				)
+				(justify right)
+			)
+		)
+	)
 	(global_label "3V3_CODEC"
 		(shape input)
@@
 		)
 	)
+	(global_label "ESP_BOOT"
+		(shape input)
+		(at 127 73.66 0)
+		(fields_autoplaced yes)
+		(effects
+			(font
+				(size 1.27 1.27)
+			)
+			(justify left)
+		)
+		(property "Intersheetrefs" "${INTERSHEET_REFS}"
+			(at 139.4799 73.66 0)
+			(hide yes)
+			(show_name no)
+			(do_not_autoplace no)
+			(effects
+				(font
+					(size 1.27 1.27)
+				)
+				(justify left)
+			)
+		)
+	)
 	(global_label "CM5_3V"
 		(shape input)
@@
 		)
 	)
-	(global_label "CM5_UART_RX"
+	(global_label "UI_UART_RX"
+		(shape input)
+		(at 50.8 58.42 180)
+		(fields_autoplaced yes)
+		(effects
+			(font
+				(size 1.27 1.27)
+			)
+			(justify right)
+		)
+		(property "Intersheetrefs" "${INTERSHEET_REFS}"
+			(at 37.1105 58.42 0)
+			(hide yes)
+			(show_name no)
+			(do_not_autoplace no)
+			(effects
+				(font
+					(size 1.27 1.27)
+				)
+				(justify right)
+			)
+		)
+	)
+	(global_label "CM5_DEBUG_UART_RX"
 		(shape input)
 		(at 125.73 81.28 0)
@@
 		)
 		(property "Intersheetrefs" "${INTERSHEET_REFS}"
-			(at 141.4151 81.28 0)
+			(at 148.9746 81.28 0)
 			(hide yes)
 			(show_name no)

Commit message: update psu
Connections:
- net +3V3 is gone; now on net CM5_3V: C68.1, C70.1, IC1.6 (IOVDD)
Changed lines of the file:
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@@
 	)
 	(junction
-		(at 149.86 168.91)
-		(diameter 0)
-		(color 0 0 0 0)
-	)
-	(junction
 		(at 124.46 154.94)
 		(diameter 0)
@@
 	(wire
 		(pts
+			(xy 146.05 166.37) (xy 144.78 166.37)
+		)
+		(stroke
+			(width 0)
+			(type default)
+		)
+	)
+	(wire
+		(pts
 			(xy 195.58 77.47) (xy 203.2 77.47)
 		)
@@
 	(wire
 		(pts
-			(xy 189.23 140.97) (xy 190.5 140.97)
+			(xy 144.78 166.37) (xy 144.78 168.91)
 		)
 		(stroke
@@
 	(wire
 		(pts
-			(xy 118.11 81.28) (xy 125.73 81.28)
+			(xy 189.23 140.97) (xy 190.5 140.97)
 		)
 		(stroke
@@
 	(wire
 		(pts
-			(xy 118.11 25.4) (xy 121.92 25.4)
+			(xy 118.11 81.28) (xy 125.73 81.28)
 		)
 		(stroke
@@
 	(wire
 		(pts
-			(xy 133.35 154.94) (xy 139.7 154.94)
+			(xy 118.11 25.4) (xy 121.92 25.4)
 		)
 		(stroke
@@
 	(wire
 		(pts
-			(xy 118.11 58.42) (xy 121.92 58.42)
+			(xy 133.35 154.94) (xy 139.7 154.94)
 		)
 		(stroke
@@
 	(wire
 		(pts
-			(xy 241.3 76.2) (xy 241.3 81.28)
+			(xy 118.11 58.42) (xy 121.92 58.42)
 		)
 		(stroke
@@
 	(wire
 		(pts
-			(xy 149.86 166.37) (xy 149.86 168.91)
+			(xy 241.3 76.2) (xy 241.3 81.28)
 		)
 		(stroke
@@
 	(global_label "CM5_3V"
 		(shape input)
+		(at 146.05 166.37 0)
+		(fields_autoplaced yes)
+		(effects
+			(font
+				(size 1.27 1.27)
+			)
+			(justify left)
+		)
+		(property "Intersheetrefs" "${INTERSHEET_REFS}"
+			(at 156.2318 166.37 0)
+			(hide yes)
+			(show_name no)
+			(do_not_autoplace no)
+			(effects
+				(font
+					(size 1.27 1.27)
+				)
+				(justify left)
+			)
+		)
+	)
+	(global_label "CM5_3V"
+		(shape input)
 		(at 36.83 121.92 180)
 		(fields_autoplaced yes)
@@
 					(unit 1)
 				)
-			)
-		)
-	)
-	(symbol
-		(lib_id "power:+3V3")
-		(at 149.86 166.37 0)
-		(unit 1)
-		(body_style 1)
-		(exclude_from_sim no)
-		(in_bom yes)
-		(on_board yes)
-		(in_pos_files yes)
-		(dnp no)
-		(property "Reference" "#PWR025"
-			(at 149.86 170.18 0)
-			(hide yes)
-			(show_name no)
-			(do_not_autoplace no)
-			(effects
-				(font
-					(size 1.27 1.27)
-				)
-			)
-		)
-		(property "Value" "+3V3"
-			(at 149.352 162.56 0)
-			(show_name no)
-			(do_not_autoplace no)
-			(effects
-				(font
-					(size 1.27 1.27)
-				)
-			)
-		)
-		(property "Footprint" ""
-			(at 149.86 166.37 0)
-			(hide yes)
-			(show_name no)
-			(do_not_autoplace no)
-			(effects
-				(font
-					(size 1.27 1.27)
-				)
-			)
-		)
-		(property "Datasheet" ""
-			(at 149.86 166.37 0)
-			(hide yes)
-			(show_name no)
-			(do_not_autoplace no)
-			(effects
-				(font
-					(size 1.27 1.27)
-				)
-			)
-		)
-		(property "Description" "Power symbol creates a global label with name \"+3V3\""
-			(at 149.86 166.37 0)
-			(hide yes)
-			(show_name no)
-			(do_not_autoplace no)
-			(effects
-				(font
-					(size 1.27 1.27)
-				)
-			)
-		)
-		(pin "1"
-		)
-		(instances
-			(project "pedalboard-hw"
-				(path "/df521c2a-9827-4355-b809-366f4b88d5d7/6bd0afd4-cd8b-4c1d-a236-891eed0b2d91"
-					(reference "#PWR025")
-					(unit 1)
-				)

Commit message: added test points
Parts:
- added TP4: CM5_3V3, TestPoint:TestPoint_Pad_D1.5mm, symbol Connector:TestPoint
Connections:
- net CM5_3V: now also TP4.1
Changed lines of the file:
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@@
 	)
 	(junction
+		(at 33.02 121.92)
+		(diameter 0)
+		(color 0 0 0 0)
+	)
+	(junction
 		(at 121.92 83.82)
 		(diameter 0)
@@
 	(wire
 		(pts
+			(xy 33.02 121.92) (xy 38.1 121.92)
+		)
+		(stroke
+			(width 0)
+			(type default)
+		)
+	)
+	(wire
+		(pts
 			(xy 167.64 52.07) (xy 168.91 52.07)
 		)
@@
 	(wire
 		(pts
-			(xy 36.83 121.92) (xy 38.1 121.92)
+			(xy 30.48 121.92) (xy 33.02 121.92)
 		)
 		(stroke
@@
 	(global_label "CM5_3V"
 		(shape input)
-		(at 36.83 121.92 180)
+		(at 30.48 121.92 180)
 		(fields_autoplaced yes)
 		(effects
@@
 		)
 		(property "Intersheetrefs" "${INTERSHEET_REFS}"
-			(at 26.6482 121.92 0)
+			(at 20.2982 121.92 0)
 			(hide yes)
 			(show_name no)
@@
 					(unit 1)
 				)
+			)
+		)
+	)
+	(symbol
+		(lib_id "Connector:TestPoint")
+		(at 33.02 121.92 0)
+		(unit 1)
+		(body_style 1)
+		(exclude_from_sim no)
+		(in_bom no)
+		(on_board yes)
+		(in_pos_files no)
+		(dnp no)
+		(property "Reference" "TP4"
+			(at 31.75 114.808 0)
+			(show_name no)
+			(do_not_autoplace no)
+			(effects
+				(font
+					(size 1.27 1.27)
+				)
+				(justify left)
+			)
+		)
+		(property "Value" "CM5_3V3"
+			(at 28.702 116.586 0)
+			(show_name no)
+			(do_not_autoplace no)
+			(effects
+				(font
+					(size 1.27 1.27)
+				)
+				(justify left)
+			)
+		)
+		(property "Footprint" "TestPoint:TestPoint_Pad_D1.5mm"
+			(at 38.1 121.92 0)
+			(hide yes)
+			(show_name no)
+			(do_not_autoplace no)
+			(effects
+				(font
+					(size 1.27 1.27)
+				)
+			)
+		)
+		(property "Datasheet" ""
+			(at 38.1 121.92 0)
+			(hide yes)
+			(show_name no)
+			(do_not_autoplace no)
+			(effects
+				(font
+					(size 1.27 1.27)
+				)
+			)
+		)
+		(property "Description" "test point"
+			(at 33.02 121.92 0)
+			(hide yes)
+			(show_name no)
+			(do_not_autoplace no)
+			(effects
+				(font
+					(size 1.27 1.27)
+				)
+			)
+		)
+		(pin "1"
+		)
+		(instances
+			(project "pedalboard-hw"
+				(path "/df521c2a-9827-4355-b809-366f4b88d5d7/6bd0afd4-cd8b-4c1d-a236-891eed0b2d91"
+					(reference "TP4")
+					(unit 1)
+				)

Commit message: initial placement fiddling
Parts:
- removed H4, H5, H6, H7: MountingHole, MountingHole:MountingHole_2.7mm_M2.5_DIN965, symbol Mechanical:MountingHole
- C81: footprint Capacitor_SMD:CP_Elec_6.3x5.8 -> Capacitor_THT:CP_Radial_D6.3mm_P2.50mm; JLCPCB part C1881583 -> (none); Manufacturer part EEE-FK1C470AL -> ECA1EHG101

Commit message: components placed.
Parts:
- C61: footprint Capacitor_SMD:C_0805_2012Metric -> Capacitor_SMD:C_0603_1608Metric; JLCPCB part C49678 -> C14663; Manufacturer part CC0805KRX7R9BB104 -> CC0603KRX7R9BB104
Other:
- note added: "U14 supply"
- moved on the sheet: C61, U14C
Changed lines of the file:
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@@
 	(text "Input gain:\n1+2 ON: LOW 1.39x\n1 ON, 2 OFF (or reverse): MID 2.21x\n1+2 OFF: HIGH 3.03x"
 		(exclude_from_sim no)
-		(at 192.024 84.836 0)
+		(at 201.168 83.312 0)
+		(effects
+			(font
+				(size 1.27 1.27)
+			)
+		)
+	)
+	(text "U14 supply"
+		(exclude_from_sim no)
+		(at 161.29 73.66 0)
 		(effects
 			(font
@@
 		)
 	)
-	(text_box "OPA1656 supply"
-		(exclude_from_sim no)
-		(at 19.05 160.02 0)
-		(size 22.86 33.02)
-		(margins 0.9525 0.9525 0.9525 0.9525)
-		(stroke
-			(width 0)
-			(type solid)
-		)
-		(fill
-			(type none)
-		)
-		(effects
-			(font
-				(size 1.27 1.27)
-			)
-			(justify left top)
-		)
-	)
 	(text_box "CODEC"
 		(exclude_from_sim no)
@@
 	)
 	(junction
-		(at 29.21 185.42)
+		(at 165.1 96.52)
 		(diameter 0)
 		(color 0 0 0 0)
@@
 	)
 	(junction
-		(at 29.21 170.18)
+		(at 165.1 81.28)
 		(diameter 0)
 		(color 0 0 0 0)
@@
 	(wire
 		(pts
-			(xy 25.4 179.07) (xy 25.4 185.42)
+			(xy 161.29 90.17) (xy 161.29 96.52)
 		)
 		(stroke
@@
 	(wire
 		(pts
-			(xy 29.21 168.91) (xy 29.21 170.18)
+			(xy 165.1 80.01) (xy 165.1 81.28)
 		)
 		(stroke
@@
 	(wire
 		(pts
-			(xy 29.21 185.42) (xy 29.21 186.69)
+			(xy 165.1 96.52) (xy 165.1 97.79)
 		)
 		(stroke
@@
 	(wire
 		(pts
-			(xy 25.4 170.18) (xy 29.21 170.18)
+			(xy 161.29 81.28) (xy 165.1 81.28)
 		)
 		(stroke
@@
 	(wire
 		(pts
-			(xy 25.4 185.42) (xy 29.21 185.42)
+			(xy 161.29 96.52) (xy 165.1 96.52)
 		)
 		(stroke
@@
 	(wire
 		(pts
-			(xy 25.4 173.99) (xy 25.4 170.18)
+			(xy 161.29 85.09) (xy 161.29 81.28)
 		)
 		(stroke
@@
 	(symbol
 		(lib_id "power:+10V")
-		(at 29.21 168.91 0)
+		(at 165.1 80.01 0)
 		(unit 1)
 		(body_style 1)
@@
 		(dnp no)
 		(property "Reference" "#PWR086"
-			(at 29.21 172.72 0)
+			(at 165.1 83.82 0)
 			(hide yes)
 			(show_name no)
@@
 		)
 		(property "Value" "+10V"
-			(at 29.718 165.1 0)
+			(at 165.608 76.2 0)
 			(show_name no)
 			(do_not_autoplace no)
@@
 		)
 		(property "Footprint" ""
-			(at 29.21 168.91 0)
+			(at 165.1 80.01 0)
 			(hide yes)
 			(show_name no)
@@
 		)
 		(property "Datasheet" ""
-			(at 29.21 168.91 0)
+			(at 165.1 80.01 0)
 			(hide yes)
 			(show_name no)
@@
 		)
 		(property "Description" "Power symbol creates a global label with name \"+10V\""
-			(at 29.21 168.91 0)
+			(at 165.1 80.01 0)
 			(hide yes)
 			(show_name no)
@@
 	(symbol
 		(lib_id "Amplifier_Operational:OPA1656ID")
-		(at 31.75 177.8 0)
+		(at 167.64 88.9 0)
 		(unit 3)
 		(body_style 1)
@@
 		(fields_autoplaced yes)
 		(property "Reference" "U14"
-			(at 30.48 176.5299 0)
+			(at 166.37 87.6299 0)
 			(show_name no)
 			(do_not_autoplace no)
@@
 		)
 		(property "Value" "OPA1656ID"
-			(at 30.48 179.0699 0)
+			(at 166.37 90.1699 0)
 			(show_name no)
 			(do_not_autoplace no)
@@
 		)
 		(property "Footprint" "Package_SO:SOIC-8_3.9x4.9mm_P1.27mm"
-			(at 31.75 177.8 0)
+			(at 167.64 88.9 0)
 			(hide yes)
 			(show_name no)
@@
 		)
 		(property "Datasheet" "https://www.ti.com/lit/ds/symlink/opa1656.pdf"
-			(at 31.75 177.8 0)
+			(at 167.64 88.9 0)
 			(hide yes)
 			(show_name no)
@@
 		)
 		(property "Description" "Dual Ultra-Low-Noise, Low-Distortion, FET-Input, Burr-Brown Audio Operational Amplifiers, SOIC-8"
-			(at 31.75 177.8 0)
+			(at 167.64 88.9 0)
 			(hide yes)
 			(show_name no)
@@
 		)
 		(property "Manufacturer" "Texas Instruments"
-			(at 31.75 177.8 0)
+			(at 167.64 88.9 0)
 			(hide yes)
 			(show_name no)
@@
 		)
 		(property "Manufacturer part" "OPA1656ID"
-			(at 31.75 177.8 0)
+			(at 167.64 88.9 0)
 			(hide yes)
 			(show_name no)
@@
 		)
 		(property "JLCPCB part" "C1346368"
-			(at 31.75 177.8 0)
+			(at 167.64 88.9 0)
 			(hide yes)
 			(show_name no)
@@
 	(symbol
 		(lib_id "power:GND")
-		(at 29.21 186.69 0)
+		(at 165.1 97.79 0)
 		(unit 1)
 		(body_style 1)
@@
 		(dnp no)
 		(property "Reference" "#PWR085"
-			(at 29.21 193.04 0)
+			(at 165.1 104.14 0)
 			(hide yes)
 			(show_name no)
@@
 		)
 		(property "Value" "GND"
-			(at 33.02 189.23 0)
+			(at 168.91 100.33 0)
 			(show_name no)
 			(do_not_autoplace no)
@@
 		)
 		(property "Footprint" ""
-			(at 29.21 186.69 0)
+			(at 165.1 97.79 0)
 			(hide yes)
 			(show_name no)
@@
 		)
 		(property "Datasheet" ""
-			(at 29.21 186.69 0)
+			(at 165.1 97.79 0)
 			(hide yes)
 			(show_name no)
@@
 		)
 		(property "Description" "Power symbol creates a global label with name \"GND\" , ground"
-			(at 29.21 186.69 0)
+			(at 165.1 97.79 0)
 			(hide yes)
 			(show_name no)
@@
 	(symbol
 		(lib_id "Device:C_Small")
-		(at 25.4 176.53 0)
+		(at 161.29 87.63 0)
 		(unit 1)
 		(body_style 1)
@@
 		(dnp no)
 		(property "Reference" "C61"
-			(at 19.558 175.006 0)
+			(at 155.448 86.106 0)
 			(show_name no)
 			(do_not_autoplace no)
@@
 		)
 		(property "Value" "100nF"
-			(at 19.05 178.308 0)
+			(at 154.94 89.408 0)
 			(show_name no)
 			(do_not_autoplace no)
@@
 			)
 		)
-		(property "Footprint" "Capacitor_SMD:C_0805_2012Metric"
-			(at 26.3652 180.34 0)
+		(property "Footprint" "Capacitor_SMD:C_0603_1608Metric"
+			(at 162.2552 91.44 0)
 			(hide yes)
 			(show_name no)
@@
 		)
 		(property "Datasheet" ""
-			(at 25.4 176.53 0)
+			(at 161.29 87.63 0)
 			(hide yes)
 			(show_name no)
@@
 		)
 		(property "Description" ""
-			(at 25.4 176.53 0)
+			(at 161.29 87.63 0)
 			(hide yes)
 			(show_name no)
@@
 		)
 		(property "Manufacturer" "Yageo"
-			(at 25.4 176.53 0)
+			(at 161.29 87.63 0)
 			(hide yes)
 			(show_name no)
@@
 			)
 		)
-		(property "Manufacturer part" "CC0805KRX7R9BB104"
-			(at 25.4 176.53 0)
+		(property "Manufacturer part" "CC0603KRX7R9BB104"
+			(at 161.29 87.63 0)
 			(hide yes)
 			(show_name no)
@@
 			)
 		)
-		(property "JLCPCB part" "C49678"
-			(at 25.4 176.53 0)
+		(property "JLCPCB part" "C14663"
+			(at 161.29 87.63 0)
 			(hide yes)
 			(show_name no)

Commit message: opamp incl power routed
Parts:
- removed C64: 100nF, Capacitor_SMD:C_1206_3216Metric_Pad1.33x1.80mm_HandSolder, symbol Device:C_Small
Changed lines of the file:
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@@
 	)
 	(junction
-		(at 180.34 46.99)
-		(diameter 0)
-		(color 0 0 0 0)
-	)
-	(junction
 		(at 91.44 184.15)
 		(diameter 0)
@@
 	(wire
 		(pts
-			(xy 180.34 39.37) (xy 180.34 46.99)
-		)
-		(stroke
-			(width 0)
-			(type default)
-		)
-	)
-	(wire
-		(pts
 			(xy 74.93 175.26) (xy 74.93 173.99)
 		)
@@
 	(wire
 		(pts
-			(xy 177.8 39.37) (xy 180.34 39.37)
-		)
-		(stroke
-			(width 0)
-			(type default)
-		)
-	)
-	(wire
-		(pts
 			(xy 179.07 46.99) (xy 189.23 46.99)
 		)
@@
 	(wire
 		(pts
-			(xy 172.72 39.37) (xy 171.45 39.37)
-		)
-		(stroke
-			(width 0)
-			(type default)
-		)
-	)
-	(wire
-		(pts
 			(xy 190.5 153.67) (xy 194.31 153.67)
 		)
@@
 	(wire
 		(pts
-			(xy 171.45 39.37) (xy 171.45 46.99)
-		)
-		(stroke
-			(width 0)
-			(type default)
-		)
-	)
-	(wire
-		(pts
 			(xy 168.91 57.15) (xy 171.45 57.15)
 		)
@@
 	)
 	(symbol
-		(lib_id "Device:C_Small")
-		(at 175.26 39.37 90)
-		(unit 1)
-		(body_style 1)
-		(exclude_from_sim no)
-		(in_bom yes)
-		(on_board yes)
-		(in_pos_files yes)
-		(dnp yes)
-		(property "Reference" "C64"
-			(at 178.816 38.354 90)
-			(show_name no)
-			(do_not_autoplace no)
-			(effects
-				(font
-					(size 1.27 1.27)
-				)
-			)
-		)
-		(property "Value" "100nF"
-			(at 170.942 38.1 90)
-			(show_name no)
-			(do_not_autoplace no)
-			(effects
-				(font
-					(size 1.27 1.27)
-				)
-			)
-		)
-		(property "Footprint" "Capacitor_SMD:C_1206_3216Metric_Pad1.33x1.80mm_HandSolder"
-			(at 175.26 39.37 0)
-			(hide yes)
-			(show_name no)
-			(do_not_autoplace no)
-			(effects
-				(font
-					(size 1.27 1.27)
-				)
-			)
-		)
-		(property "Datasheet" ""
-			(at 175.26 39.37 0)
-			(hide yes)
-			(show_name no)
-			(do_not_autoplace no)
-			(effects
-				(font
-					(size 1.27 1.27)
-				)
-			)
-		)
-		(property "Description" "C0G alternative"
-			(at 175.26 39.37 0)
-			(hide yes)
-			(show_name no)
-			(do_not_autoplace no)
-			(effects
-				(font
-					(size 1.27 1.27)
-				)
-			)
-		)
-		(pin "2"
-		)
-		(pin "1"
-		)
-		(instances
-			(project "pedalboard-hw"
-				(path "/df521c2a-9827-4355-b809-366f4b88d5d7/6bd0afd4-cd8b-4c1d-a236-891eed0b2d91"
-					(reference "C64")
-					(unit 1)
-				)
-			)
-		)
-	)
-	(symbol
 		(lib_id "Connector_Audio:AudioJack3_SwitchTR")
 		(at 252.73 121.92 180)
@@
 		(dnp no)
 		(property "Reference" "C56"
-			(at 176.784 43.942 90)
+			(at 176.53 42.418 90)
 			(show_name no)
 			(do_not_autoplace no)
@@
 		)
 		(property "Value" "100nF"
-			(at 180.594 48.768 90)
+			(at 176.784 44.196 90)
 			(show_name no)
 			(do_not_autoplace no)

Commit message: more routing.
Parts:
- removed TP4: CM5_3V3, TestPoint:TestPoint_Pad_D1.5mm, symbol Connector:TestPoint
Changed lines of the file:
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@@
 	)
 	(junction
-		(at 33.02 121.92)
-		(diameter 0)
-		(color 0 0 0 0)
-	)
-	(junction
 		(at 121.92 83.82)
 		(diameter 0)
@@
 	(wire
 		(pts
-			(xy 33.02 121.92) (xy 38.1 121.92)
+			(xy 30.48 121.92) (xy 38.1 121.92)
 		)
 		(stroke
@@
 	(wire
 		(pts
-			(xy 30.48 121.92) (xy 33.02 121.92)
-		)
-		(stroke
-			(width 0)
-			(type default)
-		)
-	)
-	(wire
-		(pts
 			(xy 167.64 44.45) (xy 168.91 44.45)
 		)
@@
 					(unit 1)
 				)
-			)
-		)
-	)
-	(symbol
-		(lib_id "Connector:TestPoint")
-		(at 33.02 121.92 0)
-		(unit 1)
-		(body_style 1)
-		(exclude_from_sim no)
-		(in_bom no)
-		(on_board yes)
-		(in_pos_files no)
-		(dnp no)
-		(property "Reference" "TP4"
-			(at 31.75 114.808 0)
-			(show_name no)
-			(do_not_autoplace no)
-			(effects
-				(font
-					(size 1.27 1.27)
-				)
-				(justify left)
-			)
-		)
-		(property "Value" "CM5_3V3"
-			(at 28.702 116.586 0)
-			(show_name no)
-			(do_not_autoplace no)
-			(effects
-				(font
-					(size 1.27 1.27)
-				)
-				(justify left)
-			)
-		)
-		(property "Footprint" "TestPoint:TestPoint_Pad_D1.5mm"
-			(at 38.1 121.92 0)
-			(hide yes)
-			(show_name no)
-			(do_not_autoplace no)
-			(effects
-				(font
-					(size 1.27 1.27)
-				)
-			)
-		)
-		(property "Datasheet" ""
-			(at 38.1 121.92 0)
-			(hide yes)
-			(show_name no)
-			(do_not_autoplace no)
-			(effects
-				(font
-					(size 1.27 1.27)
-				)
-			)
-		)
-		(property "Description" "test point"
-			(at 33.02 121.92 0)
-			(hide yes)
-			(show_name no)
-			(do_not_autoplace no)
-			(effects
-				(font
-					(size 1.27 1.27)
-				)
-			)
-		)
-		(pin "1"
-		)
-		(instances
-			(project "pedalboard-hw"
-				(path "/df521c2a-9827-4355-b809-366f4b88d5d7/6bd0afd4-cd8b-4c1d-a236-891eed0b2d91"
-					(reference "TP4")
-					(unit 1)
-				)

Commit message: various fixes.
Parts:
- D3: now fitted
Changed lines of the file:
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@@
 		(on_board yes)
 		(in_pos_files yes)
-		(dnp yes)
+		(dnp no)
 		(property "Reference" "D3"
 			(at 173.736 51.054 90)
