File: pico.kicad_sch (KiCad schematic)
At the start: 63 parts, among them J1 Jack 3.5mm, J12 Debug, J14 JST PH 4, J2 DIN5, J25 JST PH 3, J26 JST PH 3, J3 Jack 3.5mm, J4 DIN5, J5 Jack 6.35mm, J8 Jack 6.35mm, SW1 24P/R 24mm, SW10 Momentary switch, SW2 24P/R 24mm, SW3 Micro Button, SW4 Micro Button, SW5 Momentary switch, SW6 Momentary switch, SW7 Momentary switch, SW8 Momentary switch, SW9 Momentary switch, U12 AT24CS01-STUM, U2 TLP2761, U3 RP2040, U4 W25Q128JVS, Y2 ABM8-272-T3

Commit message: Changed to CM5, removed unnecessary USB chips, Changing RP2024 to STM32.
Parts:
- removed C22, C26: 15p, Capacitor_SMD:C_0805_2012Metric, symbol Device:C_Small
- removed JP1, JP2: SJP, symbol Jumper:SolderJumper_2_Bridged
- removed R11: 1K, Resistor_SMD:R_0805_2012Metric, symbol Device:R_Small
- removed Y2: ABM8-272-T3, Pedalboard Library:ABM8-272-T3_ABR, symbol pedalboard:ABM8-272-T3
- added U7: STM32G0B1CET6, Package_QFP:LQFP-48_7x7mm_P0.5mm, symbol MCU_ST_STM32G0:STM32G0B1CETx
- C17: value 100n -> 4.7uF; Digikey 1276-1180-1-ND -> (none); JLCPCB part (none) -> C1779; Manufacturer part (none) -> CL21A475KAQNNNE; Mouser 581-08055C104K -> (none); Notes 10% 16V Ceramic Capacitor X7R -> (none); Supplier https://www.digikey.ch/de/products/detail/samsung-electro-m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 -> (none)
Connections:
- net +3V3: now also U7.4 (VBAT), U7.5 (VREF+), U7.6 (VDD); no longer C18.1
- net GND: now also U7.7 (VSS)
- net USB_RP_N renamed USB_STM32_N
- net USB_RP_P renamed USB_STM32_P
- new net STM32_NRST: C18.1, U7.10 (PF2)
Other:
- note added: "Place C13/14 close to VREF"
- note added: "Place C15/17 close to VDD"
- moved on the sheet: C13, C14, C15, C17, C18

Commit message: Updated to use STM32
Parts:
- removed R10, R6: 27R, Resistor_SMD:R_0805_2012Metric, symbol Device:R_Small
- removed U3: RP2040, Pedalboard Library:RP2040-QFN-56, symbol pedalboard:RP2040
- removed U4: W25Q128JVS, Pedalboard Library:SOIC-8_5.23x5.23mm_P1.27mm, symbol pedalboard:W25Q128JVS-Memory_Flash
- added C22: 100n, Capacitor_SMD:C_0805_2012Metric, symbol Device:C_Small
- added J15: HS20S010B Left, Connector_PinSocket_2.54mm:PinSocket_1x10_P2.54mm_Vertical, symbol Connector_Generic:Conn_01x10
- added J17: HS20S010B Right, Connector_PinSocket_2.54mm:PinSocket_1x10_P2.54mm_Vertical, symbol Connector_Generic:Conn_01x10
- added TP5: TestPoint, TestPoint:TestPoint_Pad_2.0x2.0mm, symbol Connector:TestPoint
- C1, J1, J3, L1, L2, L3, L4, R3, R4, R5, U2: now not fitted
- C12: value 1u -> 10u; JLCPCB part (none) -> C15850; Manufacturer part (none) -> CL21A106KAYNNNE; Notes 25V/10% -> (none); Supplier https://www.digikey.ch/de/products/detail/samsung-electro-m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 -> (none)
- C21: value 100n -> 10u; Digikey 1276-1180-1-ND -> (none); JLCPCB part (none) -> C15850; Manufacturer part (none) -> CL21A106KAYNNNE; Mouser 581-08055C104K -> (none); Notes 10% 16V Ceramic Capacitor X7R -> (none); Supplier https://www.digikey.ch/de/products/detail/samsung-electro-m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 -> (none)
- D1: value SM4007 -> 1N4148W; JLCPCB part (none) -> C81598; Manufacturer part (none) -> 1N4148W; Supplier https://www.digikey.ch/de/products/detail/micro-commercial-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 -> (none); now not fitted
- J12: value Debug -> SWD; footprint Connector_PinHeader_2.54mm:PinHeader_1x03_P2.54mm_Vertical -> Connector_PinHeader_2.54mm:PinHeader_1x05_P2.54mm_Vertical; symbol Connector:Conn_01x03_Pin -> Connector_Generic:Conn_01x05
- R9: value DNF -> 1K; Supplier (none) -> https://www.digikey.ch/de/products/detail/stackpole-electro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; now fitted
- renumbered U7 to U3
Connections:
- net +1V1 is gone; now on net +3V3: C12.1, C16.1, C21.1
- net SWCLK is gone; now on net +3V3: J12.1 (Pin_1)
- net SWD is gone; now on net GND: J12.3 (Pin_3)
- net +3V3: now also C22.1, J15.10 (Pin_10), J15.2 (Pin_2), J17.10 (Pin_10), J17.2 (Pin_2); no longer C19.1, C20.1, R9.1
- net A_EXP1: now also C19.1, R8.1, U3.19 (PB0); no longer J5.R
- net A_EXP2: now also C20.1, R9.1, U3.20 (PB1); no longer J8.R
- net EXT_MIDI_RX: now also U3.46 (PB7)
- net EXT_MIDI_TX: now also U3.45 (PB6)
- net GND: now also C22.2, J15.1 (Pin_1), J17.1 (Pin_1); no longer J12.2 (Pin_2)
- net I2C_SCL: now also U3.47 (PB8)
- net I2C_SDA: now also U3.48 (PB9)
- net RGB_DATA: now also U3.28 (PA8)
- net ROT_GAIN_A: now also U3.13 (PA2)
- net ROT_GAIN_B: now also U3.14 (PA3)
- net ROT_VOL_A: now also U3.11 (PA0)
- net ROT_VOL_B: now also U3.12 (PA1)
- net STM32_NRST: now also J12.5 (Pin_5), SW4.2
- net SW_A: now also U3.38 (PD0)
- net SW_B: now also U3.39 (PD1)
- net SW_C: now also U3.40 (PD2)
- net SW_D: now also U3.41 (PD3)
- net SW_E: now also U3.43 (PB4)
- net SW_F: now also U3.44 (PB5)
- net SW_GAIN: now also U3.42 (PB3)
- net SW_VOL: now also U3.21 (PB2)
- net USB_STM32_N: now also U3.33 (PA9/PA11)
- net USB_STM32_P: now also U3.34 (PA10/PA12)
- net STM32_BOOT_REQ_N: now reaches U3.1 (PC13)
- net STM32_BOOT_REQ_N: now also SW3.2
- net TFT_DC: now reaches U3.15 (PA4)
- net TFT_DC: now also J15.6 (Pin_6), J17.6 (Pin_6)
- net TFT_SCK: now reaches U3.16 (PA5)
- net TFT_SCK: now also J15.3 (Pin_3), J17.3 (Pin_3)
- net TFT_BL_PWM: now reaches U3.17 (PA6)
- net TFT_BL_PWM: now also J15.8 (Pin_8), J17.8 (Pin_8)
- net TFT_MOSI: now reaches U3.18 (PA7)
- net TFT_MOSI: now also J15.4 (Pin_4), J17.4 (Pin_4)
- net TFT_LEFT_CS_N: now reaches U3.22 (PB10)
- net TFT_LEFT_CS_N: now also J15.7 (Pin_7)
- net TFT_RIGHT_CS_N: now reaches U3.23 (PB11)
- net TFT_RIGHT_CS_N: now also J17.7 (Pin_7)
- net TFT_RESET_N: now reaches U3.24 (PB12)
- net TFT_RESET_N: now also J15.5 (Pin_5), J17.5 (Pin_5)
- net STM32_STATUS_LED: now reaches U3.27 (PB15)
- net STM32_STATUS_LED: now also R21.2
- net STM32_DBG_TX: now reaches U3.29 (PA9/UCPD1_DBCC1)
- net STM32_DBG_TX: now also TP4.1
- net STM32_DBG_RX: now reaches U3.32 (PA10/UCPD1_DBCC2)
- net STM32_DBG_RX: now also TP5.1
- net STM32_SWDIO: now reaches U3.35 (PA13)
- net STM32_SWDIO: now also J12.2 (Pin_2)
- net STM32_SWCLK: now reaches U3.36 (PA14)
- net STM32_SWCLK: now also J12.4 (Pin_4)
- net at R21.1: now also D2.2 (A)
- net QSPI_SS: no longer names the net of R9.2
- net QSPI_SS: now also J8.R; no longer R8.2
- removed net ~{USB_BOOT}: R8.1, SW3.2
- new net: J5.R, R8.2
- no-connect marks 22 -> 25
Other:
- note added: "NOTE: 3V3 supply must be upgraded for two TFTs target at least 500mA usable output"
- note removed: "Alternative to USB connection between CM4 and Pico (Can be used for MIDI)"
- note removed: "Make C is close to pin 45 of RP2040"
- note removed: "Make sure C is close to pin 44 of RP2040"
- note removed: "Make sure R10 and R11 are close to RP2040"
- moved on the sheet: C12, C13, C14, C15, C16, C17, C18, C19, C20, C52, D2, H2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

Commit message: updated lcd connectors
Parts:
- removed C12, C21: 10u, Capacitor_SMD:C_0805_2012Metric, symbol Device:C_Small
- removed C16, C23: 100n, Capacitor_SMD:C_0805_2012Metric, symbol Device:C_Small
- removed J15: HS20S010B Left, Connector_PinSocket_2.54mm:PinSocket_1x10_P2.54mm_Vertical, symbol Connector_Generic:Conn_01x10
- removed J17: HS20S010B Right, Connector_PinSocket_2.54mm:PinSocket_1x10_P2.54mm_Vertical, symbol Connector_Generic:Conn_01x10
- added J15, J17: LCD left, Connector_JST:JST_PH_B8B-PH-K_1x08_P2.00mm_Vertical, symbol Connector_Generic:Conn_01x08
Connections:
- net +3V3: now also J15.8 (Pin_8), J17.8 (Pin_8)
- net GND: now also J15.7 (Pin_7), J17.7 (Pin_7)
- net TFT_BL_PWM: now also J15.1 (Pin_1), J17.1 (Pin_1)
- net TFT_DC: now also J15.3 (Pin_3), J17.3 (Pin_3)
- net TFT_LEFT_CS_N: now also J15.4 (Pin_4), J17.4 (Pin_4)
- net TFT_MOSI: now also J15.6 (Pin_6), J17.6 (Pin_6)
- net TFT_RESET_N: now also J15.2 (Pin_2), J17.2 (Pin_2)
- net TFT_SCK: now also J15.5 (Pin_5), J17.5 (Pin_5)
- no-connect marks 25 -> 23
Other:
- note added: "Foot Switches"
- note removed: "Foot Buttons"
- note removed: "NOTE: 3V3 supply must be upgraded for two TFTs target at least 500mA usable output"

Commit message: small fixes
Parts:
- J17: value LCD left -> LCD right
Connections:
- net TFT_LEFT_CS_N: no longer J17.4 (Pin_4)
- net TFT_RIGHT_CS_N: now also J17.4 (Pin_4)
Other:
- note added: "MIDI Bites allow to remove some of the board material that is used to hold the DIN5 or 3.5mm Jack connectors and instead mount the connectors to the case"
- note removed: "MIDI Bites allow to remove some of the board material that is used to hold the DIN5 or 3.5mm Jack connectors and instead mount the connectors to the case and wire them up with J15"
Changed lines of the file:
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@@
 		)
 	)
-	(text "MIDI Bites allow to remove some of the \nboard material that is used to hold the\nDIN5 or 3.5mm Jack connectors and instead\nmount the connectors to the case and wire \nthem up with J15 "
+	(text "MIDI Bites allow to remove some of the \nboard material that is used to hold the\nDIN5 or 3.5mm Jack connectors and instead\nmount the connectors to the case"
 		(exclude_from_sim no)
 		(at 28.956 195.326 0)
@@
 		)
 	)
-	(label "TFT_LEFT_CS_N"
+	(label "TFT_RIGHT_CS_N"
 		(at 276.86 100.33 180)
 		(effects
@@
 			)
 		)
-		(property "Value" "LCD left"
+		(property "Value" "LCD right"
 			(at 260.096 88.9 0)
 			(show_name no)

Commit message: small edits
Parts:
- D1: footprint Diode_SMD:D_SOD-123F -> Diode_SMD:D_SOD-123
Changed lines of the file:
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@@
 			)
 		)
-		(property "Footprint" "Diode_SMD:D_SOD-123F"
+		(property "Footprint" "Diode_SMD:D_SOD-123"
 			(at 54.61 80.01 0)
 			(hide yes)

Commit message: a few edits
Parts:
- SW3: Notes Boot -> Firmware DFU request - requires working firmware, use SWD f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
Changed lines of the file:
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@@
 			)
 		)
-		(property "Notes" "Boot"
+		(property "Notes" "Firmware DFU request - requires working firmware, use SWD for recovery"
 			(at 99.06 96.52 0)
 			(hide yes)

Commit message: Standardize values.
Parts:
- C1, C13, C15, C18, C19, C20, C22, C52: value 100n -> 100nF
- C14: value 1u -> 1uF
- R1, R2, R8, R9: value 1K -> 1k
- R18, R19: value 3K9 -> 3k9
- R21: value 2K2 -> 2k2
Changed lines of the file:
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@@
 			)
 		)
-		(property "Value" "100n"
+		(property "Value" "100nF"
 			(at 86.106 160.274 0)
 			(show_name no)
@@
 			)
 		)
-		(property "Value" "3K9"
+		(property "Value" "3k9"
 			(at 151.13 162.56 90)
 			(show_name no)
@@
 			)
 		)
-		(property "Value" "1K"
+		(property "Value" "1k"
 			(at 95.504 173.228 0)
 			(show_name no)
@@
 			)
 		)
-		(property "Value" "100n"
+		(property "Value" "100nF"
 			(at 33.02 99.06 0)
 			(show_name no)
@@
 			)
 		)
-		(property "Value" "100n"
+		(property "Value" "100nF"
 			(at 88.138 185.928 0)
 			(show_name no)
@@
 			)
 		)
-		(property "Value" "3K9"
+		(property "Value" "3k9"
 			(at 151.13 160.02 90)
 			(show_name no)
@@
 			)
 		)
-		(property "Value" "2K2"
+		(property "Value" "2k2"
 			(at 192.278 142.748 0)
 			(show_name no)
@@
 			)
 		)
-		(property "Value" "100n"
+		(property "Value" "100nF"
 			(at 96.52 53.848 0)
 			(show_name no)
@@
 			)
 		)
-		(property "Value" "100n"
+		(property "Value" "100nF"
 			(at 95.504 72.644 0)
 			(show_name no)
@@
 			)
 		)
-		(property "Value" "1K"
+		(property "Value" "1k"
 			(at 95.504 148.082 0)
 			(show_name no)
@@
 			)
 		)
-		(property "Value" "1u"
+		(property "Value" "1uF"
 			(at 106.172 53.594 0)
 			(show_name no)
@@
 			)
 		)
-		(property "Value" "100n"
+		(property "Value" "100nF"
 			(at 163.83 44.196 0)
 			(show_name no)
@@
 			)
 		)
-		(property "Value" "1K"
+		(property "Value" "1k"
 			(at 98.044 183.388 90)
 			(show_name no)
@@
 			)
 		)
-		(property "Value" "1K"
+		(property "Value" "1k"
 			(at 96.774 157.988 90)
 			(show_name no)
@@
 			)
 		)
-		(property "Value" "100n"
+		(property "Value" "100nF"
 			(at 82.804 85.598 0)
 			(show_name no)
@@
 			)
 		)
-		(property "Value" "100n"
+		(property "Value" "100nF"
 			(at 121.92 185.166 0)
 			(show_name no)
