File: pico.kicad_sch (KiCad schematic)
At the start: 54 parts, among them J1 Jack 3.5mm, J12 SWD, J14 JST PH 4, J15 LCD left, J17 LCD right, J2 DIN5, J25 JST PH 3, J26 JST PH 3, J3 Jack 3.5mm, J4 DIN5, J5 Jack 6.35mm, J8 Jack 6.35mm, SW1 24P/R 24mm, SW10 Momentary switch, SW2 24P/R 24mm, SW3 Micro Button, SW4 Micro Button, SW5 Momentary switch, SW6 Momentary switch, SW7 Momentary switch, SW8 Momentary switch, SW9 Momentary switch, U12 AT24CS01-STUM, U2 TLP2761, U3 STM32G0B1CET6

Commit message: more meta
Parts:
- removed R2: 1k, Resistor_SMD:R_0805_2012Metric, symbol Device:R_Small
- added R6: 1k, Resistor_SMD:R_0805_2012Metric, symbol Device:R_Small
- C1: Digikey 1276-1180-1-ND -> (none); JLCPCB part (none) -> C49678; Manufacturer (none) -> Yageo; Manufacturer part (none) -> C49678; Mouser 581-08055C104K -> (none); Notes 10% 16V Ceramic Capacitor X7R -> (none); Supplier https://www.digikey.ch/de/products/detail/samsung-electro-m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 -> (none)
- C13, C15, C18, C19, C20, C52: Digikey 1276-1180-1-ND -> (none); JLCPCB part (none) -> C49678; Manufacturer (none) -> Yageo; Manufacturer part (none) -> CC0805KRX7R9BB104; Mouser 581-08055C104K -> (none); Notes 10% 16V Ceramic Capacitor X7R -> (none); Supplier https://www.digikey.ch/de/products/detail/samsung-electro-m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 -> (none)
- C14: JLCPCB part (none) -> C28323; Manufacturer part (none) -> CL21B105KBFNNNE; Notes 25V/10% -> (none); Supplier https://www.digikey.ch/de/products/detail/samsung-electro-m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 -> (none)
- R1, R8, R9: JLCPCB part (none) -> C17513; Manufacturer part (none) -> 0805W8F1001T5E; Supplier https://www.digikey.ch/de/products/detail/stackpole-electro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 -> (none)
- R18, R19: JLCPCB part (none) -> C17614; Manufacturer part (none) -> 0805W8F3901T5E; Supplier https://www.digikey.ch/de/products/detail/stackpole-electro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 -> (none)
- R21: JLCPCB part (none) -> C17520; Supplier https://www.digikey.ch/de/products/detail/stackpole-electro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 -> (none)
- R3: JLCPCB part (none) -> C17557; Manufacturer part (none) -> 0805W8F2200T5E; Supplier https://www.digikey.ch/de/products/detail/stackpole-electro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 -> (none)
- R4: JLCPCB part (none) -> C17634; Supplier https://www.digikey.ch/de/products/detail/stackpole-electro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 -> (none)
- R5: JLCPCB part (none) -> C17415; Notes Resistor 10R 1% 63mW -> (none); Supplier https://www.digikey.ch/de/products/detail/stackpole-electro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 -> (none)
Connections:
- net +3V3: now also R6.1
- net at J8.T: now also R6.2

Commit message: Updated various metadata
Parts:
- C1: Manufacturer part C49678 -> CC0805KRX7R9BB104
- C14, C17: Manufacturer (none) -> Samsung Electro-Mechanics
- C22: Manufacturer (none) -> Yageo
- D1: Manufacturer (none) -> ST(Semtech)
- D2: JLCPCB part (none) -> C2296; Manufacturer (none) -> Hubei KENTO Elec; Manufacturer part (none) -> KT-0805Y; Supplier https://www.digikey.ch/en/products/detail/harvatek-corporat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 -> (none)
- J1, J3: Manufacturer (none) -> Same Sky; Manufacturer part (none) -> SJ1-3525NG; Supplier https://www.digikey.ch/de/products/detail/cui-devices/SJ1-3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 -> (none)
- J14: Manufacturer (none) -> JST; Manufacturer part (none) -> B4B-PH-SM4-TB(LF)(SN); Supplier https://www.digikey.ch/de/products/detail/jst-sales-america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 -> (none)
- J2, J4: Manufacturer (none) -> Switchcraft; Manufacturer part (none) -> 57PC5F; Supplier https://www.digikey.ch/de/products/detail/switchcraft-inc/5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 -> (none)
- J25, J26: Manufacturer (none) -> JST; Manufacturer part (none) -> B3B-PH-K-S(LF)(SN); Supplier https://www.digikey.ch/en/products/detail/jst-sales-america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 -> (none)
- J5, J8: Supplier https://www.digikey.ch/de/products/detail/schurter-inc/4833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 -> (none)
- L1, L2, L3, L4: JLCPCB part (none) -> C85831; Manufacturer (none) -> Murata Electronics; Manufacturer part (none) -> BLM18KG121TN1D; Supplier https://www.digikey.ch/de/products/detail/murata-electronic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 -> (none)
- R1, R18, R19, R3, R6, R8, R9: Manufacturer (none) -> UNI-ROYAL
- R21: Manufacturer (none) -> UNI-ROYAL; Manufacturer part (none) -> 0805W8F2201T5E
- R4: Manufacturer (none) -> UNI-ROYAL; Manufacturer part (none) -> 0805W8F330JT5E
- R5: Manufacturer (none) -> UNI-ROYAL; Manufacturer part (none) -> 0805W8F100JT5E
- SW1, SW2: Supplier https://www.digikey.ch/en/products/detail/bourns-inc/PEC11R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 -> (none)
- SW3, SW4: Supplier https://www.digikey.ch/en/products/detail/omron-electronics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 -> (none)
- U12: JLCPCB part (none) -> C616257; Manufacturer (none) -> Microchip Technology; Manufacturer part (none) -> AT24CS01-STUM-T; Supplier https://www.digikey.ch/de/products/detail/microchip-technol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 -> (none)
- U2: JLCPCB part (none) -> C4153769; Manufacturer (none) -> Toshiba Electronic Devices & Storage; Manufacturer part (none) -> TLP2761(TP,E; Supplier https://www.digikey.ch/de/products/detail/toshiba-semicondu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 -> (none)
Other:
- moved on the sheet: C52
