File: connect.kicad_sch (KiCad schematic)
At the start: 35 parts, among them J10 USB_A, J11 Conn_01x02, J9 USB_OTG, U10 AP2553W6, U11 TPD4EUSB30, U8 FSUSB42MUX, U9 USB2514B_Bi, Y1 Crystal_Small

Commit message: Checkpoint before CM5 connectivity migration
Parts:
- R29: value 36K -> 15k; JLCPCB part (none) -> C17475; Manufacturer part (none) -> 0805W8F1502T5E; Supplier https://www.digikey.ch/de/products/detail/stackpole-electro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 -> (none)
- U10: value AP2553W6 -> AP22653W6-7; Field4 Digikey -> (none); Field5 AP2553W6-7DICT-ND -> (none); JLCPCB part (none) -> C2158037; Supplier https://www.digikey.ch/en/products/detail/AP2553W6-7/AP2553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 -> (none)
Changed lines of the file:
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@@
 			)
 		)
-		(property "Value" "AP2553W6"
+		(property "Value" "AP22653W6-7"
 			(at 237.236 68.834 0)
 			(show_name no)
@@
 			)
 		)
-		(property "Datasheet" "https://www.diodes.com/assets/Datasheets/AP255x.pdf"
+		(property "Datasheet" "https://www.diodes.com/datasheet/download/AP22652_AP22653_AP22652A_AP22653A.pdf"
 			(at 241.3 81.28 0)
 			(hide yes)
@@
 			)
 		)
-		(property "Field4" "Digikey"
-			(at 237.49 74.93 0)
-			(hide yes)
-			(show_name no)
-			(do_not_autoplace no)
-			(effects
-				(font
-					(size 1.27 1.27)
-				)
-			)
-		)
-		(property "Field5" "AP2553W6-7DICT-ND"
-			(at 237.49 74.93 0)
-			(hide yes)
-			(show_name no)
-			(do_not_autoplace no)
-			(effects
-				(font
-					(size 1.27 1.27)
-				)
-			)
-		)
-		(property "Supplier" "https://www.digikey.ch/en/products/detail/AP2553W6-7/AP2553W6-7DICT-ND/3882112"
+		(property "JLCPCB part" "C2158037"
 			(at 237.49 74.93 0)
 			(hide yes)
@@
 			)
 		)
-		(property "Value" "36K"
+		(property "Value" "15k"
 			(at 249.936 82.296 0)
 			(show_name no)
@@
 			)
 		)
-		(property "Supplier" "https://www.digikey.ch/de/products/detail/stackpole-electronics-inc/RNCP0805FTD1K00/2240229"
+		(property "Supplier" ""
 			(at 254 78.74 0)
 			(hide yes)
+			(show_name no)
+			(do_not_autoplace no)
+			(effects
+				(font
+					(size 1.27 1.27)
+				)
+			)
+		)
+		(property "Manufacturer part" "0805W8F1502T5E"
+			(at 254 78.74 0)
+			(hide yes)
+			(show_name no)
+			(do_not_autoplace no)
+			(effects
+				(font
+					(size 1.27 1.27)
+				)
+			)
+		)
+		(property "JLCPCB part" "C17475"
+			(at 254 78.74 0)
+			(hide yes)

Commit message: Changed to CM5, removed unnecessary USB chips, Changing RP2024 to STM32.
Parts:
- removed C11, C25: 18p, Capacitor_SMD:C_0805_2012Metric, symbol Device:C_Small
- removed C44, C45: 10u, Capacitor_SMD:C_0805_2012Metric, symbol Device:C_Small
- removed C46, C47, C48, C49: 100n, Capacitor_SMD:C_0805_2012Metric, symbol Device:C_Small
- removed CM1: CM4, Pedalboard Library:Raspberry-Pi-4-Compute-Module, symbol pedalboard:CM4
- removed R22, R23: 2K2, Resistor_SMD:R_0805_2012Metric, symbol Device:R_Small
- removed R24: 12K, Resistor_SMD:R_0805_2012Metric, symbol Device:R_Small
- removed R25, R26, R27, R28: 36K, Resistor_SMD:R_0805_2012Metric, symbol Device:R_Small
- removed U8: FSUSB42MUX, Package_SO:TSSOP-10_3x3mm_P0.5mm, symbol Interface_USB:FSUSB42MUX
- removed U9: USB2514B_Bi, Package_DFN_QFN:QFN-36-1EP_6x6mm_P0.5mm_EP3.7x3.7mm, symbol Interface_USB:USB2514B_Bi
- removed Y1: Crystal_Small, Crystal:Crystal_SMD_5032-2Pin_5.0x3.2mm, symbol Device:Crystal_Small
- added CM2: ComputeModule5-CM5, CM5IO:Raspberry-Pi-5-Compute-Module, symbol CM5IO:ComputeModule5-CM5
- added J16: Debug, Connector_PinHeader_2.54mm:PinHeader_1x03_P2.54mm_Vertical, symbol Connector:Conn_01x03_Pin
Connections:
- net USB_OUT_N is gone; now on net USB_HOST_N: J10.2 (D-)
- net USB_OUT_P is gone; now on net USB_HOST_P: J10.3 (D+)
- net GND: now also C51.1, CM2.107 (GND), CM2.108 (GND), CM2.113 (GND), CM2.114 (GND), CM2.119 (GND), CM2.120 (GND), CM2.125 (GND), CM2.126 (GND), CM2.131 (GND), CM2.132 (GND), CM2.137 (GND), CM2.138 (GND), CM2.144 (GND), CM2.150 (GND), CM2.155 (GND), CM2.156 (GND), CM2.161 (GND), CM2.162 (GND), CM2.167 (GND), CM2.168 (GND), CM2.173 (GND), CM2.174 (GND), CM2.179 (GND), CM2.180 (GND), CM2.185 (GND), CM2.186 (GND), CM2.191 (GND), CM2.192 (GND), CM2.197 (GND), CM2.198 (GND), J16.1 (Pin_1); no longer C51.2
- net at J10.SH (Shield): now also C51.2; no longer C51.1
- net USB_HOST_VBUS_EN: now reaches U10.3 (EN)
- net USB_HOST_VBUS_EN: now also CM2.111 (VBUS_EN)
- net USB_HOST_P: now reaches U11.1 (D1+)
- net USB_HOST_P: now also CM2.163 (USB3-1-D_P)
- net USB_HOST_N: now reaches U11.2 (D1-)
- net USB_HOST_N: now also CM2.165 (USB3-1-D_N)
- net USB_D_N renamed USB_SERVICE_N
- net USB_SERVICE_N: now also CM2.103 (USB2_N); no longer U11.6 (NC)
- net USB_D_P renamed USB_SERVICE_P
- net USB_SERVICE_P: now also CM2.105 (USB2_P); no longer U11.7 (NC)
- net nOCS1: no longer names the net of U10.4 (nFault)
- new net CM5_UART_RX: J16.3 (Pin_3)
- new net CM5_UART_TX: J16.2 (Pin_2)
- new net USB_STM32_N: CM2.136 (USB3-0-D_N)
- new net USB_STM32_P: CM2.134 (USB3-0-D_P)
- no-connect marks 81 -> 9
Other:
- moved on the sheet: C38, C39, C40, C41, C42, C43, C50, C51, J10, J11, J9, R29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

Commit message: metadata
Parts:
- R30, R31: Supplier https://www.digikey.ch/de/products/detail/stackpole-electro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 -> (none)
Changed lines of the file:
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@@
 			)
 		)
-		(property "Supplier" "https://www.digikey.ch/de/products/detail/stackpole-electronics-inc/RMCF0805FT2K20/1760345"
+		(property "Supplier" ""
 			(at 157.48 30.48 0)
 			(hide yes)
@@
 			)
 		)
-		(property "Supplier" "https://www.digikey.ch/de/products/detail/stackpole-electronics-inc/RMCF0805FT2K20/1760345"
+		(property "Supplier" ""
 			(at 152.4 27.94 0)
 			(hide yes)

Commit message: a few edits
Connections:
- no-connect marks 9 -> 71
Changed lines of the file:
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@@
+	)
+	(no_connect
+		(at 104.14 68.58)
 	)
 	(no_connect
@@
 	)
 	(no_connect
+		(at 104.14 66.04)
+	)
+	(no_connect
+		(at 43.18 60.96)
+	)
+	(no_connect
 		(at 160.02 22.86)
 	)
 	(no_connect
+		(at 43.18 152.4)
+	)
+	(no_connect
+		(at 43.18 104.14)
+	)
+	(no_connect
 		(at 160.02 50.8)
 	)
 	(no_connect
+		(at 104.14 50.8)
+	)
+	(no_connect
 		(at 265.43 43.18)
 	)
 	(no_connect
+		(at 43.18 127)
+	)
+	(no_connect
+		(at 43.18 134.62)
+	)
+	(no_connect
+		(at 104.14 88.9)
+	)
+	(no_connect
+		(at 43.18 68.58)
+	)
+	(no_connect
+		(at 104.14 157.48)
+	)
+	(no_connect
+		(at 43.18 129.54)
+	)
+	(no_connect
+		(at 104.14 73.66)
+	)
+	(no_connect
 		(at 265.43 27.94)
 	)
 	(no_connect
+		(at 104.14 93.98)
+	)
+	(no_connect
+		(at 43.18 99.06)
+	)
+	(no_connect
+		(at 104.14 165.1)
+	)
+	(no_connect
+		(at 104.14 81.28)
+	)
+	(no_connect
+		(at 43.18 73.66)
+	)
+	(no_connect
+		(at 104.14 149.86)
+	)
+	(no_connect
+		(at 43.18 106.68)
+	)
+	(no_connect
+		(at 43.18 88.9)
+	)
+	(no_connect
+		(at 104.14 134.62)
+	)
+	(no_connect
+		(at 104.14 144.78)
+	)
+	(no_connect
+		(at 43.18 45.72)
+	)
+	(no_connect
+		(at 43.18 119.38)
+	)
+	(no_connect
+		(at 104.14 137.16)
+	)
+	(no_connect
+		(at 104.14 114.3)
+	)
+	(no_connect
+		(at 43.18 43.18)
+	)
+	(no_connect
+		(at 43.18 58.42)
+	)
+	(no_connect
+		(at 104.14 111.76)
+	)
+	(no_connect
+		(at 43.18 96.52)
+	)
+	(no_connect
+		(at 104.14 60.96)
+	)
+	(no_connect
+		(at 43.18 66.04)
+	)
+	(no_connect
+		(at 43.18 144.78)
+	)
+	(no_connect
+		(at 104.14 76.2)
+	)
+	(no_connect
+		(at 104.14 83.82)
+	)
+	(no_connect
+		(at 104.14 129.54)
+	)
+	(no_connect
+		(at 43.18 50.8)
+	)
+	(no_connect
 		(at 240.03 27.94)
 	)
@@
 	)
 	(no_connect
+		(at 43.18 40.64)
+	)
+	(no_connect
+		(at 43.18 53.34)
+	)
+	(no_connect
+		(at 104.14 142.24)
+	)
+	(no_connect
+		(at 104.14 106.68)
+	)
+	(no_connect
+		(at 104.14 127)
+	)
+	(no_connect
 		(at 215.9 81.28)
 	)
+	(no_connect
+		(at 104.14 58.42)
+	)
+	(no_connect
+		(at 104.14 99.06)
+	)
+	(no_connect
+		(at 43.18 160.02)
+	)
+	(no_connect
+		(at 104.14 91.44)
+	)
+	(no_connect
+		(at 43.18 137.16)
+	)
+	(no_connect
+		(at 43.18 76.2)
+	)
+	(no_connect
+		(at 43.18 149.86)
+	)
+	(no_connect
+		(at 43.18 111.76)
+	)
+	(no_connect
+		(at 104.14 152.4)
+	)
+	(no_connect
+		(at 43.18 121.92)
+	)
+	(no_connect
+		(at 104.14 160.02)
+	)
+	(no_connect
+		(at 43.18 114.3)
+	)
+	(no_connect
+		(at 43.18 157.48)
+	)
+	(no_connect
+		(at 104.14 101.6)
+	)
+	(no_connect
+		(at 104.14 104.14)
+	)
+	(no_connect
+		(at 43.18 165.1)
+	)
+	(no_connect
+		(at 104.14 96.52)
+	)
+	(no_connect
+		(at 43.18 142.24)
+	)
+	(no_connect
+		(at 43.18 91.44)
+	)
 	(wire

Commit message: Standardize values.
Parts:
- C38, C39, C40, C41, C42: value 10u -> 10uF
- C43: value 100u -> 100uF
- C50, C51: value 1n -> 1nF
- R30, R31: value 5K1 -> 5k1
Changed lines of the file:
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@@
 			)
 		)
-		(property "Value" "10u"
+		(property "Value" "10uF"
 			(at 238.76 81.788 0)
 			(show_name no)
@@
 			)
 		)
-		(property "Value" "10u"
+		(property "Value" "10uF"
 			(at 190.881 76.073 0)
 			(show_name no)
@@
 			)
 		)
-		(property "Value" "10u"
+		(property "Value" "10uF"
 			(at 243.84 81.788 0)
 			(show_name no)
@@
 			)
 		)
-		(property "Value" "10u"
+		(property "Value" "10uF"
 			(at 248.92 82.042 0)
 			(show_name no)
@@
 			)
 		)
-		(property "Value" "1n"
+		(property "Value" "1nF"
 			(at 180.34 63.5 90)
 			(show_name no)
@@
 			)
 		)
-		(property "Value" "5K1"
+		(property "Value" "5k1"
 			(at 157.734 34.036 90)
 			(show_name no)
@@
 			)
 		)
-		(property "Value" "5K1"
+		(property "Value" "5k1"
 			(at 152.4 26.162 90)
 			(show_name no)
@@
 			)
 		)
-		(property "Value" "10u"
+		(property "Value" "10uF"
 			(at 233.68 82.296 0)
 			(show_name no)
@@
 			)
 		)
-		(property "Value" "1n"
+		(property "Value" "1nF"
 			(at 218.44 50.038 0)
 			(show_name no)
@@
 			)
 		)
-		(property "Value" "100u"
+		(property "Value" "100uF"
 			(at 230.632 82.296 0)
 			(show_name no)

Commit message: more meta
Parts:
- added C16: 100nF, Capacitor_SMD:C_0603_1608Metric, symbol Device:C_Small
Connections:
- net +5VP: now also C16.1
- net GND: now also C16.2
Other:
- moved on the sheet: C40, C41, C42
Changed lines of the file:
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@@
 	)
 	(junction
-		(at 247.65 76.2)
+		(at 250.19 76.2)
 		(diameter 0)
 		(color 0 0 0 0)
@@
 	)
 	(junction
-		(at 242.57 76.2)
+		(at 243.84 76.2)
 		(diameter 0)
 		(color 0 0 0 0)
@@
 	)
 	(junction
-		(at 247.65 86.36)
+		(at 250.19 86.36)
 		(diameter 0)
 		(color 0 0 0 0)
@@
 	)
 	(junction
-		(at 242.57 86.36)
+		(at 243.84 86.36)
 		(diameter 0)
 		(color 0 0 0 0)
@@
 	(wire
 		(pts
-			(xy 242.57 76.2) (xy 242.57 77.47)
+			(xy 243.84 76.2) (xy 243.84 77.47)
 		)
 		(stroke
@@
 	(wire
 		(pts
+			(xy 182.88 78.74) (xy 187.96 78.74)
+		)
+		(stroke
+			(width 0)
+			(type default)
+		)
+	)
+	(wire
+		(pts
 			(xy 154.94 27.94) (xy 160.02 27.94)
 		)
@@
 	(wire
 		(pts
-			(xy 242.57 76.2) (xy 247.65 76.2)
-		)
-		(stroke
-			(width 0)
-			(type default)
-		)
-	)
-	(wire
-		(pts
 			(xy 106.68 63.5) (xy 106.68 55.88)
 		)
@@
 	(wire
 		(pts
-			(xy 247.65 76.2) (xy 252.73 76.2)
-		)
-		(stroke
-			(width 0)
-			(type default)
-		)
-	)
-	(wire
-		(pts
 			(xy 231.14 76.2) (xy 237.49 76.2)
 		)
@@
 	(wire
 		(pts
-			(xy 247.65 76.2) (xy 247.65 77.47)
+			(xy 250.19 76.2) (xy 250.19 77.47)
 		)
 		(stroke
@@
 	(wire
 		(pts
-			(xy 247.65 86.36) (xy 252.73 86.36)
+			(xy 182.88 77.47) (xy 182.88 78.74)
 		)
 		(stroke
@@
 	(wire
 		(pts
-			(xy 237.49 86.36) (xy 242.57 86.36)
+			(xy 237.49 86.36) (xy 256.54 86.36)
 		)
 		(stroke
@@
 	(wire
 		(pts
-			(xy 252.73 76.2) (xy 252.73 77.47)
+			(xy 256.54 76.2) (xy 256.54 77.47)
 		)
 		(stroke
@@
 	(wire
 		(pts
+			(xy 182.88 72.39) (xy 187.96 72.39)
+		)
+		(stroke
+			(width 0)
+			(type default)
+		)
+	)
+	(wire
+		(pts
 			(xy 106.68 55.88) (xy 104.14 55.88)
 		)
@@
 	(wire
 		(pts
-			(xy 247.65 82.55) (xy 247.65 86.36)
+			(xy 250.19 82.55) (xy 250.19 86.36)
 		)
 		(stroke
@@
 	(wire
 		(pts
-			(xy 237.49 76.2) (xy 242.57 76.2)
+			(xy 237.49 76.2) (xy 256.54 76.2)
 		)
 		(stroke
@@
 	(wire
 		(pts
-			(xy 252.73 82.55) (xy 252.73 86.36)
+			(xy 256.54 82.55) (xy 256.54 86.36)
 		)
 		(stroke
@@
 	(wire
 		(pts
-			(xy 242.57 82.55) (xy 242.57 86.36)
+			(xy 243.84 82.55) (xy 243.84 86.36)
 		)
 		(stroke
@@
 	(wire
 		(pts
-			(xy 242.57 86.36) (xy 247.65 86.36)
-		)
-		(stroke
-			(width 0)
-			(type default)
-		)
-	)
-	(wire
-		(pts
 			(xy 227.33 38.1) (xy 240.03 38.1)
 		)
@@
 	(symbol
 		(lib_id "Device:C_Small")
-		(at 242.57 80.01 0)
+		(at 243.84 80.01 0)
 		(unit 1)
 		(body_style 1)
@@
 		(dnp no)
 		(property "Reference" "C40"
-			(at 238.506 78.486 0)
+			(at 239.776 78.486 0)
 			(show_name no)
 			(do_not_autoplace no)
@@
 		)
 		(property "Value" "10uF"
-			(at 238.76 81.788 0)
+			(at 238.76 82.296 0)
 			(show_name no)
 			(do_not_autoplace no)
@@
 		)
 		(property "Footprint" "Capacitor_SMD:C_0805_2012Metric"
-			(at 243.5352 83.82 0)
+			(at 244.8052 83.82 0)
 			(hide yes)
 			(show_name no)
@@
 		)
 		(property "Datasheet" "https://www.samsungsem.com/resources/file/global/support/product_catalog/MLCC.pdf"
-			(at 242.57 80.01 0)
+			(at 243.84 80.01 0)
 			(hide yes)
 			(show_name no)
@@
 		)
 		(property "Description" ""
-			(at 242.57 80.01 0)
+			(at 243.84 80.01 0)
 			(hide yes)
 			(show_name no)
@@
 		)
 		(property "Notes" "10% or 20% 35V Ceramic Capacitor X6S 0805 (2012 Metric)"
-			(at 242.57 80.01 0)
+			(at 243.84 80.01 0)
 			(hide yes)
 			(show_name no)
@@
 		)
 		(property "Supplier" "https://www.digikey.ch/de/products/detail/samsung-electro-mechanics/CL21X106KAYNNNE/5961182"
-			(at 242.57 80.01 0)
+			(at 243.84 80.01 0)
 			(hide yes)
 			(show_name no)
@@
 	(symbol
 		(lib_id "Device:C_Small")
-		(at 247.65 80.01 0)
+		(at 250.19 80.01 0)
 		(unit 1)
 		(body_style 1)
@@
 		(dnp no)
 		(property "Reference" "C41"
-			(at 243.84 78.232 0)
+			(at 246.38 78.232 0)
 			(show_name no)
 			(do_not_autoplace no)
@@
 		)
 		(property "Value" "10uF"
-			(at 243.84 81.788 0)
+			(at 245.11 82.296 0)
 			(show_name no)
 			(do_not_autoplace no)
@@
 		)
 		(property "Footprint" "Capacitor_SMD:C_0805_2012Metric"
-			(at 248.6152 83.82 0)
+			(at 251.1552 83.82 0)
 			(hide yes)
 			(show_name no)
@@
 		)
 		(property "Datasheet" "https://www.samsungsem.com/resources/file/global/support/product_catalog/MLCC.pdf"
-			(at 247.65 80.01 0)
+			(at 250.19 80.01 0)
 			(hide yes)
 			(show_name no)
@@
 		)
 		(property "Description" ""
-			(at 247.65 80.01 0)
+			(at 250.19 80.01 0)
 			(hide yes)
 			(show_name no)
@@
 		)
 		(property "Notes" "10% or 20% 35V Ceramic Capacitor X6S 0805 (2012 Metric)"
-			(at 247.65 80.01 0)
+			(at 250.19 80.01 0)
 			(hide yes)
 			(show_name no)
@@
 		)
 		(property "Supplier" "https://www.digikey.ch/de/products/detail/samsung-electro-mechanics/CL21X106KAYNNNE/5961182"
-			(at 247.65 80.01 0)
+			(at 250.19 80.01 0)
 			(hide yes)
 			(show_name no)
@@
 	)
 	(symbol
+		(lib_id "Device:C_Small")
+		(at 182.88 74.93 0)
+		(unit 1)
+		(body_style 1)
+		(exclude_from_sim no)
+		(in_bom yes)
+		(on_board yes)
+		(in_pos_files yes)
+		(dnp no)
+		(property "Reference" "C16"
+			(at 177.038 73.406 0)
+			(show_name no)
+			(do_not_autoplace no)
+			(effects
+				(font
+					(size 1.27 1.27)
+				)
+				(justify left)
+			)
+		)
+		(property "Value" "100nF"
+			(at 176.53 76.708 0)
+			(show_name no)
+			(do_not_autoplace no)
+			(effects
+				(font
+					(size 1.27 1.27)
+				)
+				(justify left)
+			)
+		)
+		(property "Footprint" "Capacitor_SMD:C_0603_1608Metric"
+			(at 183.8452 78.74 0)
+			(hide yes)
+			(show_name no)
+			(do_not_autoplace no)
+			(effects
+				(font
+					(size 1.27 1.27)
+				)
+			)
+		)
+		(property "Datasheet" ""
+			(at 182.88 74.93 0)
+			(hide yes)
+			(show_name no)
+			(do_not_autoplace no)
+			(effects
+				(font
+					(size 1.27 1.27)
+				)
+			)
+		)
+		(property "Description" ""
+			(at 182.88 74.93 0)
+			(hide yes)
+			(show_name no)
+			(do_not_autoplace no)
+			(effects
+				(font
+					(size 1.27 1.27)
+				)
+			)
+		)
+		(property "Manufacturer" ""
+			(at 182.88 74.93 0)
+			(hide yes)
+			(show_name no)
+			(do_not_autoplace no)
+			(effects
+				(font
+					(size 1.27 1.27)
+				)
+			)
+		)
+		(property "Manufacturer part" ""
+			(at 182.88 74.93 0)
+			(hide yes)
+			(show_name no)
+			(do_not_autoplace no)
+			(effects
+				(font
+					(size 1.27 1.27)
+				)
+			)
+		)
+		(property "JLCPCB part" "C14663"
+			(at 182.88 74.93 0)
+			(hide yes)
+			(show_name no)
+			(do_not_autoplace no)
+			(effects
+				(font
+					(size 1.27 1.27)
+				)
+			)
+		)
+		(pin "1"
+		)
+		(pin "2"
+		)
+		(instances
+			(project "pedalboard-hw"
+				(path "/df521c2a-9827-4355-b809-366f4b88d5d7/e8ab7a61-8d57-4690-876b-f6a417060d03"
+					(reference "C16")
+					(unit 1)
+				)
+			)
+		)
+	)
+	(symbol
 		(lib_id "power:GND")
 		(at 231.14 86.36 0)
@@
 	(symbol
 		(lib_id "Device:C_Small")
-		(at 252.73 80.01 0)
+		(at 256.54 80.01 0)
 		(unit 1)
 		(body_style 1)
@@
 		(dnp no)
 		(property "Reference" "C42"
-			(at 248.666 78.486 0)
+			(at 252.476 78.486 0)
 			(show_name no)
 			(do_not_autoplace no)
@@
 		)
 		(property "Value" "10uF"
-			(at 248.92 82.042 0)
+			(at 251.46 82.042 0)
 			(show_name no)
 			(do_not_autoplace no)
@@
 		)
 		(property "Footprint" "Capacitor_SMD:C_0805_2012Metric"
-			(at 253.6952 83.82 0)
+			(at 257.5052 83.82 0)
 			(hide yes)
 			(show_name no)
@@
 		)
 		(property "Datasheet" "https://www.samsungsem.com/resources/file/global/support/product_catalog/MLCC.pdf"
-			(at 252.73 80.01 0)
+			(at 256.54 80.01 0)
 			(hide yes)
 			(show_name no)
@@
 		)
 		(property "Description" ""
-			(at 252.73 80.01 0)
+			(at 256.54 80.01 0)
 			(hide yes)
 			(show_name no)
@@
 		)
 		(property "Notes" "10% or 20% 35V Ceramic Capacitor X6S 0805 (2012 Metric)"
-			(at 252.73 80.01 0)
+			(at 256.54 80.01 0)
 			(hide yes)
 			(show_name no)
@@
 		)
 		(property "Supplier" "https://www.digikey.ch/de/products/detail/samsung-electro-mechanics/CL21X106KAYNNNE/5961182"
-			(at 252.73 80.01 0)
+			(at 256.54 80.01 0)
 			(hide yes)
 			(show_name no)
@@
 		)
 		(property "Value" "10uF"
-			(at 233.68 82.296 0)
+			(at 232.41 82.55 0)
 			(show_name no)
 			(do_not_autoplace no)
