File: connect.kicad_sch (KiCad schematic)
At the start: 19 parts, among them J10 USB_A, J11 Conn_01x02, J16 Debug, J9 USB_OTG, U10 AP22653W6-7, U11 TPD4EUSB30

Commit message: U10 components metadata
Parts:
- removed C41, C42: 10uF, Capacitor_SMD:C_0805_2012Metric, symbol Device:C_Small
- C38, C39, C40: JLCPCB part (none) -> C15850; Manufacturer (none) -> Samsung Electro-Mechanics; Manufacturer part (none) -> CL21A106KAYNNNE; Notes 10% or 20% 35V Ceramic Capacitor X6S 0805 (2012 Metric) -> 25V, X5R, ±10%, JLCPCB Basic; Supplier https://www.digikey.ch/de/products/detail/samsung-electro-m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 -> (none)
- C43: JLCPCB part (none) -> C189619; Manufacturer (none) -> Panasonic Industry; Manufacturer part (none) -> EEF-CX0J101R; Notes Capacitor, SP-Cap, 100u, 6.3V, 15mR ESR -> 6.3V aluminum-polymer, ±20%, 15mΩ ESR. Required USB bulk ca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; Supplier https://www.digikey.ch/de/products/detail/panasonic-electro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 -> (none)
- R29: Manufacturer (none) -> UNI-ROYAL
- U10: value AP22653W6-7 -> AP22653; Manufacturer (none) -> Diodes Incorporated; Manufacturer part (none) -> AP22653W6-7; Notes (none) -> Extended part
Other:
- moved on the sheet: C43, R29

Commit message: Updated various metadata
Parts:
- removed C51: 1nF, Capacitor_SMD:C_0805_2012Metric, symbol Device:C_Small
- removed U11: TPD4EUSB30, Package_SON:USON-10_2.5x1.0mm_P0.5mm, symbol Power_Protection:TPD4EUSB30
- added R53: 1M, Resistor_SMD:R_0603_1608Metric, symbol Device:R_Small
- added U11, U16: TPD2E2U06DCK, Package_TO_SOT_SMD:SOT-323_SC-70, symbol Power_Protection:TPD2E2U06DCK
- C16: Manufacturer (none) -> Yageo; Manufacturer part (none) -> CC0603KRX7R9BB104; Notes (none) -> 100nF, 50V, X7R, ±10%. U10 input bypass. place close to U10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
- C50: footprint Capacitor_SMD:C_0805_2012Metric -> Capacitor_SMD:C_1206_3216Metric; JLCPCB part (none) -> C521240; Manufacturer (none) -> Murata; Manufacturer part (none) -> GRM31C5C3A102JWA3L; Notes 1000 pF, 50 V -> 1kV C0G; chassis-to-signal-ground HF/ESD bond; Supplier https://www.digikey.ch/de/products/detail/samsung-electro-m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 -> (none)
- CM2: value ComputeModule5-CM5 -> Raspberry Pi CM5; Field4 Amphenol -> (none); Field5 2x 10164227-1001A1RLF -> (none); Manufacturer (none) -> Raspberry Pi ltd; Notes (none) -> CM5 module supplied separately. Carrier requires 2x Ampheno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
- J10: value USB_A -> USB-A HOST; Manufacturer (none) -> Molex; Manufacturer part (none) -> 67643-3910; Notes (none) -> USB 2.0 host connector. Through-hole, intended for manual f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
- J11: value Conn_01x02 -> CM5 BOOT; now not fitted
- J16: value Debug -> CM5 UART DEBUG
- J9: value USB_OTG -> USB-C SERVICE; JLCPCB part (none) -> C3025063; Manufacturer (none) -> Global Connector Technology; Manufacturer part (none) -> USB4105-GF-A-060; Notes (none) -> Self-powered USB 2.0 service and flashing port. VBUS intent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
- R29: Notes (none) -> 1% - sets U10 current limit to approximately 1.74A typical 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
- R30, R31: JLCPCB part (none) -> C25905; Manufacturer (none) -> UNI-ROYAL; Manufacturer part (none) -> 0402WGF5101TCE
- U10: Notes Extended part -> USB-A active-high current-limited load switch. Constant-cur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
Connections:
- net GND: now also R53.2, U11.3, U16.3
- net USB_HOST_N: now also U11.2
- net USB_HOST_P: now also U11.1
- net USB_SERVICE_N: now also U16.2
- net USB_SERVICE_P: now also U16.1
- net CHASSIS: now reaches J10.SH (Shield)
- net CHASSIS: now also C50.2, J9.SH (SHIELD), R53.1
- no-connect marks 71 -> 67
Other:
- note added: "Fit manually if required. Install jumper before power-up to force CM5 USB boot mode."
- note added: "Optional 3.3V CM5 debug UART. Pin order: GND, TX, RX."
- note added: "PCB placement: C16 and C38 close to U10 IN/GND. R29 close to ILIM/GND. C39 or C40 close to OUT/GND. C43 near J10 VBUS."
- note added: "USB-host protection"
- note added: "USB-service protection"
- moved on the sheet: C16, C38, C39, C40, C43, C50, J10, J16, J9, R29, R30, U10

Commit message: Moving to seperate ui board using ESP32
Parts:
- added J21: UI LINK 2x5, Pedalboard Library:J_Wurth_WR-BHD_61201021621, symbol Connector_Generic:Conn_02x05_Odd_Even
- J9: Notes Self-powered USB 2.0 service and flashing port. VBUS intent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 -> Self-powered CM5 USB 2.0 service port for rpiboot flashing,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
Connections:
- net +5VP: now also J21.1 (Pin_1), J21.3 (Pin_3)
- net CM5_UART_RX: now also J21.7 (Pin_7); no longer J16.3 (Pin_3)
- net CM5_UART_TX: now also J21.5 (Pin_5); no longer J16.2 (Pin_2)
- net GND: now also J21.2 (Pin_2), J21.4 (Pin_4), J21.6 (Pin_6), J21.8 (Pin_8)
- net USB_STM32_N: no longer names the net of CM2.136 (USB3-0-D_N)
- net USB_STM32_P: no longer names the net of CM2.134 (USB3-0-D_P)
- new net CM5_DEBUG_UART_RX: J16.3 (Pin_3)
- new net CM5_DEBUG_UART_TX: J16.2 (Pin_2)
- new net ESP_BOOT: J21.10 (Pin_10)
- new net ESP_RESET: J21.9 (Pin_9)
- no-connect marks 67 -> 69

Commit message: update 3d model of J21
Parts:
- J21: now not fitted
Connections:
- net CM5_UART_RX renamed UI_UART_RX
- net CM5_UART_TX renamed UI_UART_TX
Changed lines of the file:
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@@
 		)
 	)
-	(global_label "CM5_UART_TX"
+	(global_label "UI_UART_TX"
 		(shape input)
 		(at 137.16 172.72 180)
@@
 		)
 		(property "Intersheetrefs" "${INTERSHEET_REFS}"
-			(at 121.4749 172.72 0)
+			(at 123.4705 172.72 0)
 			(hide yes)
 			(show_name no)
@@
 		)
 	)
-	(global_label "CM5_UART_RX"
+	(global_label "UI_UART_RX"
 		(shape input)
 		(at 137.16 175.26 180)
@@
 		)
 		(property "Intersheetrefs" "${INTERSHEET_REFS}"
-			(at 121.1725 175.26 0)
+			(at 123.1681 175.26 0)
 			(hide yes)
 			(show_name no)
@@
 		(on_board yes)
 		(in_pos_files yes)
-		(dnp no)
+		(dnp yes)
 		(fields_autoplaced yes)
 		(property "Reference" "J21"

Commit message: initital pcb work
Connections:
- net USB_SERVICE_VBUS_UNUSED: now reaches J9.A4 (VBUS), J9.A9 (VBUS), J9.B4 (VBUS), J9.B9 (VBUS)
- no-connect marks 69 -> 68
Other:
- moved on the sheet: C50, J10, J9, R30, R31, R53

Commit message: 5V power to CM5
Connections:
- net +5VP: now also J21.10 (Pin_10); no longer J21.3 (Pin_3)
- net ESP_BOOT: now also J21.8 (Pin_8); no longer J21.10 (Pin_10)
- net ESP_RESET: now also J21.3 (Pin_3); no longer J21.9 (Pin_9)
- net GND: now also J21.7 (Pin_7), J21.9 (Pin_9); no longer J21.6 (Pin_6), J21.8 (Pin_8)
- net UI_UART_RX: now also J21.5 (Pin_5); no longer J21.7 (Pin_7)
- net UI_UART_TX: now also J21.6 (Pin_6); no longer J21.5 (Pin_5)

Commit message: more psu
Parts:
- C43: footprint Capacitor_Tantalum_SMD:CP_EIA-7343-31_Kemet-D -> Capacitor_THT:CP_Radial_D8.0mm_P3.50mm; symbol Device:C_Polarized -> Device:C_Small_US; JLCPCB part C189619 -> (none); Manufacturer Panasonic Industry -> Nichicon; Manufacturer part EEF-CX0J101R -> RR71C101MDN1; Notes 6.3V aluminum-polymer, ±20%, 15mΩ ESR. Required USB bulk ca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 -> 100uF 16V aluminum-polymer, ±20%, 7mΩ ESR; USB VBUS bulk ca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
- J21: now fitted
Changed lines of the file:
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@@
 	)
 	(junction
+		(at 254 82.55)
+		(diameter 0)
+		(color 0 0 0 0)
+	)
+	(junction
 		(at 40.64 139.7)
 		(diameter 0)
@@
 	)
 	(junction
-		(at 254 82.55)
-		(diameter 0)
-		(color 0 0 0 0)
-	)
-	(junction
 		(at 106.68 86.36)
 		(diameter 0)
@@
 	(wire
 		(pts
-			(xy 254 82.55) (xy 269.24 82.55)
-		)
-		(stroke
-			(width 0)
-			(type default)
-		)
-	)
-	(wire
-		(pts
 			(xy 166.37 45.72) (xy 166.37 48.26)
 		)
@@
 	(wire
 		(pts
+			(xy 254 82.55) (xy 269.24 82.55)
+		)
+		(stroke
+			(width 0)
+			(type default)
+		)
+	)
+	(wire
+		(pts
 			(xy 175.26 72.39) (xy 181.61 72.39)
 		)
@@
 	(wire
 		(pts
+			(xy 254 82.55) (xy 254 83.82)
+		)
+		(stroke
+			(width 0)
+			(type default)
+		)
+	)
+	(wire
+		(pts
 			(xy 208.28 86.36) (xy 208.28 85.09)
 		)
@@
 	(wire
 		(pts
-			(xy 254 90.17) (xy 254 92.71)
+			(xy 254 88.9) (xy 254 92.71)
 		)
 		(stroke
@@
 	)
 	(symbol
-		(lib_id "Device:C_Polarized")
+		(lib_id "Device:C_Small_US")
 		(at 254 86.36 0)
 		(mirror y)
@@
 			)
 		)
-		(property "Footprint" "Capacitor_Tantalum_SMD:CP_EIA-7343-31_Kemet-D"
-			(at 253.0348 90.17 0)
+		(property "Footprint" "Capacitor_THT:CP_Radial_D8.0mm_P3.50mm"
+			(at 254 86.36 0)
 			(hide yes)
 			(show_name no)
@@
 			)
 		)
-		(property "Datasheet" "https://industrial.panasonic.com/cdbs/www-data/pdf/ABE0000/ABE0000C49.pdf"
+		(property "Datasheet" "https://www.nichicon.com/getmedia/36a40bf2-5311-4e83-96af-12226794ab9f/e-rr7.pdf"
 			(at 254 86.36 0)
 			(hide yes)
@@
 			)
 		)
-		(property "Description" ""
+		(property "Description" "capacitor, small US symbol"
 			(at 254 86.36 0)
 			(hide yes)
@@
 			)
 		)
-		(property "Notes" "6.3V aluminum-polymer, ±20%, 15mΩ ESR. Required USB bulk capacitor"
+		(property "Notes" "100uF 16V aluminum-polymer, ±20%, 7mΩ ESR; USB VBUS bulk capacitor; hand solder"
 			(at 254 86.36 0)
 			(hide yes)
@@
 			)
 		)
-		(property "Manufacturer" "Panasonic Industry"
+		(property "Manufacturer" "Nichicon"
 			(at 254 86.36 0)
 			(hide yes)
@@
 			)
 		)
-		(property "Manufacturer part" "EEF-CX0J101R"
+		(property "Manufacturer part" "RR71C101MDN1"
 			(at 254 86.36 0)
 			(hide yes)
@@
 			)
 		)
-		(property "JLCPCB part" "C189619"
+		(property "JLCPCB part" ""
 			(at 254 86.36 0)
 			(hide yes)
@@
 		(on_board yes)
 		(in_pos_files yes)
-		(dnp yes)
+		(dnp no)
 		(fields_autoplaced yes)
 		(property "Reference" "J21"

Commit message: various fixes.
Parts:
- J11: now fitted
Changed lines of the file:
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@@
 		(on_board yes)
 		(in_pos_files yes)
-		(dnp yes)
+		(dnp no)
 		(fields_autoplaced yes)
 		(property "Reference" "J11"
