File: connect.kicad_sch (KiCad schematic)
At the start: 19 parts, among them J10 USB-A HOST, J11 CM5 BOOT, J16 CM5 UART DEBUG, J21 UI LINK 2x5, J9 USB-C SERVICE, U10 AP22653, U11 TPD2E2U06DCK, U16 TPD2E2U06DCK

Commit message: Updated parts to available jlcpcb parts.
Parts:
- J9: JLCPCB part C3025063 -> C5184243; Manufacturer part USB4105-GF-A-060 -> USB4105-GF-A-120
- U11, U16: value TPD2E2U06DCK -> TPD2E2U06QDCKRQ1; JLCPCB part C1855726 -> C915089; Manufacturer part TPD2E2U06DCKR -> TPD2E2U06QDCKRQ1
Changed lines of the file:
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@@
 			)
 		)
-		(property "Value" "TPD2E2U06DCK"
+		(property "Value" "TPD2E2U06QDCKRQ1"
 			(at 265.43 64.7699 0)
 			(show_name no)
@@
 			)
 		)
-		(property "Datasheet" "https://www.ti.com/lit/ds/symlink/tpd2e2u06.pdf"
+		(property "Datasheet" "https://www.ti.com/lit/ds/symlink/tpd2e2u06-q1.pdf"
 			(at 256.54 58.42 0)
 			(hide yes)
@@
 			)
 		)
-		(property "Manufacturer part" "TPD2E2U06DCKR"
+		(property "Manufacturer part" "TPD2E2U06QDCKRQ1"
 			(at 261.62 63.5 0)
 			(hide yes)
@@
 			)
 		)
-		(property "JLCPCB part" "C1855726"
+		(property "JLCPCB part" "C915089"
 			(at 261.62 63.5 0)
 			(hide yes)
@@
 					(reference "CM2")
 					(unit 2)
+					(variant
+						(name "JLCPCB-SMT")
+						(in_bom no)
+						(in_pos_files no)
+					)
 				)
 			)
@@
 			)
 		)
-		(property "Value" "TPD2E2U06DCK"
+		(property "Value" "TPD2E2U06QDCKRQ1"
 			(at 262.89 34.2899 0)
 			(show_name no)
@@
 			)
 		)
-		(property "Datasheet" "https://www.ti.com/lit/ds/symlink/tpd2e2u06.pdf"
+		(property "Datasheet" "https://www.ti.com/lit/ds/symlink/tpd2e2u06-q1.pdf"
 			(at 254 27.94 0)
 			(hide yes)
@@
 			)
 		)
-		(property "Manufacturer part" "TPD2E2U06DCKR"
+		(property "Manufacturer part" "TPD2E2U06QDCKRQ1"
 			(at 259.08 33.02 0)
 			(hide yes)
@@
 			)
 		)
-		(property "JLCPCB part" "C1855726"
+		(property "JLCPCB part" "C915089"
 			(at 259.08 33.02 0)
 			(hide yes)
@@
 			)
 		)
-		(property "Manufacturer part" "USB4105-GF-A-060"
+		(property "Manufacturer part" "USB4105-GF-A-120"
 			(at 181.61 48.26 0)
 			(hide yes)
@@
 			)
 		)
-		(property "JLCPCB part" "C3025063"
+		(property "JLCPCB part" "C5184243"
 			(at 181.61 48.26 0)
 			(hide yes)
