File: psu.kicad_sch (KiCad schematic)
At the start: 44 parts, among them J6 Screw_Terminal_01x02, J7 Barrel_Jack_MountingPin, Q1 FDS4435BZ, U13 LT3045xMSE, U5 NCP1117-3.3_SOT223, U6 AP64501SP-13

Commit message: Supply work on TAC5212
Parts:
- added C71, C72: 1u, Capacitor_SMD:C_0805_2012Metric, symbol Device:C_Small
- added U15: TPS7A20xxxDBV, Package_TO_SOT_SMD:SOT-23-5, symbol Regulator_Linear:TPS7A20xxxDBV
Connections:
- net +5VP: now also C71.1, U15.1 (IN), U15.3 (EN)
- net GND: now also C71.2, C72.2, U15.2 (GND)
- new net 3V3_CODEC: C72.1, U15.5 (OUT)

Commit message: Checkpoint before CM5 connectivity migration
Parts:
- removed C10, C7, C8, C9: 10u, Capacitor_SMD:C_0805_2012Metric, symbol Device:C_Small
- removed C29, C34: 1n, Capacitor_SMD:C_0805_2012Metric, symbol Device:C_Small
- removed C31: 1.2n, Capacitor_SMD:C_0805_2012Metric, symbol Device:C_Small
- removed C33: 100u, Capacitor_Tantalum_SMD:CP_EIA-7343-31_Kemet-D, symbol Device:C_Polarized
- removed C35: 100n, Capacitor_SMD:C_0805_2012Metric, symbol Device:C_Small
- removed U5: NCP1117-3.3_SOT223, Package_TO_SOT_SMD:SOT-223-3_TabPin2, symbol Regulator_Linear:NCP1117-3.3_SOT223
- removed U6: AP64501SP-13, Pedalboard Library:SOIC-8-1EP_3.9x4.9mm_P1.27mm_EP2.95x4.9mm_Mask2.71x3.4mm_ThermalVias, symbol pedalboard:AP64351
- added U5: TPS7A2033PDBVR, Package_TO_SOT_SMD:SOT-23-5, symbol Regulator_Linear:TPS7A20xxxDBV
- added U6: TPS56637RPAR, Pedalboard Library:RPA0010A, symbol TPS56637:TPS56637RPAR
- C2, C3, C4, C5: value 10u -> 10uF; JLCPCB part (none) -> C440198; Manufacturer part (none) -> GRM21BR61H106KE43L; Notes 10% or 20% 35V Ceramic Capacitor X6S 0805 (2012 Metric) -> (none); Supplier https://www.digikey.ch/de/products/detail/samsung-electro-m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 -> (none)
- C24, C27, C28, C32, C36, C37: value 10u -> 10uF; JLCPCB part (none) -> C15850; Manufacturer part (none) -> CL21A106KAYNNNE; Notes 10% or 20% 35V Ceramic Capacitor X6S 0805 (2012 Metric) -> (none); Supplier https://www.digikey.ch/de/products/detail/samsung-electro-m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 -> (none)
- C30: value 100n -> 100nF; Digikey 1276-1180-1-ND -> (none); JLCPCB part (none) -> C49678; Manufacturer part (none) -> CC0805KRX7R9BB104; Notes 10% 16V Ceramic Capacitor X7R -> (none); Supplier https://www.digikey.ch/de/products/detail/samsung-electro-m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 -> (none)
- C53: value 4.7u -> 4.7uF; JLCPCB part (none) -> C1779; Manufacturer part (none) -> CL21A475KAQNNNE; Notes JLCPCB C1779 -> (none)
- C54: value 10u -> 22uF; footprint Capacitor_SMD:C_0805_2012Metric -> Capacitor_SMD:C_1206_3216Metric; JLCPCB part (none) -> C12891; Manufacturer part (none) -> CL31A226KAHNNNE; Notes 10% or 20% 35V Ceramic Capacitor X6S 0805 (2012 Metric) -> (none); Supplier https://www.digikey.ch/de/products/detail/samsung-electro-m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 -> (none)
- C55: value 4.7u -> 10uF; JLCPCB part (none) -> C440198; Manufacturer part (none) -> GRM21BR61H106KE43L; Notes JLCPCB C1779 -> (none)
- C6: value 10u -> 100nF; JLCPCB part (none) -> C49678; Manufacturer part (none) -> CC0805KRX7R9BB104; Notes 10% or 20% 35V Ceramic Capacitor X6S 0805 (2012 Metric) -> (none); Supplier https://www.digikey.ch/de/products/detail/samsung-electro-m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 -> (none)
- F1: value Polyfuse 1.8A -> PTC 4A 15V; footprint Fuse:Fuse_1812_4532Metric -> Fuse:Fuse_2920_7451Metric; JLCPCB part (none) -> C720182; Manufacturer part (none) -> 2920L400/15MR; Supplier https://www.digikey.ch/de/products/detail/littelfuse-inc/18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 -> (none)
- L5: value SRN6045TA-3R3Y -> 3.3uH; footprint Inductor_SMD:L_Bourns_SRN6045TA -> Inductor_SMD:L_Sunlord_MWSA0804S; JLCPCB part (none) -> C17700166; Manufacturer part (none) -> MWSA0804S-3R3MT; Notes 3.3µH Semi-Shielded Wirewound Inductor 7.8A 21mOhm Nonstand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 -> (none); Supplier https://www.digikey.ch/de/products/detail/bourns-inc/SRN604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 -> (none)
- R12: value 12K -> 68k; JLCPCB part (none) -> C17801; Manufacturer part (none) -> 0805W8F6802T5E; Notes Resistor 12K 1% 63mW -> Resistor 68k 1% 63mW; Supplier https://www.digikey.ch/de/products/detail/stackpole-electro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 -> (none)
- R13: value 10R -> 68k; JLCPCB part (none) -> C17801; Manufacturer part (none) -> 0805W8F6802T5E; Notes Resistor 10R 1% 63mW -> Resistor 68k 1% 63mW; Supplier https://www.digikey.ch/de/products/detail/stackpole-electro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 -> (none)
- R14: value 20K -> 10k; JLCPCB part (none) -> C17414; Manufacturer part (none) -> 0805W8F1002T5E; Notes Resistor 20K 1% 63mW -> Resistor 10k 1% 63mW; Supplier https://www.digikey.ch/de/products/detail/stackpole-electro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 -> (none)
- R15: value 2K2 -> 9.1k; JLCPCB part (none) -> C17855; Manufacturer part (none) -> 0805W8F9101T5E; Notes Resistor 2.2K 1% 63mW -> Resistor 9.1k 1% 63mW; Supplier https://www.digikey.ch/de/products/detail/stackpole-electro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 -> (none)
- R32: JLCPCB part (none) -> C25803; Manufacturer part (none) -> 0603WAF1003T5E; Notes JLCPCB C25803 -> (none)
- R35, R36: footprint Resistor_SMD:R_0201_0603Metric -> Resistor_SMD:R_0603_1608Metric
- U13: value LT3045xMSE -> LT3045EMSE#PBF; JLCPCB part (none) -> C580012; Manufacturer part (none) -> LT3045EMSE#PBF
- U15: value TPS7A20xxxDBV -> TPS7A2033PDBVR; JLCPCB part (none) -> C2862740; Supplier (none) -> Texas Instruments TPS7A2033PDBVR
Connections:
- net +3V3: now also U5.5 (OUT)
- net +5VP: now also U5.1 (IN), U5.3 (EN)
- net GND: now also R14.2, U5.2 (GND), U6.3 (AGND), U6.9 (PGND)
- net polarity_checked: now also R13.1, U6.8 (VIN)
- net switch: now also C30.2, U6.6 (SW); no longer R13.1
- net at R13.2: now also R14.1, U6.1 (EN); no longer C30.1
- net at R12.2, R15.1: now also U6.2 (FB)
- new net: C30.1, U6.7 (BOOT)
- no-connect marks 2 -> 4
Other:
- note added: "5.5mm × 2.1mm, Center Positive"
- note removed: "+5v @ 3A PSU ( 7.5v-28v Input )"
- note removed: "5.5mm x 2.1mm, Center Negative."
- note removed: "5v @ 3A PSU"
- moved on the sheet: C3, C30, C36, C6, L5, R12, R13, R14, R15, TP1, TP2, TP3

Commit message: a few edits
Parts:
- U6: footprint Pedalboard Library:RPA0010A -> RPA0010A
Changed lines of the file:
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@@
 			)
 		)
-		(property "Footprint" "Pedalboard Library:RPA0010A"
+		(property "Footprint" "RPA0010A"
 			(at 119.38 130.81 0)
 			(hide yes)

Commit message: fixed warnings.
Parts:
- U6: footprint RPA0010A -> Pedalboard Library:RPA0010A
Changed lines of the file:
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@@
 			)
 		)
-		(property "Footprint" "RPA0010A"
+		(property "Footprint" "Pedalboard Library:RPA0010A"
 			(at 119.38 130.81 0)
 			(hide yes)

Commit message: Standardize values.
Parts:
- C59: value 10u -> 10uF
- C60: value 100n -> 100nF
- C71, C72: value 1u -> 1uF
- R15: value 9.1k -> 9k1
- R35: value 15K -> 15k
- R36: value 10K -> 10k
Changed lines of the file:
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@@
 			)
 		)
-		(property "Value" "1u"
+		(property "Value" "1uF"
 			(at 217.932 79.248 0)
 			(show_name no)
@@
 			)
 		)
-		(property "Value" "9.1k"
+		(property "Value" "9k1"
 			(at 159.258 147.193 0)
 			(show_name no)
@@
 			)
 		)
-		(property "Value" "10K"
+		(property "Value" "10k"
 			(at 149.352 75.946 0)
 			(show_name no)
@@
 			)
 		)
-		(property "Value" "15K"
+		(property "Value" "15k"
 			(at 147.828 67.818 90)
 			(show_name no)
@@
 			)
 		)
-		(property "Value" "1u"
+		(property "Value" "1uF"
 			(at 246.126 79.756 0)
 			(show_name no)
@@
 			)
 		)
-		(property "Value" "100n"
+		(property "Value" "100nF"
 			(at 167.64 76.454 0)
 			(show_name no)
@@
 			)
 		)
-		(property "Value" "10u"
+		(property "Value" "10uF"
 			(at 158.242 75.692 0)
 			(show_name no)

Commit message: edited metadata
Parts:
- U13: value LT3045EMSE#PBF -> LT3045; Manufacturer (none) -> Analog Devices
- U15: value TPS7A2033PDBVR -> TPS7A20; Manufacturer (none) -> Texas Instruments; Manufacturer part (none) -> TPS7A2033PDBVR; Supplier Texas Instruments TPS7A2033PDBVR -> (none)
- U5: value TPS7A2033PDBVR -> TPS7A20; Manufacturer (none) -> Texas Insturments
Other:
- moved on the sheet: C71, C72

Commit message: more meta
Parts:
- C2, C4: Manufacturer (none) -> Murata
- C24, C27, C28, C32, C36, C37: Manufacturer (none) -> Samsung
- C30: Manufacturer (none) -> Yageo
- U5: Manufacturer Texas Insturments -> Texas Instruments
- U6: Manufacturer (none) -> Texas Instruments
Other:
- note added: "MODE open => Selects FCCM."
- note added: "Place C3, C5 and C6 directly at U6 VIN/PGND. Place C30 directly between BOOT and SW. Place C27, C28, C32, C36 and C37 close to L5/U6 PGND. Connect the +5VP load after this bank. Place R12/R15 close to FB; route FB away from SW/L5 and sense +5VP at the output-capacitor bank."
- moved on the sheet: C28, C3, C30, C32, C36, C37, C5, C6, C71, C72, L5, R12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
