File: psu.kicad_sch (KiCad schematic)
At the start: 38 parts, among them J6 Screw_Terminal_01x02, J7 Barrel_Jack_MountingPin, Q1 FDS4435BZ, U13 LT3045, U15 TPS7A20, U5 TPS7A20, U6 TPS56637RPAR

Commit message: Changed 5V chip to TLVM13660
Parts:
- removed C36, C37: 10uF, Capacitor_SMD:C_0805_2012Metric, symbol Device:C_Small
- removed C6: 100nF, Capacitor_SMD:C_0805_2012Metric, symbol Device:C_Small
- removed L5: 3.3uH, Inductor_SMD:L_Sunlord_MWSA0804S, symbol Device:L
- removed TP1, TP2, TP3: TestPoint, TestPoint:TestPoint_Pad_2.0x2.0mm, symbol Connector:TestPoint
- removed U6: TPS56637RPAR, Pedalboard Library:RPA0010A, symbol TPS56637:TPS56637RPAR
- added R17: 13k, Resistor_SMD:R_0805_2012Metric, symbol Device:R_Small
- added U6: TLVM13660, Pedalboard Library:B3QFN20_RDL_TEX, symbol TLVM13660:TLVM13660RDLR
- C28, C32: value 10uF -> 47uF; footprint Capacitor_SMD:C_0805_2012Metric -> Capacitor_SMD:C_1210_3225Metric; JLCPCB part C15850 -> C415541; Manufacturer Samsung -> Murata; Manufacturer part CL21A106KAYNNNE -> GRM32ER71A476ME15L; Notes (none) -> Extended part
- C3, C5: footprint Capacitor_SMD:C_0805_2012Metric -> Capacitor_SMD:C_1210_3225Metric; JLCPCB part C440198 -> C2168464; Manufacturer (none) -> Taiyo Yuden; Manufacturer part GRM21BR61H106KE43L -> UMJ325KB7106KMHT; Notes (none) -> Extended part
- C30: value 100nF -> 22pF; JLCPCB part C49678 -> C1804; Manufacturer Yageo -> Samsung Electro-Mechanics; Manufacturer part CC0805KRX7R9BB104 -> CL21C220JBANNNC
- R12: value 68k -> 40.2k; JLCPCB part C17801 -> C17678; Manufacturer (none) -> UNI-ROYAL; Manufacturer part 0805W8F6802T5E -> 0805W8F4022T5E; Notes Resistor 68k 1% 63mW -> Resistor 40.2k 1% 125mW
- R13: Manufacturer (none) -> UNI-ROYAL; Notes Resistor 68k 1% 63mW -> Resistor 68k 1% 125mW
- R14: Manufacturer (none) -> UNI-ROYAL; Notes Resistor 10k 1% 63mW -> Resistor 10k 1% 125mW
- R15: value 9k1 -> 10k; JLCPCB part C17855 -> C17414; Manufacturer (none) -> UNI-ROYAL; Manufacturer part 0805W8F9101T5E -> 0805W8F1002T5E; Notes Resistor 9.1k 1% 63mW -> Resistor 10k 1% 125mW
Connections:
- net switch is gone; now on an unnamed net: C30.2
- net +5VP: now also C30.1, U6.5 (VLDOIN), U6.8 (VOUT1), U6.9 (VOUT2)
- net GND: now also R15.1, R17.2, U6.11 (AGND), U6.17 (PGND), U6.18 (PGND), U6.19 (PGND), U6.20 (PGND), U6.6 (AGND); no longer R15.2
- net polarity_checked: now also U6.1 (VIN1), U6.16 (VIN2)
- net at R13.2, R14.1: now also U6.14 (EN)
- net at R12.2: now also R15.2, U6.10 (FB); no longer R15.1
- new net: R17.1, U6.12 (RT)
- no-connect marks 4 -> 6
Other:
- note added: "PCB layout: Place C3/C5 close to VIN and PGND. Place C28/C32 close to VOUT and PGND. Keep R12, R15, C30 and R17 close to U6 and away from noisy power copper."
- note removed: "MODE open => Selects FCCM."
- note removed: "Place C3, C5 and C6 directly at U6 VIN/PGND. Place C30 directly between BOOT and SW. Place C27, C28, C32, C36 and C37 close to L5/U6 PGND. Connect the +5VP load after this bank. Place R12/R15 close to FB; route FB away from SW/L5 and sense +5VP at the output-capacitor bank."

Commit message: Updated various metadata
Parts:
- added R20: 100k, Resistor_SMD:R_0603_1608Metric, symbol Device:R_Small
- C24: Manufacturer Samsung -> Samsung Electro-Mechanics; Notes (none) -> 10uF, 25V, X5R, ±10%. U5 output capacitor. JLCPCB Basic.
- C27: Manufacturer Samsung -> Samsung Electro-Mechanics; Notes (none) -> 10uF, 25V, X5R, ±10%. U5 input capacitor. JLCPCB Basic.
- C53, C54: Manufacturer (none) -> Samsung Electro-Mechanics
- C55: Manufacturer (none) -> Murata
- C59: Manufacturer (none) -> Samsung Electro-Mechanics; Manufacturer part (none) -> CL10A106KP8NNNC; Supplier Samsung CL10A106KP8NNNC -> (none)
- C60: Manufacturer (none) -> Yageo; Manufacturer part (none) -> CC0603KRX7R9BB104; Notes 10% 50V Ceramic Capacitor X7R -> (none); Supplier Yageo CC0603KRX7R9BB104 -> (none)
- C71: Manufacturer (none) -> Samsung Electro-Mechanics; Manufacturer part (none) -> CL21B105KBFNNNE; Notes (none) -> 1uF, 50V, X7R, ±10%. U15 input capacitor. JLCPCB Basic.; Supplier Samsung CL21B105KBFNNNE -> (none)
- C72: Manufacturer (none) -> Samsung Electro-Mechanics; Manufacturer part (none) -> CL21B105KBFNNNE; Notes (none) -> 1uF, 50V, X7R, ±10%. U15 output capacitor. JLCPCB Basic.; Supplier Samsung CL21B105KBFNNNE -> (none)
- F1: Manufacturer (none) -> Littelfuse
- J6: Manufacturer (none) -> Phoenix Contact; Manufacturer part (none) -> 1715022; Supplier https://www.digikey.ch/de/products/detail/phoenix-contact/1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 -> (none)
- J7: Manufacturer (none) -> Würth Elektronik; Manufacturer part (none) -> 694106301002; Supplier https://www.digikey.ch/de/products/detail/w%C3%BCrth-elektr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 -> (none)
- Q1: Manufacturer (none) -> onsemi; Manufacturer part (none) -> FDS4435BZ; Supplier https://www.digikey.ch/de/products/detail/onsemi/FDS4435BZ/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 -> (none)
- R13: value 68k -> 62k; JLCPCB part C17801 -> C17783; Manufacturer part 0805W8F6802T5E -> 0805W8F6202T5E; Notes Resistor 68k 1% 125mW -> (none)
- R32: Manufacturer (none) -> UNI-ROYAL
- R35: Manufacturer (none) -> UNI-ROYAL; Manufacturer part (none) -> 0603WAF1502T5E; Supplier UNI-ROYAL 0603WAF1502T5E -> (none)
- R36: Manufacturer (none) -> UNI-ROYAL; Manufacturer part (none) -> 0603WAF1002T5E; Supplier UNI-ROYAL 0603WAF1002T5E -> (none)
- U15: Notes (none) -> Dedicated TAC5212 AVDD regulator. Required in full and mini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
- U5: Notes (none) -> General 3.3V rail and TAC5212 IOVDD. Required in full and m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
Connections:
- net +5VP: now also R20.1; no longer U15.3 (EN), U5.3 (EN)
- net 5V_PG: now reaches U6.13 (PG)
- net 5V_PG: now also U15.3 (EN), U5.3 (EN), R20.2
- no-connect marks 6 -> 5
Other:
- moved on the sheet: C71, R17, U15

Commit message: changed to lt3042
Parts:
- removed U13: LT3045, Package_SO:MSOP-12-1EP_3x4.039mm_P0.65mm_EP1.651x2.845mm, symbol Regulator_Linear:LT3045xMSE
- added U13: LT3042, Package_SO:MSOP-10-1EP_3x3mm_P0.5mm_EP1.68x1.88mm, symbol Regulator_Linear:LT3042xMSE
Connections:
- net +10V: now also U13.10 (OUT), U13.9 (OUTS)
- net GND: now also U13.11 (GND), U13.5 (ILIM), U13.8 (GND)
- net polarity_checked: now also U13.1 (IN), U13.2 (IN), U13.3 (EN/UV), U13.6 (PGFB)
- net at C53.1, R32.1: now also U13.7 (SET)
Other:
- note added: "Kelvin SET return: R32 and C53 share this return node. Route it directly to C54 negative/load ground. Do not connect this node to U13 GND or the ground plane before C54−."
- note added: "Kelvin VOUT sense: OUTS is the same electrical net as OUT. Route OUTS separately from pin 9 to the COUT positive/load node, and join OUT there."
- moved on the sheet: C54, C59, C60, R32, R35, R36

Commit message: update components
Parts:
- removed C53: 4.7uF, Capacitor_SMD:C_0805_2012Metric, symbol Device:C_Small
- added C53: 4.7uF, Capacitor_Tantalum_SMD:CP_EIA-3216-18_Kemet-A, symbol Device:C_Polarized_Small_US
- C55: value 10uF -> 4.7uF; footprint Capacitor_SMD:C_0805_2012Metric -> Capacitor_SMD:C_1206_3216Metric; JLCPCB part C440198 -> C77096; Manufacturer part GRM21BR61H106KE43L -> GRM31CR71H475KA12L
- U13: JLCPCB part (none) -> C69847
Connections:
- net GND: now also C53.2
- net at R32.1, U13.7 (SET): now also C53.1
Other:
- moved on the sheet: C71

Commit message: more edits
Parts:
- C55: value 4.7uF -> 10uF; JLCPCB part C77096 -> C13585; Manufacturer Murata -> Samsung Electro-Mechanics; Manufacturer part GRM31CR71H475KA12L -> CL31A106KBHNNNE
Changed lines of the file:
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@@
 			)
 		)
-		(property "Value" "4.7uF"
+		(property "Value" "10uF"
 			(at 141.732 37.592 0)
 			(show_name no)
@@
 			)
 		)
-		(property "Manufacturer" "Murata"
+		(property "Manufacturer" "Samsung Electro-Mechanics"
 			(at 147.32 35.56 0)
 			(hide yes)
@@
 			)
 		)
-		(property "Manufacturer part" "GRM31CR71H475KA12L"
+		(property "Manufacturer part" "CL31A106KBHNNNE"
 			(at 147.32 35.56 0)
 			(hide yes)
@@
 			)
 		)
-		(property "JLCPCB part" "C77096"
+		(property "JLCPCB part" "C13585"
 			(at 147.32 35.56 0)
 			(hide yes)

Commit message: update psu
Parts:
- removed C24, C27: 10uF, Capacitor_SMD:C_0805_2012Metric, symbol Device:C_Small
- removed U5: TPS7A20, Package_TO_SOT_SMD:SOT-23-5, symbol Regulator_Linear:TPS7A20xxxDBV

Commit message: added test points
Parts:
- removed C2, C4: 10uF, Capacitor_SMD:C_0805_2012Metric, symbol Device:C_Small
- added C2: 100uF, Capacitor_THT:CP_Radial_D6.3mm_P2.50mm, symbol Device:C_Polarized_Small_US
- added TP1: VIN, TestPoint:TestPoint_Pad_D1.5mm, symbol Connector:TestPoint
- added TP2: 10V, TestPoint:TestPoint_Pad_D1.5mm, symbol Connector:TestPoint
- added TP3: CODEC_3V3, TestPoint:TestPoint_Pad_D1.5mm, symbol Connector:TestPoint
- added TP5: Gnd, TestPoint:TestPoint_Pad_D1.5mm, symbol Connector:TestPoint
- added TP6: 5V, TestPoint:TestPoint_Pad_D1.5mm, symbol Connector:TestPoint
- F1: value PTC 4A 15V -> PTC 4A 30V; JLCPCB part C720182 -> C19078761; Manufacturer Littelfuse -> LUTE; Manufacturer part 2920L400/15MR -> 2920L400/30GR
Connections:
- net +10V: now also TP2.1
- net +5VP: now also TP6.1
- net 3V3_CODEC: now also TP3.1
- net GND: now also C2.2, TP5.1
- net fused: now also C2.1
- net polarity_checked: now also TP1.1
Other:
- note added: "POWER INPUT: 12 VDC regulated, 4 A recommended"

Commit message: small edit
Connections:
- net fused: no longer C2.1
- net polarity_checked: now also C2.1
Other:
- moved on the sheet: C2, TP1
Changed lines of the file:
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@@
 	)
 	(junction
-		(at 73.66 73.66)
+		(at 140.97 27.94)
 		(diameter 0)
 		(color 0 0 0 0)
 	)
 	(junction
-		(at 140.97 27.94)
+		(at 184.15 30.48)
 		(diameter 0)
 		(color 0 0 0 0)
 	)
 	(junction
-		(at 184.15 30.48)
+		(at 64.77 144.78)
 		(diameter 0)
 		(color 0 0 0 0)
 	)
 	(junction
-		(at 64.77 144.78)
+		(at 101.6 40.64)
 		(diameter 0)
 		(color 0 0 0 0)
@@
 	)
 	(junction
+		(at 90.17 73.66)
+		(diameter 0)
+		(color 0 0 0 0)
+	)
+	(junction
 		(at 120.65 171.45)
 		(diameter 0)
@@
 		(color 0 0 0 0)
 	)
-	(junction
-		(at 73.66 40.64)
-		(diameter 0)
-		(color 0 0 0 0)
-	)
 	(no_connect
 		(at 39.37 46.99)
@@
 	(wire
 		(pts
-			(xy 33.02 171.45) (xy 33.02 172.72)
+			(xy 101.6 73.66) (xy 90.17 73.66)
 		)
 		(stroke
@@
 	(wire
 		(pts
-			(xy 152.4 93.98) (xy 157.48 93.98)
+			(xy 33.02 171.45) (xy 33.02 172.72)
 		)
 		(stroke
@@
 	(wire
 		(pts
-			(xy 172.72 46.99) (xy 172.72 43.18)
+			(xy 152.4 93.98) (xy 157.48 93.98)
 		)
 		(stroke
@@
 	(wire
 		(pts
-			(xy 251.46 87.63) (xy 251.46 91.44)
+			(xy 172.72 46.99) (xy 172.72 43.18)
 		)
 		(stroke
@@
 	(wire
 		(pts
-			(xy 157.48 86.36) (xy 157.48 83.82)
+			(xy 251.46 87.63) (xy 251.46 91.44)
 		)
 		(stroke
@@
 	(wire
 		(pts
-			(xy 187.96 25.4) (xy 187.96 27.94)
+			(xy 157.48 86.36) (xy 157.48 83.82)
 		)
 		(stroke
@@
 	(wire
 		(pts
-			(xy 54.61 73.66) (xy 73.66 73.66)
+			(xy 187.96 25.4) (xy 187.96 27.94)
 		)
 		(stroke
@@
 	(wire
 		(pts
-			(xy 73.66 40.64) (xy 82.55 40.64)
+			(xy 69.85 40.64) (xy 82.55 40.64)
 		)
 		(stroke
@@
 	(wire
 		(pts
-			(xy 73.66 73.66) (xy 90.17 73.66)
+			(xy 54.61 73.66) (xy 90.17 73.66)
 		)
 		(stroke
@@
 	(wire
 		(pts
-			(xy 73.66 40.64) (xy 73.66 53.34)
-		)
-		(stroke
-			(width 0)
-			(type default)
-		)
-	)
-	(wire
-		(pts
 			(xy 64.77 147.32) (xy 64.77 144.78)
 		)
@@
 	(wire
 		(pts
+			(xy 101.6 40.64) (xy 121.92 40.64)
+		)
+		(stroke
+			(width 0)
+			(type default)
+		)
+	)
+	(wire
+		(pts
 			(xy 114.3 154.94) (xy 133.35 154.94)
 		)
@@
 	(wire
 		(pts
-			(xy 69.85 40.64) (xy 73.66 40.64)
+			(xy 177.8 27.94) (xy 184.15 27.94)
 		)
 		(stroke
@@
 	(wire
 		(pts
-			(xy 177.8 27.94) (xy 184.15 27.94)
+			(xy 101.6 40.64) (xy 101.6 53.34)
 		)
 		(stroke
@@
 	(wire
 		(pts
-			(xy 114.3 167.64) (xy 116.84 167.64)
+			(xy 101.6 58.42) (xy 101.6 73.66)
 		)
 		(stroke
@@
 	(wire
 		(pts
-			(xy 133.35 137.16) (xy 133.35 154.94)
+			(xy 114.3 167.64) (xy 116.84 167.64)
 		)
 		(stroke
@@
 	(wire
 		(pts
-			(xy 45.72 73.66) (xy 45.72 77.47)
+			(xy 133.35 137.16) (xy 133.35 154.94)
 		)
 		(stroke
@@
 	(wire
 		(pts
-			(xy 152.4 91.44) (xy 152.4 93.98)
+			(xy 45.72 73.66) (xy 45.72 77.47)
 		)
 		(stroke
@@
 	(wire
 		(pts
-			(xy 152.4 35.56) (xy 152.4 43.18)
+			(xy 152.4 91.44) (xy 152.4 93.98)
 		)
 		(stroke
@@
 	(wire
 		(pts
-			(xy 233.68 92.71) (xy 233.68 90.17)
+			(xy 152.4 35.56) (xy 152.4 43.18)
 		)
 		(stroke
@@
 	(wire
 		(pts
-			(xy 73.66 58.42) (xy 73.66 73.66)
+			(xy 233.68 92.71) (xy 233.68 90.17)
 		)
 		(stroke
@@
 	(wire
 		(pts
-			(xy 96.52 40.64) (xy 116.84 40.64)
+			(xy 96.52 40.64) (xy 101.6 40.64)
 		)
 		(stroke
@@
 	)
 	(label "polarity_checked"
-		(at 115.57 40.64 180)
+		(at 119.38 40.64 180)
 		(effects
 			(font
@@
 	(symbol
 		(lib_id "Device:C_Polarized_Small_US")
-		(at 73.66 55.88 0)
+		(at 101.6 55.88 0)
 		(unit 1)
 		(body_style 1)
@@
 		(dnp yes)
 		(property "Reference" "C2"
-			(at 68.072 54.864 0)
+			(at 96.012 54.864 0)
 			(show_name no)
 			(do_not_autoplace no)
@@
 		)
 		(property "Value" "100uF"
-			(at 68.834 57.15 0)
+			(at 96.774 57.15 0)
 			(show_name no)
 			(do_not_autoplace no)
@@
 		)
 		(property "Footprint" "Capacitor_THT:CP_Radial_D6.3mm_P2.50mm"
-			(at 73.66 55.88 0)
+			(at 101.6 55.88 0)
 			(hide yes)
 			(show_name no)
@@
 		)
 		(property "Datasheet" ""
-			(at 73.66 55.88 0)
+			(at 101.6 55.88 0)
 			(hide yes)
 			(show_name no)
@@
 		)
 		(property "Description" ""
-			(at 73.66 55.88 0)
+			(at 101.6 55.88 0)
 			(hide yes)
 			(show_name no)
@@
 		)
 		(property "Manufacturer part" "NHG"
-			(at 73.66 55.88 0)
+			(at 101.6 55.88 0)
 			(hide yes)
 			(show_name no)
@@
 		)
 		(property "Manufacturer" "Panasonic"
-			(at 73.66 55.88 0)
+			(at 101.6 55.88 0)
 			(hide yes)
 			(show_name no)
@@
 		)
 		(property "Notes" "Input damping capacitor. Fit manually before power-up."
-			(at 73.66 55.88 0)
+			(at 101.6 55.88 0)
 			(hide yes)
 			(show_name no)
@@
 		)
 		(property "JLCPCB part" ""
-			(at 73.66 55.88 0)
+			(at 101.6 55.88 0)
 			(hide yes)
 			(show_name no)
@@
 			)
 		)
-		(property "Datasheet" "https://www.littelfuse.com/assetdocs/2920l_datasheet_update.pdf"
+		(property "Datasheet" "https://www.lcsc.com/datasheet/C19078761.pdf"
 			(at 66.04 40.64 0)
 			(hide yes)
@@
 	(symbol
 		(lib_id "Connector:TestPoint")
-		(at 116.84 40.64 0)
+		(at 121.92 40.64 0)
 		(unit 1)
 		(body_style 1)
@@
 		(dnp no)
 		(property "Reference" "TP1"
-			(at 115.57 33.528 0)
+			(at 120.65 33.528 0)
 			(show_name no)
 			(do_not_autoplace no)
@@
 		)
 		(property "Value" "VIN"
-			(at 115.316 35.56 0)
+			(at 120.396 35.56 0)
 			(show_name no)
 			(do_not_autoplace no)
@@
 		)
 		(property "Footprint" "TestPoint:TestPoint_Pad_D1.5mm"
-			(at 121.92 40.64 0)
+			(at 127 40.64 0)
 			(hide yes)
 			(show_name no)
@@
 		)
 		(property "Datasheet" ""
-			(at 121.92 40.64 0)
+			(at 127 40.64 0)
 			(hide yes)
 			(show_name no)
@@
 		)
 		(property "Description" "test point"
-			(at 116.84 40.64 0)
+			(at 121.92 40.64 0)
 			(hide yes)
 			(show_name no)
