File: psu.kicad_sch (KiCad schematic)
At the start: 34 parts, among them J6 Screw_Terminal_01x02, J7 Barrel_Jack_MountingPin, Q1 FDS4435BZ, U13 LT3042, U15 TPS7A20, U6 TLVM13660

Commit message: initial placement fiddling
Parts:
- C30: footprint Capacitor_SMD:C_0805_2012Metric -> Capacitor_SMD:C_0402_1005Metric; JLCPCB part C1804 -> C1555; Manufacturer part CL21C220JBANNNC -> 0402CG220J500NT
- R12: footprint Resistor_SMD:R_0805_2012Metric -> Resistor_SMD:R_0402_1005Metric; JLCPCB part C17678 -> C25893; Manufacturer part 0805W8F4022T5E -> 0402WGF4022TCE; Notes Resistor 40.2k 1% 125mW -> Resistor 40.2k 1% 62.5mW - "Promotional extended"
- R13: footprint Resistor_SMD:R_0805_2012Metric -> Resistor_SMD:R_0402_1005Metric; JLCPCB part C17783 -> C37825; Manufacturer part 0805W8F6202T5E -> 0402WGF6202TCE
- R14, R15: footprint Resistor_SMD:R_0805_2012Metric -> Resistor_SMD:R_0402_1005Metric; JLCPCB part C17414 -> C25744; Manufacturer part 0805W8F1002T5E -> 0402WGF1002TCE; Notes Resistor 10k 1% 125mW -> Resistor 10k 1% 62.5mW
- R17: footprint Resistor_SMD:R_0805_2012Metric -> Resistor_SMD:R_0402_1005Metric; JLCPCB part C17455 -> C25754; Manufacturer part 0805W8F1302T5E -> 0402WGF1302TCE; Notes Resistor 13k 1% 125mW -> (none)
Changed lines of the file:
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@@
 			)
 		)
-		(property "Footprint" "Resistor_SMD:R_0805_2012Metric"
+		(property "Footprint" "Resistor_SMD:R_0402_1005Metric"
 			(at 131.572 163.83 90)
 			(hide yes)
@@
 			)
 		)
-		(property "Notes" "Resistor 10k 1% 125mW"
+		(property "Notes" "Resistor 10k 1% 62.5mW"
 			(at 133.35 163.83 0)
 			(hide yes)
@@
 			)
 		)
-		(property "Manufacturer part" "0805W8F1002T5E"
+		(property "Manufacturer part" "0402WGF1002TCE"
 			(at 133.35 163.83 0)
 			(hide yes)
@@
 			)
 		)
-		(property "JLCPCB part" "C17414"
+		(property "JLCPCB part" "C25744"
 			(at 133.35 163.83 0)
 			(hide yes)
@@
 			)
 		)
-		(property "Footprint" "Resistor_SMD:R_0805_2012Metric"
+		(property "Footprint" "Resistor_SMD:R_0402_1005Metric"
 			(at 131.572 157.48 90)
 			(hide yes)
@@
 			)
 		)
-		(property "Manufacturer part" "0805W8F6202T5E"
+		(property "Manufacturer part" "0402WGF6202TCE"
 			(at 133.35 157.48 0)
 			(hide yes)
@@
 			)
 		)
-		(property "JLCPCB part" "C17783"
+		(property "JLCPCB part" "C37825"
 			(at 133.35 157.48 0)
 			(hide yes)
@@
 			)
 		)
-		(property "Footprint" "Capacitor_SMD:C_0805_2012Metric"
+		(property "Footprint" "Capacitor_SMD:C_0402_1005Metric"
 			(at 59.3852 172.72 0)
 			(hide yes)
@@
 			)
 		)
-		(property "Manufacturer part" "CL21C220JBANNNC"
+		(property "Manufacturer part" "0402CG220J500NT"
 			(at 58.42 168.91 0)
 			(hide yes)
@@
 			)
 		)
-		(property "JLCPCB part" "C1804"
+		(property "JLCPCB part" "C1555"
 			(at 58.42 168.91 0)
 			(hide yes)
@@
 			)
 		)
-		(property "Footprint" "Resistor_SMD:R_0805_2012Metric"
+		(property "Footprint" "Resistor_SMD:R_0402_1005Metric"
 			(at 51.562 168.91 90)
 			(hide yes)
@@
 			)
 		)
-		(property "JLCPCB part" "C17678"
+		(property "JLCPCB part" "C25893"
 			(at 53.34 168.91 0)
 			(hide yes)
@@
 			)
 		)
-		(property "Manufacturer part" "0805W8F4022T5E"
+		(property "Manufacturer part" "0402WGF4022TCE"
 			(at 53.34 168.91 0)
 			(hide yes)
@@
 			)
 		)
-		(property "Notes" "Resistor 40.2k 1% 125mW"
+		(property "Notes" "Resistor 40.2k 1% 62.5mW - \"Promotional extended\""
 			(at 53.34 168.91 0)
 			(hide yes)
@@
 			)
 		)
-		(property "Footprint" "Resistor_SMD:R_0805_2012Metric"
+		(property "Footprint" "Resistor_SMD:R_0402_1005Metric"
 			(at 118.872 167.64 90)
 			(hide yes)
@@
 			)
 		)
-		(property "Manufacturer part" "0805W8F1302T5E"
+		(property "Manufacturer part" "0402WGF1302TCE"
 			(at 120.65 167.64 0)
 			(hide yes)
@@
 			)
 		)
-		(property "JLCPCB part" "C17455"
+		(property "JLCPCB part" "C25754"
 			(at 120.65 167.64 0)
 			(hide yes)
@@
 		)
 		(property "Manufacturer" "UNI-ROYAL"
-			(at 120.65 167.64 90)
-			(hide yes)
-			(show_name no)
-			(do_not_autoplace no)
-			(effects
-				(font
-					(size 1.27 1.27)
-				)
-			)
-		)
-		(property "Notes" "Resistor 13k 1% 125mW"
 			(at 120.65 167.64 90)
 			(hide yes)
@@
 			)
 		)
-		(property "Footprint" "Resistor_SMD:R_0805_2012Metric"
+		(property "Footprint" "Resistor_SMD:R_0402_1005Metric"
 			(at 48.26 174.498 90)
 			(hide yes)
@@
 			)
 		)
-		(property "Notes" "Resistor 10k 1% 125mW"
+		(property "Notes" "Resistor 10k 1% 62.5mW"
 			(at 48.26 172.72 0)
 			(hide yes)
@@
 			)
 		)
-		(property "Manufacturer part" "0805W8F1002T5E"
+		(property "Manufacturer part" "0402WGF1002TCE"
 			(at 48.26 172.72 0)
 			(hide yes)
@@
 			)
 		)
-		(property "JLCPCB part" "C17414"
+		(property "JLCPCB part" "C25744"
 			(at 48.26 172.72 0)
 			(hide yes)

Commit message: components placed.
Parts:
- C53: value 4.7uF -> 10uF; footprint Capacitor_Tantalum_SMD:CP_EIA-3216-18_Kemet-A -> Capacitor_SMD:C_1206_3216Metric; symbol Device:C_Polarized_Small_US -> Device:C_Small; JLCPCB part C7189 -> C13585; Manufacturer KYOCERA AVX -> Samsung; Manufacturer part TAJA475K025RNJ -> CL31A106KBHNNNE
Changed lines of the file:
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@@
 	)
 	(symbol
-		(lib_id "Device:C_Polarized_Small_US")
+		(lib_id "Device:C_Small")
 		(at 168.91 46.99 90)
 		(unit 1)
@@
 			)
 		)
-		(property "Value" "4.7uF"
+		(property "Value" "10uF"
 			(at 168.91 51.562 90)
 			(show_name no)
@@
 			)
 		)
-		(property "Footprint" "Capacitor_Tantalum_SMD:CP_EIA-3216-18_Kemet-A"
+		(property "Footprint" "Capacitor_SMD:C_1206_3216Metric"
 			(at 168.91 46.99 0)
 			(hide yes)
@@
 			)
 		)
-		(property "Description" "Polarized capacitor, small US symbol"
+		(property "Description" "Unpolarized capacitor, small symbol"
+			(at 179.07 46.99 0)
+			(hide yes)
+			(show_name no)
+			(do_not_autoplace no)
+			(effects
+				(font
+					(size 1.27 1.27)
+				)
+			)
+		)
+		(property "Manufacturer" "Samsung"
 			(at 168.91 46.99 0)
 			(hide yes)
@@
 			)
 		)
-		(property "Manufacturer" "KYOCERA AVX"
+		(property "Manufacturer part" "CL31A106KBHNNNE"
 			(at 168.91 46.99 0)
 			(hide yes)
@@
 			)
 		)
-		(property "Manufacturer part" "TAJA475K025RNJ"
+		(property "JLCPCB part" "C13585"
 			(at 168.91 46.99 0)
 			(hide yes)
-			(show_name no)
-			(do_not_autoplace no)
-			(effects
-				(font
-					(size 1.27 1.27)
-				)
-			)
-		)
-		(property "JLCPCB part" "C7189"
-			(at 168.91 46.99 0)
-			(hide yes)

Commit message: more psu
Parts:
- added C80: 10uF, Capacitor_SMD:C_1206_3216Metric, symbol Device:C_Small
- added C82: 22uF, Capacitor_SMD:C_1206_3216Metric, symbol Device:C_Small
- C53: value 10uF -> 4.7uF; footprint Capacitor_SMD:C_1206_3216Metric -> Capacitor_SMD:C_1812_4532Metric; JLCPCB part C13585 -> (none); Manufacturer Samsung -> Rubycon; Manufacturer part CL31A106KBHNNNE -> 35MU475KC44532
Connections:
- net +10V: now also C82.1
- net GND: now also C80.2, C82.2
- net polarity_checked: now also C80.1

Commit message: opamp incl power routed
Parts:
- C54: footprint Capacitor_SMD:C_1206_3216Metric -> Capacitor_SMD:C_1210_3225Metric_Pad1.33x2.70mm_HandSolder; JLCPCB part C12891 -> C309062; Manufacturer part CL31A226KAHNNNE -> CL32B226KAJNNNE
- C55: value 10uF -> 22uF; footprint Capacitor_SMD:C_1206_3216Metric -> Capacitor_SMD:C_1210_3225Metric_Pad1.33x2.70mm_HandSolder; JLCPCB part C13585 -> C309062; Manufacturer part CL31A106KBHNNNE -> CL32B226KAJNNNE
- C80: value 10uF -> 22uF; footprint Capacitor_SMD:C_1206_3216Metric -> Capacitor_SMD:C_1210_3225Metric_Pad1.33x2.70mm_HandSolder; JLCPCB part C13585 -> C309062; Manufacturer part CL31A106KBHNNNE -> CL32B226KAJNNNE; now not fitted
- C82: footprint Capacitor_SMD:C_1206_3216Metric -> Capacitor_SMD:C_1210_3225Metric_Pad1.33x2.70mm_HandSolder; JLCPCB part C12891 -> C309062; Manufacturer part CL31A226KAHNNNE -> CL32B226KAJNNNE; now not fitted
Other:
- note added: "4V analog bias"
- note removed: "5V analog bias"

Commit message: Fiddles. Moved J6
Parts:
- C2: now fitted
Changed lines of the file:
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@@
 		(on_board yes)
 		(in_pos_files yes)
-		(dnp yes)
+		(dnp no)
 		(property "Reference" "C2"
 			(at 96.012 54.864 0)

Commit message: various fixes.
Parts:
- J7: now fitted
Changed lines of the file:
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@@
 		(on_board yes)
 		(in_pos_files yes)
-		(dnp yes)
+		(dnp no)
 		(property "Reference" "J7"
 			(at 41.91 54.61 0)
