File: pedalboard-hw.kicad_pcb (KiCad board)
At the start: 4 copper layers, 174 x 111 mm, 120 parts, among them IC1 TAC5212IRGER, J10 USB-A HOST, J11 CM5 BOOT, J13 Headphones 3.5mm, J16 CM5 UART DEBUG, J18 GUITAR INPUT, J19 LINE OUT LEFT, J20 LINE OUT RIGHT, J21 UI LINK 2x5, J22 BALANCED LINE INPUT, J6 Screw_Terminal_01x02, J7 Barrel_Jack_MountingPin, J9 USB-C SERVICE, Q1 FDS4435BZ, SW11 EM-02-Q, U10 AP22653, U11 TPD2E2U06DCK, U13 LT3042, U14 OPA1656ID, U15 TPS7A20, U16 TPD2E2U06DCK, U6 TLVM13660

Commit message: vias
Parts:
- moved TP5 15.4 mm to (152.2, 30.7)
- moved TP1 6.82 mm to (153.5, 37.2)
- moved R14 0.19 mm to (125.3, 42.0)
- moved R13 0.11 mm to (124.9, 40.4)
Routing:
- net +5VP: track 0.00 -> 8.89 mm
- net /Power Supply/5V_PG: track 0.00 -> 4.14 mm
- net Net-(U6-FB): track 0.00 -> 3.88 mm
- net Net-(U6-EN): track 0.00 -> 3.24 mm
- net Net-(U6-RT): track 0.00 -> 1.66 mm
- net GND: vias 0 -> 4
- net /Power Supply/polarity_checked: vias 0 -> 18
- added copper zone on F.Cu, net +5VP
- added copper zone on F.Cu, net /Power Supply/polarity_checked
- added copper zone on In2.Cu, net /Power Supply/polarity_checked
- added copper zone on F.Cu, net GND
- added copper zone on In1.Cu, net GND

Commit message: more via
Routing:
- net GND: vias 4 -> 30
- net /Power Supply/polarity_checked: vias 18 -> 21
- net +5VP: vias 0 -> 12
- added copper zone on In2.Cu, net +5VP
