File: pedalboard-hw.kicad_pcb (KiCad board)
At the start: 4 copper layers, 174 x 111 mm, 120 parts, among them IC1 TAC5212IRGER, J10 USB-A HOST, J11 CM5 BOOT, J13 Headphones 3.5mm, J16 CM5 UART DEBUG, J18 GUITAR INPUT, J19 LINE OUT LEFT, J20 LINE OUT RIGHT, J21 UI LINK 2x5, J22 BALANCED LINE INPUT, J6 Screw_Terminal_01x02, J7 Barrel_Jack_MountingPin, J9 USB-C SERVICE, Q1 FDS4435BZ, SW11 EM-02-Q, U10 AP22653, U11 TPD2E2U06DCK, U13 LT3042, U14 OPA1656ID, U15 TPS7A20, U16 TPD2E2U06DCK, U6 TLVM13660

Commit message: 5V power to CM5
Parts:
- moved TP1 7.39 mm to (159.9, 33.5)
Connections:
- J21 pad 10: ESP_BOOT -> +5VP
- J21 pad 3: +5VP -> ESP_RESET
- J21 pad 5: UI_UART_TX -> UI_UART_RX
- J21 pad 6: GND -> UI_UART_TX
- J21 pad 7: UI_UART_RX -> GND
- J21 pad 8: GND -> ESP_BOOT
- J21 pad 9: ESP_RESET -> GND
Routing:
- net /Power Supply/polarity_checked: track 0.00 -> 8.22 mm
- net +5VP: track 8.89 -> 16.6 mm, vias 12 -> 18
- added copper zone on B.Cu, net GND
Changed lines of the file:
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@@
 	(footprint "TestPoint:TestPoint_Pad_D1.5mm"
 		(layer "F.Cu")
-		(at 153.5 37.2)
+		(at 159.9 33.5)
 		(descr "SMD pad as test Point, diameter 1.5mm")
 		(tags "test point SMD pad")
@@
 			(layers "*.Cu" "*.Mask")
 			(remove_unused_layers no)
-			(net "+5VP")
+			(net "ESP_RESET")
 			(pinfunction "Pin_3_3")
 			(pintype "passive")
@@
 			(layers "*.Cu" "*.Mask")
 			(remove_unused_layers no)
-			(net "UI_UART_TX")
+			(net "UI_UART_RX")
 			(pinfunction "Pin_5_5")
 			(pintype "passive")
@@
 			(layers "*.Cu" "*.Mask")
 			(remove_unused_layers no)
-			(net "GND")
+			(net "UI_UART_TX")
 			(pinfunction "Pin_6_6")
 			(pintype "passive")
@@
 			(layers "*.Cu" "*.Mask")
 			(remove_unused_layers no)
-			(net "UI_UART_RX")
+			(net "GND")
 			(pinfunction "Pin_7_7")
 			(pintype "passive")
@@
 			(layers "*.Cu" "*.Mask")
 			(remove_unused_layers no)
-			(net "GND")
+			(net "ESP_BOOT")
 			(pinfunction "Pin_8_8")
 			(pintype "passive")
@@
 			(layers "*.Cu" "*.Mask")
 			(remove_unused_layers no)
-			(net "ESP_RESET")
+			(net "GND")
 			(pinfunction "Pin_9_9")
 			(pintype "passive")
@@
 			(layers "*.Cu" "*.Mask")
 			(remove_unused_layers no)
-			(net "ESP_BOOT")
+			(net "+5VP")
 			(pinfunction "Pin_10_10")
 			(pintype "passive")
@@
 		(net "GND")
 	)
+	(segment
+		(start 161.35 37.35)
+		(end 165.115 37.35)
+		(width 0.2)
+		(layer "F.Cu")
+		(net "/Power Supply/polarity_checked")
+	)
+	(segment
+		(start 159.9 33.5)
+		(end 159.9 35.9)
+		(width 0.2)
+		(layer "F.Cu")
+		(net "/Power Supply/polarity_checked")
+	)
+	(segment
+		(start 159.9 35.9)
+		(end 161.35 37.35)
+		(width 0.2)
+		(layer "F.Cu")
+		(net "/Power Supply/polarity_checked")
+	)
 	(via
 		(at 127.76 42.25)
@@
 	)
 	(segment
+		(start 104.8 64)
+		(end 104.9 64.1)
+		(width 0.2)
+		(layer "F.Cu")
+		(net "+5VP")
+	)
+	(segment
+		(start 104.6 64.4)
+		(end 104.9 64.1)
+		(width 0.2)
+		(layer "F.Cu")
+		(net "+5VP")
+	)
+	(segment
+		(start 104.6 64.8)
+		(end 104.9 65.1)
+		(width 0.2)
+		(layer "F.Cu")
+		(net "+5VP")
+	)
+	(segment
 		(start 122.2875 42.75)
 		(end 121.3825 42.75)
@@
 	)
 	(segment
+		(start 103.79 63.6)
+		(end 104.7 63.6)
+		(width 0.2)
+		(layer "F.Cu")
+		(net "+5VP")
+	)
+	(segment
 		(start 121.0825 42.51)
 		(end 121.1125 42.48)
@@
 	)
 	(segment
+		(start 103.79 65.2)
+		(end 104.8 65.2)
+		(width 0.2)
+		(layer "F.Cu")
+		(net "+5VP")
+	)
+	(segment
+		(start 103.79 64)
+		(end 104.8 64)
+		(width 0.2)
+		(layer "F.Cu")
+		(net "+5VP")
+	)
+	(segment
+		(start 104.7 63.6)
+		(end 104.9 63.8)
+		(width 0.2)
+		(layer "F.Cu")
+		(net "+5VP")
+	)
+	(segment
+		(start 104.9 65.3)
+		(end 104.9 65.1)
+		(width 0.2)
+		(layer "F.Cu")
+		(net "+5VP")
+	)
+	(segment
+		(start 103.79 64.4)
+		(end 104.6 64.4)
+		(width 0.2)
+		(layer "F.Cu")
+		(net "+5VP")
+	)
+	(segment
+		(start 103.79 64.8)
+		(end 104.6 64.8)
+		(width 0.2)
+		(layer "F.Cu")
+		(net "+5VP")
+	)
+	(segment
+		(start 104.8 65.2)
+		(end 104.9 65.1)
+		(width 0.2)
+		(layer "F.Cu")
+		(net "+5VP")
+	)
+	(segment
 		(start 121.1 33.7)
 		(end 120.624685 34.175315)
@@
 	)
 	(segment
+		(start 104.9 63.8)
+		(end 104.9 64.1)
+		(width 0.2)
+		(layer "F.Cu")
+		(net "+5VP")
+	)
+	(segment
+		(start 103.79 65.6)
+		(end 104.6 65.6)
+		(width 0.2)
+		(layer "F.Cu")
+		(net "+5VP")
+	)
+	(segment
 		(start 120.624685 34.175315)
 		(end 120.624685 34.75)
@@
 	)
 	(segment
+		(start 104.6 65.6)
+		(end 104.9 65.3)
+		(width 0.2)
+		(layer "F.Cu")
+		(net "+5VP")
+	)
+	(segment
 		(start 122.499937 34.499941)
 		(end 122.499937 33.899937)
@@
 	)
 	(via
+		(at 105.8 65.1)
+		(size 0.8)
+		(drill 0.4)
+		(layers "F.Cu" "B.Cu")
+		(free yes)
+		(net "+5VP")
+	)
+	(via
+		(at 105.8 64.1)
+		(size 0.8)
+		(drill 0.4)
+		(layers "F.Cu" "B.Cu")
+		(free yes)
+		(net "+5VP")
+	)
+	(via
 		(at 115.95 41.34)
 		(size 0.8)
@@
 	)
 	(via
+		(at 106.7 64.1)
+		(size 0.8)
+		(drill 0.4)
+		(layers "F.Cu" "B.Cu")
+		(free yes)
+		(net "+5VP")
+	)
+	(via
+		(at 104.9 65.1)
+		(size 0.8)
+		(drill 0.4)
+		(layers "F.Cu" "B.Cu")
+		(free yes)
+		(net "+5VP")
+	)
+	(via
 		(at 115.95 40.44)
 		(size 0.8)
@@
 	)
 	(via
+		(at 106.7 65.1)
+		(size 0.8)
+		(drill 0.4)
+		(layers "F.Cu" "B.Cu")
+		(free yes)
+		(net "+5VP")
+	)
+	(via
 		(at 115.95 42.25)
 		(size 0.8)
@@
 	)
 	(via
-		(at 115.95 31.5)
+		(at 104.9 64.1)
 		(size 0.8)
 		(drill 0.4)
@@
 	)
 	(via
-		(at 115.95 33.3)
+		(at 115.95 31.5)
 		(size 0.8)
 		(drill 0.4)
@@
 	)
 	(via
+		(at 115.95 33.3)
+		(size 0.8)
+		(drill 0.4)
+		(layers "F.Cu" "B.Cu")
+		(free yes)
+		(net "+5VP")
+	)
+	(via
 		(at 118.59 31.5)
 		(size 0.8)
@@
 	)
 	(zone
+		(net "+5VP")
+		(layer "F.Cu")
+		(hatch edge 0.5)
+		(priority 13)
+		(connect_pads yes
+			(clearance 0.2)
+		)
+		(min_thickness 0.2)
+		(fill yes
+			(thermal_gap 0.5)
+			(thermal_bridge_width 0.5)
+			(island_removal_mode 0)
+		)
+		(polygon
+			(pts
+				(xy 104.4 63.5) (xy 104.4 65.7) (xy 107.5 65.7) (xy 107.5 63.5)
+			)
+		)
+	)
+	(zone
 		(net "GND")
 		(layer "F.Cu")
@@
 	(zone
 		(net "GND")
+		(layer "B.Cu")
+		(hatch edge 0.5)
+		(priority 12)
+		(connect_pads thru_hole_only
+			(clearance 0.2)
+		)
+		(min_thickness 0.2)
+		(fill yes
+			(thermal_gap 0.5)
+			(thermal_bridge_width 0.5)
+			(island_removal_mode 0)
+		)
+		(polygon
+			(pts
+				(xy 16 18) (xy 194 18) (xy 194 132) (xy 16 132)
+			)
+		)
+	)
+	(zone
+		(net "GND")
 		(layer "In1.Cu")
 		(hatch edge 0.5)
@@
 		(polygon
 			(pts
-				(xy 115.45 31) (xy 115.45 33.8) (xy 116.75 33.8) (xy 116.75 39.95) (xy 115.45 39.95) (xy 115.45 42.75)
-				(xy 119.125 42.75) (xy 119.125 31)
+				(xy 115.45 30.8) (xy 95 33) (xy 95 39) (xy 108.5 39) (xy 115.45 34) (xy 116.75 34) (xy 116.75 39.7)
+				(xy 115.45 39.7) (xy 103.7 54.113333) (xy 103.7 66) (xy 108 66) (xy 108.1 54.7) (xy 119.12 42.9)
+				(xy 119.12 30.8)
 			)
 		)

Commit message: grounding CM5
Parts:
- moved TP4 3.21 mm to (114.5, 73.5)
Routing:
- net GND: track 0.00 -> 31.1 mm, vias 30 -> 45

Commit message: more psu
Parts:
- added C80: 10uF, Capacitor_SMD:C_1206_3216Metric, F.Cu at (168.0, 45.8)
- added C82: 22uF, Capacitor_SMD:C_1206_3216Metric, F.Cu at (168.0, 50.5)
- C43: footprint Capacitor_Tantalum_SMD:CP_EIA-7343-31_Kemet-D -> Capacitor_THT:CP_Radial_D8.0mm_P3.50mm
- C53: value 10uF -> 4.7uF; footprint Capacitor_SMD:C_1206_3216Metric -> Capacitor_SMD:C_1812_4532Metric
- moved TP6 25.7 mm to (118.5, 28.1)
- moved R29 19.1 mm to (96.4, 27.2), turned to 180 degrees
- moved U10 13.4 mm to (95.5, 30.2)
- moved C16 13.3 mm to (95.3, 33.1)
- moved C38 13.2 mm to (95.4, 34.9)
- moved J21 11.0 mm to (98.3, 41.4)
- moved C39 10.7 mm to (92.7, 30.1), turned to -90 degrees
- moved TP5 8.73 mm to (159.8, 26.4)
- moved C79 6.10 mm to (119.1, 74.9)
- moved R52 6.10 mm to (122.8, 82.3)
- moved TP4 6.10 mm to (114.3, 79.7)
- moved C71 6.10 mm to (123.3, 62.1)
- moved CM2 6.10 mm to (101.6, 55.6)
- moved J11 6.10 mm to (112.1, 59.9)
- moved C57 6.10 mm to (133.5, 75.8)
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Routing:
- net GND: track 31.1 -> 64.2 mm, vias 45 -> 87
- net /Connectivity/VBUS: track 0.00 -> 21.5 mm
- net +5VP: track 16.6 -> 28.2 mm
- net /Power Supply/polarity_checked: track 8.22 -> 18.3 mm
- net +10V: track 0.00 -> 7.42 mm
- net Net-(U10-ILIM): track 0.00 -> 1.88 mm
- added copper zone on F.Cu, net +10V
Other:
- board text added: "Line in (bal.)"
- board text removed: "Line (bal.)"

Commit message: opamp incl power routed
Parts:
- removed C64: 100nF, Capacitor_SMD:C_1206_3216Metric_Pad1.33x1.80mm_HandSolder
- C54, C82: footprint Capacitor_SMD:C_1206_3216Metric -> Capacitor_SMD:C_1210_3225Metric_Pad1.33x2.70mm_HandSolder
- C55, C80: value 10uF -> 22uF; footprint Capacitor_SMD:C_1206_3216Metric -> Capacitor_SMD:C_1210_3225Metric_Pad1.33x2.70mm_HandSolder
- moved TP2 14.4 mm to (162.6, 62.5)
- moved C82 0.85 mm to (168.8, 50.8)
- moved C80 0.80 mm to (168.8, 45.8)
- moved R35 0.55 mm to (164.8, 64.2)
- moved R36 0.55 mm to (167.8, 64.2)
- moved C53 0.41 mm to (163.9, 55.4)
- moved C54 0.32 mm to (165.6, 50.8)
- moved R33 0.30 mm to (168.2, 69.7)
- moved D8 0.20 mm to (34.0, 68.7)
- moved C55 0.11 mm to (165.6, 45.8)
- moved R34 0.05 mm to (161.3, 71.0)
Routing:
- net Net-(R37-Pad1): track 0.00 -> 30.7 mm
- net Net-(R34-Pad2): track 0.00 -> 27.1 mm
- net +10V: track 7.42 -> 30.2 mm, vias 0 -> 2
- net GND: track 64.2 -> 84.3 mm, vias 87 -> 90
- net Net-(R54-Pad2): track 0.00 -> 15.5 mm
- net Net-(C81-Pad1): track 0.00 -> 14.5 mm, vias 0 -> 1
- net Net-(U13-SET): track 0.00 -> 8.45 mm
- net Net-(U14B--): track 0.00 -> 8.27 mm
- net VBIAS_4V: track 0.00 -> 8.02 mm
- net Net-(U14A--): track 0.00 -> 7.59 mm
- net Net-(U14A-+): track 0.00 -> 6.75 mm
- net Net-(D3-A2): track 0.00 -> 6.12 mm
- net /Audio/TAC_IN1P: track 0.00 -> 5.85 mm
- net /Audio/TAC_IN1M: track 0.00 -> 5.74 mm
- net Net-(R54-Pad1): track 0.00 -> 4.17 mm
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
Commit message: Routing IC1
Parts:
- moved TP4 19.8 mm to (96.9, 70.1)
- moved R16 7.03 mm to (117.1, 81.0)
- moved D6 5.43 mm to (114.4, 81.9)
- moved C71 0.60 mm to (123.3, 61.5)
- moved R52 0.15 mm to (122.8, 82.4)
- moved R51 0.05 mm to (124.3, 82.4)
Routing:
- net +5VP: track 28.2 -> 52.9 mm
- net /Power Supply/5V_PG: track 4.14 -> 28.0 mm, vias 0 -> 2
- net 3V3_CODEC: track 0.00 -> 11.7 mm
- net CM5_3V: track 0.00 -> 8.35 mm, vias 0 -> 2
- net Net-(IC1-DREG): track 0.00 -> 3.95 mm
- net /Audio/conf_i2c_scl: track 0.00 -> 2.66 mm, vias 0 -> 1
- net Net-(IC1-VREF): track 0.00 -> 2.56 mm
- net /Audio/conf_i2c_sda: track 0.00 -> 2.43 mm, vias 0 -> 1
- net /Audio/TAC_IN2P: track 0.00 -> 1.38 mm, vias 0 -> 1
- net /Audio/TAC_IN2M: track 0.00 -> 0.93 mm, vias 0 -> 1
- net GND: vias 90 -> 94

Commit message: more routing.
Parts:
- moved TP4 1.02 mm to (97.1, 71.1)
- moved D6 1.00 mm to (114.5, 82.9)
- moved C67 1.00 mm to (125.3, 70.6)
- moved C66 0.95 mm to (125.1, 72.4)
- moved R43 0.89 mm to (135.6, 85.3)
- moved R44 0.89 mm to (134.1, 85.3)
- moved R16 0.71 mm to (116.4, 80.9), turned to 0 degrees
Routing:
- net /Audio/TAC_OUT2M: track 0.00 -> 129.9 mm, vias 0 -> 1
- net /Audio/TAC_OUT2P: track 0.00 -> 129.3 mm, vias 0 -> 1
- net Net-(C63-Pad2): track 0.00 -> 40.7 mm
- net Net-(C62-Pad2): track 0.00 -> 37.9 mm
- net /Audio/TAC_OUT1P: track 0.00 -> 27.9 mm, vias 0 -> 2
- net /Audio/conf_i2c_sda: track 2.43 -> 29.8 mm, vias 1 -> 2
- net CM5_3V: track 8.35 -> 35.1 mm
- net /Audio/TAC_OUT1M: track 0.00 -> 25.8 mm, vias 0 -> 2
- net /Audio/conf_i2c_scl: track 2.66 -> 27.9 mm, vias 1 -> 2
- net /Audio/audio_pcm_fs: track 0.00 -> 24.5 mm, vias 0 -> 2
- net Net-(C63-Pad1): track 0.00 -> 21.2 mm
- net /Audio/audio_pcm_din: track 0.00 -> 21.0 mm
- net /Audio/audio_pcm_dout: track 0.00 -> 21.0 mm
- net /Audio/audio_pcm_clk: track 0.00 -> 19.6 mm
- net Net-(C62-Pad1): track 0.00 -> 16.7 mm
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
Commit message: more routing.
Parts:
- removed TP4: CM5_3V3, TestPoint:TestPoint_Pad_D1.5mm
- moved TP6 6.35 mm to (113.2, 31.6)
- moved R51 1.72 mm to (122.7, 82.9), turned to 180 degrees
- moved R52 1.04 mm to (122.7, 81.4), turned to 0 degrees
- moved C68 0.76 mm to (118.7, 80.5)
- moved C70 0.76 mm to (120.5, 80.2)
- moved D6 0.76 mm to (115.2, 83.2)
- moved R16 0.57 mm to (116.0, 80.5), turned to 90 degrees
Routing:
- net /Audio/TAC_OUT1M: track 25.8 -> 165.2 mm
- net /Audio/TAC_OUT1P: track 27.9 -> 149.5 mm
- net ESP_BOOT: track 0.00 -> 45.4 mm, vias 0 -> 1
- net UI_UART_RX: track 0.00 -> 45.0 mm
- net ESP_RESET: track 0.00 -> 44.5 mm, vias 0 -> 1
- net UI_UART_TX: track 0.00 -> 36.9 mm
- net CM_BOOT: track 0.00 -> 12.6 mm
- net Net-(D4-A2): track 0.00 -> 11.4 mm
- net Net-(D5-A2): track 0.00 -> 11.4 mm
- net /Audio/CM5_LED_ACT: track 0.00 -> 10.7 mm
- net /Audio/conf_i2c_sda: track 29.8 -> 34.2 mm
- net /Audio/TAC_OUT2M: track 129.9 -> 127.0 mm
- net +5VP: track 52.9 -> 55.7 mm
- net /Audio/conf_i2c_scl: track 27.9 -> 30.6 mm
- net Net-(D6-A): track 0.00 -> 1.84 mm
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