File: pedalboard-hw.kicad_pcb (KiCad board)
At the start: 4 copper layers, 174 x 111 mm, 120 parts, among them IC1 TAC5212IRGER, J10 USB-A HOST, J11 CM5 BOOT, J13 Headphones 3.5mm, J16 CM5 UART DEBUG, J18 GUITAR INPUT, J19 LINE OUT LEFT, J20 LINE OUT RIGHT, J21 UI LINK 2x5, J22 BALANCED LINE INPUT, J6 Screw_Terminal_01x02, J7 Barrel_Jack_MountingPin, J9 USB-C SERVICE, Q1 FDS4435BZ, SW11 EM-02-Q, U10 AP22653, U11 TPD2E2U06DCK, U13 LT3042, U14 OPA1656ID, U15 TPS7A20, U16 TPD2E2U06DCK, U6 TLVM13660

Commit message: yet more routing.
Parts:
- moved U16 0.55 mm to (47.8, 30.6)
- moved R30 0.40 mm to (49.8, 28.9)
- moved R31 0.34 mm to (45.6, 28.9)
Routing:
- net /Connectivity/USB_SERVICE_P: track 0.00 -> 78.3 mm
- net /Connectivity/USB_SERVICE_N: track 0.00 -> 76.0 mm
- net /Connectivity/USB_HOST_VBUS_EN: track 0.00 -> 75.2 mm, vias 0 -> 2
- net /Connectivity/USB_HOST_P: track 0.00 -> 45.9 mm
- net /Connectivity/USB_HOST_N: track 0.00 -> 44.9 mm
- net Net-(D8-A2): track 0.00 -> 8.65 mm
- net /Connectivity/USB_SERVICE_VBUS_UNUSED: track 0.00 -> 6.49 mm
- net Net-(C77-Pad2): track 0.00 -> 1.91 mm
- net Net-(J9-CC2): track 0.00 -> 1.70 mm
- net Net-(J9-CC1): track 0.00 -> 1.69 mm
- net GND: track 85.3 -> 85.6 mm, vias 107 -> 112

Commit message: bit more routing.
Routing:
- net Net-(D9-A2): track 0.00 -> 7.21 mm
- net Net-(C75-Pad2): track 0.00 -> 1.91 mm
Changed lines of the file:
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@@
+	)
+	(segment
+		(start 34.685 92.765)
+		(end 34.65 92.8)
+		(width 0.3)
+		(layer "F.Cu")
+		(net "Net-(D9-A2)")
+	)
+	(segment
+		(start 38.225 92.8)
+		(end 38.425 93)
+		(width 0.3)
+		(layer "F.Cu")
+		(net "Net-(D9-A2)")
+	)
+	(segment
+		(start 34 92.8)
+		(end 34.65 92.8)
+		(width 0.3)
+		(layer "F.Cu")
+		(net "Net-(D9-A2)")
+	)
+	(segment
+		(start 34.685 90.115)
+		(end 34.685 92.765)
+		(width 0.3)
+		(layer "F.Cu")
+		(net "Net-(D9-A2)")
+	)
+	(segment
+		(start 34.65 92.8)
+		(end 38.225 92.8)
+		(width 0.3)
+		(layer "F.Cu")
+		(net "Net-(D9-A2)")
 	)
 	(segment
@@
 	)
 	(segment
+		(start 40.075 93)
+		(end 41.275 93)
+		(width 0.3)
+		(layer "F.Cu")
+		(net "Net-(C75-Pad2)")
+	)
+	(segment
+		(start 41.275 93)
+		(end 41.775 93.5)
+		(width 0.3)
+		(layer "F.Cu")
+		(net "Net-(C75-Pad2)")
+	)
+	(segment

Commit message: Fiddles. Moved J6
Parts:
- moved C50 19.1 mm to (59.0, 25.1), turned to -90 degrees
- moved J6 18.1 mm to (157.2, 28.2)
- moved R53 17.1 mm to (57.0, 25.8), turned to 90 degrees
- moved TP5 7.99 mm to (155.8, 33.4)
Routing:
- net CHASSIS: track 0.00 -> 44.1 mm
- net GND: track 85.6 -> 83.7 mm, vias 112 -> 115
- net Net-(C62-Pad2): track 37.9 -> 39.1 mm
- net /Connectivity/USB_SERVICE_N: track 76.0 -> 75.1 mm
